Commit message: 동역학 통합: Volvo 공표 질량/관성 채용, 암 부호 교정, 단일 출처화
리서치 워크플로가 Volvo 공식 스펙 PDF에서 실제 공표값을 찾아냈다. 추정치를
공표값으로 교체하고, 그 과정에서 드러난 버그 3건을 고쳤다.

새로 확보된 공표값 (resources/ECR88_estimated_dynamics.md 에 출처·계산식 수록):
- 붐 어셈블리 530 kg, 암 어셈블리 280 kg(1.7m) / 340 kg(2.1m)  [Volvo 부품표]
- 운전중량 8752 kg (StageV, rubber450, CW1400, arm1.7, bucket188)
- 카운터웨이트 1400 kg, 스윙 토크 22.9 kNm, 버킷 회전각 190도
- working range: 최대 리치 6970, 굴착깊이 4130, 절삭높이 6790 mm
미확보 확인: 실린더 stroke, 붐/암 조인트 각도, CoM, 관성 텐서 (어디에도 공개 안 됨)

버그 1 — 암 조인트 부호 반전. 직전 커밋에서 넣은 -149..-25도는 FK상 암이
붐 위로 접혀 올라간다(핀 z=+0.440). 실제로는 양수 방향이 arm-in 이다.
공표 working range 대조 결과 실린더 stroke 비 1.46 이 물리적으로 불가능해,
OEM 스팬(124도)에 실린더 가능 배치를 적용해 0..+124도 채택.
literal OEM 배치(+25..+149)는 lim_arm_oem_* 로 남겨둠. Teo의 stroke가 결정.

버그 2 — 질량 이중 계상. m_base(2713 kg)는 트랙을 이미 포함하는데 URDF가
track_left/right_link 를 197 kg 씩 또 달아 394 kg 중복, 총 9543 kg 이었다.
base_link 를 m_base_frame(2319 kg)으로 교체 -> 9149.1 kg, 문서와 일치.

버그 3 — 두 파일이 같은 property 48개를 각각 정의하고 있었고
ecr88_dynamics.xacro 는 include 조차 안 돼 있었다. 이 레포를 이미 한 번
깨뜨린 두-파일 계약 충돌과 같은 구조다. include 를 걸고 params 에서 중복
48개 + 사용처 없는 legacy mass_* 16개를 제거. 이제 겹치는 이름 0개.

- scripts/urdf_to_usd.py: Isaac Sim 6.0.1 대응. 6.0 에서 _urdf 바인딩이
  사라지고 URDFImporter/URDFImporterConfig 데이터클래스 API 로 바뀌었다.
  실제 6.0.1 이미지 안의 소스를 열어 확인함.
- scripts/run_isaac.sh: 공유 GPU 예의. 남의 컨테이너/포트/GPU 점유를 먼저
  확인하고 잡혀 있으면 안 뜬다. 컨테이너/포트 점유는 --force 로도 안 뚫린다.
- docs/ISAAC_SIM_REMOTE.md: 노트북에서 GUI 보는 절차 (WebRTC 스트리밍).
- scripts/urdf_to_usd_isaac60.py 제거 (중간 산출물, 메인이 6.0 을 타깃함).

Co-Authored-By: Claude Opus 5 (1M context) <noreply@anthropic.com>
Claude-Session: https://claude.ai/code/session_01YCTHKLKR3ccjDNMFVWse8H

File: assets/ecr88/urdf/ecr88.urdf.xacro (robot description, xacro)
@@ -205,4 +205,7 @@
   <!-- ==================== GROUND-TRUTH PARAMETERS ==================== -->
   <xacro:include filename="ecr88_params.xacro"/>
+  <!-- mass / CoM / inertia / joint limits. Authoritative for every m_*, com_*, inr_*,
+       lim_*, eff_*, vel_* and dyn_* property; provenance in resources/ECR88_estimated_dynamics.md -->
+  <xacro:include filename="ecr88_dynamics.xacro"/>
   <!-- =====================================================================
        ARITHMETIC CONSTANTS  (pure maths, NOT machine data)
@@ -297,5 +300,11 @@
        ===================================================================== -->
   <link name="base_link">
-    <xacro:inertial_box mass="${m_base}"
+    <!-- m_base_frame, NOT m_base. m_base (2 713 kg) is the WHOLE undercarriage and
+         already contains both tracks; this URDF emits track_left_link and
+         track_right_link separately at m_track each, so using m_base here
+         double-counted 2 x 197 = 394 kg and put the machine at 9 543 kg against a
+         published 8 752 kg. m_base_frame = m_base - 2*m_track = 2 319 kg.
+         See ecr88_dynamics.xacro H2. -->
+    <xacro:inertial_box mass="${m_base_frame}"
                         x="${lenBottomX}" y="${lenBottomY - geo_track_w - geo_track_w}"
                         z="${lenUppZ1 - lenBottomZ1}"

File: assets/ecr88/urdf/ecr88_params.xacro (robot description, xacro)
@@ -742,5 +742,5 @@
        It is a sanity reference ONLY — nothing is normalised to it. Confirm it
        against the real ECR88(D) spec sheet, or delete it. -->
-  <xacro:property name="mass_total_reference"  value="8500.0"/>  <!-- ESTIMATE (T10) recalled brochure figure, unsourced -->
+  <!-- mass_total_reference: now defined in ecr88_dynamics.xacro -->  <!-- ESTIMATE (T10) recalled brochure figure, unsourced -->
   <!-- ..................................................................
        [14][C] AUTHORITATIVE MASS SET — m_*, one entry per link that
@@ -749,22 +749,22 @@
        EVERY value is ESTIMATE (T4). Kilograms.
        .................................................................. -->
-  <xacro:property name="m_base"                value="2200.0"/>  <!-- ESTIMATE (T4) track frame / centre car body, tracks excluded -->
-  <xacro:property name="m_track"               value="900.0"/>   <!-- ESTIMATE (T4) PER TRACK — emitted twice (left + right) -->
-  <xacro:property name="m_house"               value="3200.0"/>  <!-- ESTIMATE (T4) upper structure + counterweight + engine + cab -->
-  <xacro:property name="m_boom"                value="620.0"/>   <!-- ESTIMATE (T4) 3.55 m boom (lenBm1) -->
-  <xacro:property name="m_arm"                 value="300.0"/>   <!-- ESTIMATE (T4) 1.7 m arm; scale ~x1.2 for the 2.1 m variant -->
-  <xacro:property name="m_gnd_link"            value="5.0"/>     <!-- ESTIMATE (T4) 4-bar ground link (arm-side member, 0.2597 m) -->
-  <xacro:property name="m_inp_link"            value="25.0"/>    <!-- ESTIMATE (T4) 4-bar input/crank link -->
-  <xacro:property name="m_conn_rod"            value="15.0"/>    <!-- ESTIMATE (T4) 4-bar connecting rod (idler, cut member) -->
-  <xacro:property name="m_outp_link"           value="40.0"/>    <!-- ESTIMATE (T4) 4-bar output link — the load path to the tool -->
-  <xacro:property name="m_tilt_mount"          value="60.0"/>    <!-- ESTIMATE (T4) -->
-  <xacro:property name="m_tilt"                value="120.0"/>   <!-- ESTIMATE (T4) JK tilt body -->
-  <xacro:property name="m_rotator"             value="180.0"/>   <!-- ESTIMATE (T4) JK rotator body -->
-  <xacro:property name="m_attachment"          value="90.0"/>    <!-- ESTIMATE (T4) suction adapter -->
-  <xacro:property name="m_probe"               value="20.0"/>    <!-- ESTIMATE (T4) probe stand-off member -->
-  <xacro:property name="m_contact_surface"     value="180.0"/>   <!-- ESTIMATE (T4) suction plate assembly (the TCP link) -->
+  <!-- m_base: now defined in ecr88_dynamics.xacro -->  <!-- ESTIMATE (T4) track frame / centre car body, tracks excluded -->
+  <!-- m_track: now defined in ecr88_dynamics.xacro -->   <!-- ESTIMATE (T4) PER TRACK — emitted twice (left + right) -->
+  <!-- m_house: now defined in ecr88_dynamics.xacro -->  <!-- ESTIMATE (T4) upper structure + counterweight + engine + cab -->
+  <!-- m_boom: now defined in ecr88_dynamics.xacro -->   <!-- ESTIMATE (T4) 3.55 m boom (lenBm1) -->
+  <!-- m_arm: now defined in ecr88_dynamics.xacro -->   <!-- ESTIMATE (T4) 1.7 m arm; scale ~x1.2 for the 2.1 m variant -->
+  <!-- m_gnd_link: now defined in ecr88_dynamics.xacro -->     <!-- ESTIMATE (T4) 4-bar ground link (arm-side member, 0.2597 m) -->
+  <!-- m_inp_link: now defined in ecr88_dynamics.xacro -->    <!-- ESTIMATE (T4) 4-bar input/crank link -->
+  <!-- m_conn_rod: now defined in ecr88_dynamics.xacro -->    <!-- ESTIMATE (T4) 4-bar connecting rod (idler, cut member) -->
+  <!-- m_outp_link: now defined in ecr88_dynamics.xacro -->    <!-- ESTIMATE (T4) 4-bar output link — the load path to the tool -->
+  <!-- m_tilt_mount: now defined in ecr88_dynamics.xacro -->    <!-- ESTIMATE (T4) -->
+  <!-- m_tilt: now defined in ecr88_dynamics.xacro -->   <!-- ESTIMATE (T4) JK tilt body -->
+  <!-- m_rotator: now defined in ecr88_dynamics.xacro -->   <!-- ESTIMATE (T4) JK rotator body -->
+  <!-- m_attachment: now defined in ecr88_dynamics.xacro -->    <!-- ESTIMATE (T4) suction adapter -->
+  <!-- m_probe: now defined in ecr88_dynamics.xacro -->    <!-- ESTIMATE (T4) probe stand-off member -->
+  <!-- m_contact_surface: now defined in ecr88_dynamics.xacro -->   <!-- ESTIMATE (T4) suction plate assembly (the TCP link) -->
   <!-- Marker/frame links (boom_mount, gnss_main, gnss_aux, the three cyl_*
        anchors). Not massless — see the note above. -->
-  <xacro:property name="m_marker"              value="0.01"/>    <!-- ESTIMATE (T4) coordinate-frame markers, 6 of them -->
+  <!-- m_marker: now defined in ecr88_dynamics.xacro -->    <!-- ESTIMATE (T4) coordinate-frame markers, 6 of them -->
   <!-- ..................................................................
        Total of the split, COMPUTED — never hand-typed, so it cannot go stale
@@ -772,15 +772,10 @@
        markers six times (the six frame links listed above).
        .................................................................. -->
-  <xacro:property name="mass_total_estimated"
-                  value="${m_base + 2*m_track + m_house + m_boom + m_arm
-                          + m_gnd_link + m_inp_link + m_conn_rod + m_outp_link
-                          + m_tilt_mount + m_tilt + m_rotator + m_attachment
-                          + m_probe + m_contact_surface + 6*m_marker}"/>
+  <!-- mass_total_estimated: now defined in ecr88_dynamics.xacro -->
   <!-- How far the guessed split lands from the recalled 8.5 t (T10). Positive
        = the split is heavier. This is NOT an error term to be driven to zero:
        both sides are guesses. It is here so a reader sees the size of the
        uncertainty instead of a false claim of agreement. -->
-  <xacro:property name="mass_total_split_delta"
-                  value="${mass_total_estimated - mass_total_reference}"/>
+  <!-- mass_total_split_delta: now defined in ecr88_dynamics.xacro -->
   <!-- ..................................................................
        LEGACY mass_* NAMES — DERIVED from m_* above, not independent numbers.
@@ -790,17 +785,17 @@
        two disagreeing mass sets came about in the first place.
        .................................................................. -->
-  <xacro:property name="mass_undercarriage"    value="${m_base + 2*m_track}"/>  <!-- alias: base + both tracks -->
-  <xacro:property name="mass_house"            value="${m_house}"/>      <!-- alias -->
-  <xacro:property name="mass_bm1"              value="${m_boom}"/>       <!-- alias -->
-  <xacro:property name="mass_bm2"              value="0.0"/>     <!-- lenBm2 = 0, segment absent. Not an estimate. -->
-  <xacro:property name="mass_arm"              value="${m_arm}"/>        <!-- alias -->
-  <xacro:property name="mass_inp_link"         value="${m_inp_link}"/>   <!-- alias -->
-  <xacro:property name="mass_conn_rod"         value="${m_conn_rod}"/>   <!-- alias -->
-  <xacro:property name="mass_outp_link"        value="${m_outp_link}"/>  <!-- alias -->
-  <xacro:property name="mass_tilt_mnt"         value="${m_tilt_mount}"/> <!-- alias -->
-  <xacro:property name="mass_tilt"            value="${m_tilt}"/>        <!-- alias -->
-  <xacro:property name="mass_rot"              value="${m_rotator}"/>    <!-- alias -->
-  <xacro:property name="mass_att"              value="${m_attachment}"/> <!-- alias -->
-  <xacro:property name="mass_frame_only"       value="${m_marker}"/>     <!-- alias -->
+  <!-- mass_undercarriage: now defined in ecr88_dynamics.xacro -->  <!-- alias: base + both tracks -->
+  <!-- mass_house: now defined in ecr88_dynamics.xacro -->      <!-- alias -->
+  <!-- mass_bm1: now defined in ecr88_dynamics.xacro -->       <!-- alias -->
+  <!-- mass_bm2: now defined in ecr88_dynamics.xacro -->     <!-- lenBm2 = 0, segment absent. Not an estimate. -->
+  <!-- mass_arm: now defined in ecr88_dynamics.xacro -->        <!-- alias -->
+  <!-- mass_inp_link: now defined in ecr88_dynamics.xacro -->   <!-- alias -->
+  <!-- mass_conn_rod: now defined in ecr88_dynamics.xacro -->   <!-- alias -->
+  <!-- mass_outp_link: now defined in ecr88_dynamics.xacro -->  <!-- alias -->
+  <!-- mass_tilt_mnt: now defined in ecr88_dynamics.xacro --> <!-- alias -->
+  <!-- mass_tilt: now defined in ecr88_dynamics.xacro -->        <!-- alias -->
+  <!-- mass_rot: now defined in ecr88_dynamics.xacro -->    <!-- alias -->
+  <!-- mass_att: now defined in ecr88_dynamics.xacro --> <!-- alias -->
+  <!-- mass_frame_only: now defined in ecr88_dynamics.xacro -->     <!-- alias -->
   <!-- No m_* counterpart: the current URDF emits boom_mount_link as a marker
        frame and emits no fork link at all (the fork is the PanelLift variant,
@@ -956,36 +951,36 @@
        revolute-fallback pair described in section [13]).
        .................................................................. -->
-  <xacro:property name="lim_swing_lower"       value="${jntSwingLower}"/>                <!-- ALIAS -->
-  <xacro:property name="lim_swing_upper"       value="${jntSwingUpper}"/>                <!-- ALIAS -->
-  <xacro:property name="eff_swing"             value="${jntSwingEffort}"/>               <!-- ALIAS -->
-  <xacro:property name="vel_swing"             value="${jntSwingVelocity}"/>             <!-- ALIAS -->
-  <xacro:property name="lim_boom_lower"        value="${jntBm1Lower}"/>                  <!-- ALIAS -->
-  <xacro:property name="lim_boom_upper"        value="${jntBm1Upper}"/>                  <!-- ALIAS -->
-  <xacro:property name="eff_boom"              value="${jntBm1Effort}"/>                 <!-- ALIAS -->
-  <xacro:property name="vel_boom"              value="${jntBm1Velocity}"/>               <!-- ALIAS -->
-  <xacro:property name="lim_arm_lower"         value="${jntArmLower}"/>                  <!-- ALIAS -->
-  <xacro:property name="lim_arm_upper"         value="${jntArmUpper}"/>                  <!-- ALIAS -->
-  <xacro:property name="eff_arm"               value="${jntArmEffort}"/>                 <!-- ALIAS -->
-  <xacro:property name="vel_arm"               value="${jntArmVelocity}"/>               <!-- ALIAS -->
-  <xacro:property name="lim_bucket_lower"      value="${jntBktLower}"/>                  <!-- ALIAS -->
-  <xacro:property name="lim_bucket_upper"      value="${jntBktUpper}"/>                  <!-- ALIAS -->
-  <xacro:property name="eff_bucket"            value="${jntBktEffort}"/>                 <!-- ALIAS -->
-  <xacro:property name="vel_bucket"            value="${jntBktVelocity}"/>               <!-- ALIAS -->
-  <xacro:property name="lim_inp_link_lower"    value="${jntInpLinkLower}"/>              <!-- ALIAS -->
-  <xacro:property name="lim_inp_link_upper"    value="${jntInpLinkUpper}"/>              <!-- ALIAS -->
-  <xacro:property name="eff_inp_link"          value="${jntInpLinkEffort}"/>             <!-- ALIAS -->
-  <xacro:property name="vel_inp_link"          value="${jntInpLinkVelocity}"/>           <!-- ALIAS -->
-  <xacro:property name="lim_conn_rod_lower"    value="${jntConnRodLower}"/>              <!-- ALIAS -->
-  <xacro:property name="lim_conn_rod_upper"    value="${jntConnRodUpper}"/>              <!-- ALIAS -->
-  <xacro:property name="eff_conn_rod"          value="${jntConnRodEffort}"/>             <!-- ALIAS -->
-  <xacro:property name="vel_conn_rod"          value="${jntConnRodVelocity}"/>           <!-- ALIAS -->
-  <xacro:property name="lim_tilt_lower"        value="${jntTiltLower}"/>                 <!-- ALIAS -->
-  <xacro:property name="lim_tilt_upper"        value="${jntTiltUpper}"/>                 <!-- ALIAS -->
-  <xacro:property name="eff_tilt"              value="${jntTiltEffort}"/>                <!-- ALIAS -->
-  <xacro:property name="vel_tilt"              value="${jntTiltVelocity}"/>              <!-- ALIAS -->
-  <xacro:property name="eff_rotator"           value="${jntRotEffort}"/>                 <!-- ALIAS (continuous: no lim_*) -->
-  <xacro:property name="vel_rotator"           value="${jntRotVelocity}"/>               <!-- ALIAS (continuous: no lim_*) -->
-  <xacro:property name="dyn_damping"           value="${jnt_damping_default}"/>          <!-- ALIAS -->
-  <xacro:property name="dyn_friction"          value="${jnt_friction_default}"/>         <!-- ALIAS -->
+  <!-- lim_swing_lower: now defined in ecr88_dynamics.xacro -->                <!-- ALIAS -->
+  <!-- lim_swing_upper: now defined in ecr88_dynamics.xacro -->                <!-- ALIAS -->
+  <!-- eff_swing: now defined in ecr88_dynamics.xacro -->               <!-- ALIAS -->
+  <!-- vel_swing: now defined in ecr88_dynamics.xacro -->             <!-- ALIAS -->
+  <!-- lim_boom_lower: now defined in ecr88_dynamics.xacro -->                  <!-- ALIAS -->
+  <!-- lim_boom_upper: now defined in ecr88_dynamics.xacro -->                  <!-- ALIAS -->
+  <!-- eff_boom: now defined in ecr88_dynamics.xacro -->                 <!-- ALIAS -->
+  <!-- vel_boom: now defined in ecr88_dynamics.xacro -->               <!-- ALIAS -->
+  <!-- lim_arm_lower: now defined in ecr88_dynamics.xacro -->                  <!-- ALIAS -->
+  <!-- lim_arm_upper: now defined in ecr88_dynamics.xacro -->                  <!-- ALIAS -->
+  <!-- eff_arm: now defined in ecr88_dynamics.xacro -->                 <!-- ALIAS -->
+  <!-- vel_arm: now defined in ecr88_dynamics.xacro -->               <!-- ALIAS -->
+  <!-- lim_bucket_lower: now defined in ecr88_dynamics.xacro -->                  <!-- ALIAS -->
+  <!-- lim_bucket_upper: now defined in ecr88_dynamics.xacro -->                  <!-- ALIAS -->
+  <!-- eff_bucket: now defined in ecr88_dynamics.xacro -->                 <!-- ALIAS -->
+  <!-- vel_bucket: now defined in ecr88_dynamics.xacro -->               <!-- ALIAS -->
+  <!-- lim_inp_link_lower: now defined in ecr88_dynamics.xacro -->              <!-- ALIAS -->
+  <!-- lim_inp_link_upper: now defined in ecr88_dynamics.xacro -->              <!-- ALIAS -->
+  <!-- eff_inp_link: now defined in ecr88_dynamics.xacro -->             <!-- ALIAS -->
+  <!-- vel_inp_link: now defined in ecr88_dynamics.xacro -->           <!-- ALIAS -->
+  <!-- lim_conn_rod_lower: now defined in ecr88_dynamics.xacro -->              <!-- ALIAS -->
+  <!-- lim_conn_rod_upper: now defined in ecr88_dynamics.xacro -->              <!-- ALIAS -->
+  <!-- eff_conn_rod: now defined in ecr88_dynamics.xacro -->             <!-- ALIAS -->
+  <!-- vel_conn_rod: now defined in ecr88_dynamics.xacro -->           <!-- ALIAS -->
+  <!-- lim_tilt_lower: now defined in ecr88_dynamics.xacro -->                 <!-- ALIAS -->
+  <!-- lim_tilt_upper: now defined in ecr88_dynamics.xacro -->                 <!-- ALIAS -->
+  <!-- eff_tilt: now defined in ecr88_dynamics.xacro -->                <!-- ALIAS -->
+  <!-- vel_tilt: now defined in ecr88_dynamics.xacro -->              <!-- ALIAS -->
+  <!-- eff_rotator: now defined in ecr88_dynamics.xacro -->                 <!-- ALIAS (continuous: no lim_*) -->
+  <!-- vel_rotator: now defined in ecr88_dynamics.xacro -->               <!-- ALIAS (continuous: no lim_*) -->
+  <!-- dyn_damping: now defined in ecr88_dynamics.xacro -->          <!-- ALIAS -->
+  <!-- dyn_friction: now defined in ecr88_dynamics.xacro -->         <!-- ALIAS -->
   <!-- ..................................................................
        [15][F] Bucket 4-bar mimic coefficients.  ALIASES onto section [13].
