Commit message: 프리미티브 형상 개선: 굴삭기로 보이게
Isaac Sim 에서 처음 띄워보니 키네마틱은 맞는데 굴삭기로 안 보였다.
붐 발치 위치도 리치도 지면 접촉도 정상인데, 모든 부재가 곧은 막대이고
상부체가 2.28 x 2.46 x 2.03 m 짜리 민짜 큐브 하나였다. 마일스톤 1 의
목적이 "카메라/라이다를 어디에 달지 눈으로 판단"인데 큐브는 아무것도
말해주지 않는다.

조인트 원점, 링크 길이, 질량, 관성은 하나도 건드리지 않았다. 형상만 바뀐다.

- 붐: 곧은 실린더 -> 굽은 2 세그먼트 빔. Volvo 공표 mono boom 이
  3700 x 1244 x 335 인데, 곧은 3.55 m 부재라면 envelope 높이가 제 단면
  깊이 수준이어야 한다. 즉 1244 는 굽힘이다. 코드 위로의 융기 =
  1.244 - 0.335 = 0.909 m, 정점은 코드의 45%.
  세그먼트 양 끝은 실제 핀(붐 발치, arm_joint)이라 융기값을 바꿔도
  키네마틱은 불변이다.
- 암: 실린더 -> 공표 단면 박스. 2.1m 는 562 x 305, 1.7m 는 518 x 305
  (variant 로 자동 선택).
- 상부체: 큐브 하나 -> 데크 + 카운터웨이트(후방) + 캡(전방, +Y 오프셋).
  캡을 +Y 로 둔 건 붐 발치가 -Y 쪽이기 때문(distChsToBmMnt_y = -0.15).
  캡 높이는 독립 추정이 아니라 geo_house_h 의 나머지로 잡아서
  데크 + 캡 = geo_house_h 가 정확히 유지된다. 전체 envelope 불변.
- 하부: 도저 블레이드 추가. 장식이 아니라 캘리브레이션 절차가
  "Dozer full down (Pitch > 5)" 로 이 자세를 전제한다. 조인트는 만들지
  않았다 - 파라미터 시트에 블레이드 조인트가 없고, 없는 가동부를 트리에
  넣으면 아무도 명령할 수 없는 관절이 생긴다.

캡/카운터웨이트를 처음엔 시트의 코너 원점(lenUppX1)으로 배치했다가
되돌렸다. 데크 박스는 T6 에 따라 스윙축 중심인데 코너 원점을 섞으면
카운터웨이트가 장비 한가운데로, 캡이 코 앞으로 튀어나간다. 같은 규약
(중심 + 크기)으로 통일.

새 매크로 detail: viscol 과 같은 visual+collision 쌍이지만 use_meshes 가
켜지면 통째로 사라진다. 메쉬가 들어오면 형상 전체를 메쉬가 들고 있으므로.

USD 재생성. 검증 18 pass / 0 fail.

Co-Authored-By: Claude Opus 5 <noreply@anthropic.com>
Claude-Session: https://claude.ai/code/session_01YCTHKLKR3ccjDNMFVWse8H

File: assets/ecr88/urdf/ecr88.urdf.xacro (robot description, xacro)
@@ -276,4 +276,24 @@
     </collision>
   </xacro:macro>
+  <!-- An EXTRA placeholder solid on a link that already has a viscol. Same visual +
+       collision pair, but it vanishes entirely once real meshes are switched on,
+       because a mesh already carries the whole shape. Use it to break one link into
+       the few solids that make it recognisable (deck / cab / counterweight, or the
+       two halves of a bent boom) instead of one featureless box.
+       Shape only: it never touches a joint origin, a length, a mass or an inertia. -->
+  <xacro:macro name="detail"
+               params="material:='xpanner_yellow' xyz:='0 0 0' rpy:='0 0 0' *prim">
+    <xacro:unless value="$(arg use_meshes)">
+      <visual>
+        <origin xyz="${xyz}" rpy="${rpy}"/>
+        <geometry><xacro:insert_block name="prim"/></geometry>
+        <material name="${material}"/>
+      </visual>
+      <collision>
+        <origin xyz="${xyz}" rpy="${rpy}"/>
+        <geometry><xacro:insert_block name="prim"/></geometry>
+      </collision>
+    </xacro:unless>
+  </xacro:macro>
   <!-- A structural member drawn as a capsule-ish cylinder running from the link origin
        to the offset (dx,dy,dz). Length and pitch are DERIVED from the offset, so the
@@ -318,4 +338,13 @@
       <box size="${lenBottomX} ${lenBottomY - geo_track_w - geo_track_w} ${lenUppZ1 - lenBottomZ1}"/>
     </xacro:viscol>
+    <!-- SHAPE: dozer blade. The machine has one and the calibration procedure gates on
+         it ("Dozer full down, Pitch angle > 5"), so it is not decoration for the SIL
+         work either. Drawn on base_link and NOT articulated: there is no blade joint
+         in the parameter sheet, and inventing one would put a moving part in the tree
+         that nothing can command. Cosmetic mass is ignored - it sits inside m_base. -->
+    <xacro:detail material="xpanner_dark"
+                  xyz="${lenBottomX * half + geo_blade_t * half} 0 ${lenBottomZ1 + geo_blade_h * half}">
+      <box size="${geo_blade_t} ${lenBottomY} ${geo_blade_h}"/>
+    </xacro:detail>
   </link>
   <!-- Tracks. FIXED for now (T12): travel is not simulated yet. To drive the machine,
@@ -360,8 +389,34 @@
                         x="${lenUppX}" y="${lenUppY}" z="${geo_house_h}"
                         xyz="0 0 ${lenUppZ1 + geo_house_h * half}"/>
+    <!-- SHAPE: the upper structure used to be ONE box, lenUppX x lenUppY x geo_house_h,
+         i.e. a 2.28 x 2.46 x 2.03 m cube that swallowed the boom foot and told a viewer
+         nothing. It is now the three solids a person recognises. Same footprint, same
+         overall height, same m_house and same inertia box: only the picture changed.
+           deck  - engine/pump deck, full footprint, low
+           cw    - counterweight, at the rear (-X), the ECR88 tail swing mass
+           cab   - operator cab, front, offset to +Y so the boom runs up its -Y side,
+                   which is where the boom foot actually is (distChsToBmMnt_y = -0.15)
+         The cab is the piece that matters for milestone 1: camera and lidar candidates
+         get judged against where the operator can and cannot see. -->
     <xacro:viscol name="house_link" material="xpanner_yellow"
-                  xyz="0 0 ${lenUppZ1 + geo_house_h * half}">
-      <box size="${lenUppX} ${lenUppY} ${geo_house_h}"/>
-    </xacro:viscol>
+                  xyz="0 0 ${lenUppZ1 + geo_deck_h * half}">
+      <box size="${lenUppX} ${lenUppY} ${geo_deck_h}"/>
+    </xacro:viscol>
+    <!-- Placed on the SAME convention as the deck box above: centred on the swing axis
+         in X and Y, sizes only (T6). Do not reach for lenUppX1 / lenUppY1 here - those
+         are the sheet's corner origins, which T6 concludes are in the Leica instrument
+         frame, and mixing them with the centred deck puts the counterweight in the
+         middle of the machine and the cab out past its nose.
+         Counterweight at the rear (-X), cab at the front (+X) and offset to +Y so the
+         boom runs up its -Y side, which is the side the boom foot is actually on
+         (distChsToBmMnt_y = -0.15). -->
+    <xacro:detail material="xpanner_dark"
+                  xyz="${-(lenUppX * half) + geo_cw_x * half} 0 ${lenUppZ1 + geo_cw_h * half}">
+      <box size="${geo_cw_x} ${lenUppY * 0.94} ${geo_cw_h}"/>
+    </xacro:detail>
+    <xacro:detail material="xpanner_yellow"
+                  xyz="${(lenUppX * half) - geo_cab_x * half} ${(lenUppY * half) - geo_cab_y * half} ${lenUppZ1 + geo_deck_h + geo_cab_h * half}">
+      <box size="${geo_cab_x} ${geo_cab_y} ${geo_cab_h}"/>
+    </xacro:detail>
   </link>
   <joint name="swing_joint" type="revolute">
@@ -448,8 +503,31 @@
                              length="${lenBm1 + lenBm2}"
                              xyz="${(lenBm1 + lenBm2) * half} 0 0" rpy="0 ${half_pi} 0"/>
+    <!-- SHAPE: a real excavator boom is BENT, and the bend is the single strongest
+         visual cue that this is an excavator rather than a robot arm. Volvo publishes
+         the mono boom as 3700 long x 1244 high x 335 wide; a straight 3.55 m member
+         would envelope at about its own section depth, so the 1244 is the arc. The
+         rise above the pin-to-pin chord is therefore 1.244 - 0.335 = 0.909 m
+         (geo_boom_rise), apexed at 45% of the chord.
+         Drawn as two straight box segments, foot -> apex -> tip. The ENDPOINTS are
+         the real pins: segment A starts at the boom foot (0,0,0) and segment B ends
+         at the arm pin (lenBm1, 0, 0), which is exactly where arm_joint is. So the
+         bend is cosmetic and the kinematics are untouched: no matter what
+         geo_boom_rise is set to, both pins stay put.
+         Pitch of a box drawn along +X and rotated by p about +Y sends +X to
+         (cos p, 0, -sin p), hence the minus sign in the atan2 arguments. -->
+    <xacro:property name="bm_apex_x" value="${(lenBm1 + lenBm2) * geo_boom_apex_frac}"/>
+    <xacro:property name="bm_tip_dx" value="${(lenBm1 + lenBm2) - bm_apex_x}"/>
+    <!-- foot -> apex -->
     <xacro:viscol name="boom_link" material="xpanner_yellow"
-                  xyz="${(lenBm1 + lenBm2) * half} 0 0" rpy="0 ${half_pi} 0">
-      <cylinder radius="${geo_boom_r}" length="${lenBm1 + lenBm2}"/>
-    </xacro:viscol>
+                  xyz="${bm_apex_x * half} 0 ${geo_boom_rise * half}"
+                  rpy="0 ${-atan2(geo_boom_rise, bm_apex_x)} 0">
+      <box size="${sqrt(bm_apex_x * bm_apex_x + geo_boom_rise * geo_boom_rise)} ${geo_boom_sec_w} ${geo_boom_sec_h}"/>
+    </xacro:viscol>
+    <!-- apex -> arm pin -->
+    <xacro:detail material="xpanner_yellow"
+                  xyz="${bm_apex_x + bm_tip_dx * half} 0 ${geo_boom_rise * half}"
+                  rpy="0 ${atan2(geo_boom_rise, bm_tip_dx)} 0">
+      <box size="${sqrt(bm_tip_dx * bm_tip_dx + geo_boom_rise * geo_boom_rise)} ${geo_boom_sec_w} ${geo_boom_sec_h}"/>
+    </xacro:detail>
   </link>
   <joint name="boom_joint" type="revolute">
@@ -499,7 +577,12 @@
     <xacro:inertial_cylinder mass="${m_arm}" radius="${geo_arm_r}" length="${lenArm}"
                              xyz="${lenArm * half} 0 0" rpy="0 ${half_pi} 0"/>
+    <!-- SHAPE: the dipper is a fabricated box beam, not a rod. Volvo publishes the
+         2.1 m dipper as 2684 x 562 x 305 mm (1.7 m: 2283 x 518 x 305), so use the
+         published section instead of geo_arm_r. Length stays lenArm (pin to pin);
+         the published 2684 is the physical part envelope and is a different
+         quantity, see the note in ecr88_params.xacro [15][D2]. -->
     <xacro:viscol name="arm_link" material="xpanner_yellow"
-                  xyz="${lenArm * half} 0 0" rpy="0 ${half_pi} 0">
-      <cylinder radius="${geo_arm_r}" length="${lenArm}"/>
+                  xyz="${lenArm * half} 0 0">
+      <box size="${lenArm} ${geo_arm_sec_w} ${geo_arm_sec_h}"/>
     </xacro:viscol>
   </link>

File: assets/ecr88/urdf/ecr88_params.xacro (robot description, xacro)
@@ -959,4 +959,54 @@
   <xacro:property name="geo_marker_r"          value="0.03"/>    <!-- ESTIMATE (T11) m, cosmetic -->
   <!-- ..................................................................
+       [15][D2] SHAPE, not size.  Added 2026-09-11 after the first Isaac Sim
+       view: the kinematics were right but the machine did not read as an
+       excavator, because every member was a straight rod and the whole upper
+       structure was one featureless 2 m cube.
+       None of this changes a joint origin, a link length, a mass or an inertia.
+       It only changes what the placeholder primitives LOOK like, and it is worth
+       doing because the entire point of milestone 1 is letting people judge
+       sensor placement by eye. A cube tells them nothing about where a camera
+       would actually see from.
+       The section dimensions below are PUBLISHED: Volvo "Boom and dipper arm"
+       dimension table (the sheet Teo shared 2026-09-11).
+           Mono boom 3.55 m : length 3700, height 1244, width  335 mm
+           Dipper 1.7 m     : length 2283, height  518, width  305 mm
+           Dipper 2.1 m     : length 2684, height  562, width  305 mm
+       Note LENGTH here is the physical part envelope (3700), which is longer than
+       lenBm1 = 3550, the PIN-TO-PIN distance the kinematics use. They are different
+       quantities and both are correct; do not "fix" one against the other.
+       .................................................................. -->
+  <xacro:property name="geo_boom_sec_h"        value="0.335"/>   <!-- PUBLISHED  boom section width 335 mm, used as the beam depth -->
+  <xacro:property name="geo_boom_sec_w"        value="0.335"/>   <!-- PUBLISHED  boom width 335 mm -->
+  <!-- The published 1244 mm boom envelope height is what the BEND costs: a straight
+       3.55 m member would envelope at roughly its own section depth. So the rise of
+       the arc above the pin-to-pin chord is the envelope height minus the section:
+       1.244 - 0.335 = 0.909 m. ASSUMPTION: apex at 45% of the chord, which is where
+       it sits on the Volvo side-view drawing. Both numbers are cosmetic. -->
+  <xacro:property name="geo_boom_h_env"        value="1.244"/>   <!-- PUBLISHED  boom envelope height 1244 mm -->
+  <xacro:property name="geo_boom_rise"         value="${geo_boom_h_env - geo_boom_sec_h}"/>
+  <xacro:property name="geo_boom_apex_frac"    value="0.45"/>    <!-- ASSUMPTION  cosmetic -->
+  <!-- Dipper section, per variant. -->
+  <xacro:property name="geo_arm_sec_h"         value="${0.562 if lenArm &gt; 1.9 else 0.518}"/> <!-- PUBLISHED -->
+  <xacro:property name="geo_arm_sec_w"         value="0.305"/>   <!-- PUBLISHED  both dipper lengths are 305 mm wide -->
+  <!-- Upper structure broken into the three masses a person actually recognises.
+       Heights split geo_house_h; footprint split lenUppX / lenUppY. All ASSUMPTION,
+       all cosmetic, none of it feeds inertia (m_house keeps its single box). -->
+  <xacro:property name="geo_deck_h"            value="${geo_house_h * 0.46}"/>  <!-- ASSUMPTION  engine deck height -->
+  <xacro:property name="geo_cab_x"             value="1.00"/>    <!-- ASSUMPTION  cab footprint, m -->
+  <xacro:property name="geo_cab_y"             value="0.92"/>    <!-- ASSUMPTION -->
+  <!-- Cab height is the REMAINDER of geo_house_h above the deck, not an independent
+       guess. That keeps the three solids inside the same overall envelope the single
+       box used, so the machine does not silently grow taller than the T6 derivation
+       says it is: deck + cab = geo_house_h exactly. -->
+  <xacro:property name="geo_cab_h"             value="${geo_house_h - geo_deck_h}"/>  <!-- DERIVED from geo_house_h -->
+  <xacro:property name="geo_cw_x"              value="0.62"/>    <!-- ASSUMPTION  counterweight depth, m -->
+  <xacro:property name="geo_cw_h"              value="${geo_house_h * 0.62}"/>  <!-- ASSUMPTION -->
+  <!-- Dozer blade. The machine has one: the calibration procedure gates on
+       "Dozer full down (Pitch angle > 5)". Cosmetic here, but it is the shape that
+       most says "compact excavator" at a glance. Drawn on base_link, not articulated. -->
+  <xacro:property name="geo_blade_h"           value="0.42"/>    <!-- ASSUMPTION  m -->
+  <xacro:property name="geo_blade_t"           value="0.13"/>    <!-- ASSUMPTION  m -->
+  <!-- ..................................................................
        [15][E] Joint limits / actuation.  ALL ALIASES onto section [13].
        No number is authored here — section [13] holds every value together

Commit message: 형상 2차: 트랙 실루엣, 숏테일 후미 호, 캡 글라스하우스, 붐/암 테이퍼
- 트랙: 슬래브 -> 아이들러/스프로킷에 감긴 벨트 실루엣. 구름반경은
  측정된 차체 높이(lenUppZ1 - lenBottomZ1)의 절반이고 두 휠을 양 끝에서
  반경만큼 안쪽에 두어 벨트 envelope 이 정확히 lenBottomX 를 유지한다.
  측정값에서 유도되므로 실측 하부 치수를 넘어설 수 없다. 둥근 것만 장식.
- 상부 후미: 스윙축 중심 원호 추가. ECR88 은 reduced tail swing 기종이고
  후미가 원호인 게 이 모델의 존재 이유이자 위에서 볼 때 가장 알아보기 쉬운
  특징이다. 반경 = 측정 하우스 길이의 절반이라 데크 박스와 같은 후단에서
  끝난다.
- 캡: 단일 박스 -> 하부 몸체 + 안쪽으로 들어간 글라스하우스.
  마일스톤 1 이 판정되는 지점이라(카메라/라이다 후보를 오퍼레이터 시야와
  대조) 캡이 캡으로 보여야 한다.
- 붐/암: 팁 쪽 단면 테이퍼. 모든 굴삭기 부재가 핀 쪽으로 좁아진다.

전부 형상뿐. 조인트 원점, 링크 길이, 질량, 관성 불변. 검증 18 pass / 0 fail.
USD 지오메트리 52 -> 66 개.

부수 수정: 측면도 미리보기 스크립트가 URDF 실린더 축을 잘못 투영하고 있었다.
<cylinder> 축은 자기 프레임의 +Z 이고 element 의 rpy 가 이미 방향을 잡는데,
그 위에 Y축 pi/2 를 한 번 더 걸고 있었다. 그래서 Y축/Z축 실린더 -- 정확히
방금 추가한 트랙 휠과 후미 호 -- 가 전부 X 방향으로 누운 것처럼 그려졌다.
로컬 실루엣(반경은 X, 길이는 Z)을 그리도록 수정.

Co-Authored-By: Claude Opus 5 <noreply@anthropic.com>
Claude-Session: https://claude.ai/code/session_01YCTHKLKR3ccjDNMFVWse8H

File: assets/ecr88/urdf/ecr88.urdf.xacro (robot description, xacro)
@@ -355,8 +355,21 @@
                         x="${lenBottomX}" y="${geo_track_w}" z="${lenUppZ1 - lenBottomZ1}"
                         xyz="0 0 ${(lenBottomZ1 + lenUppZ1) * half}"/>
+    <!-- SHAPE: belt over idler + sprocket, not a slab. The straight run carries the
+         collision; the two end wheels are what make the silhouette read as a crawler.
+         Envelope still spans exactly lenBottomX - see geo_track_wheel_dx. -->
     <xacro:viscol name="track_left_link" material="xpanner_dark"
                   xyz="0 0 ${(lenBottomZ1 + lenUppZ1) * half}">
-      <box size="${lenBottomX} ${geo_track_w} ${lenUppZ1 - lenBottomZ1}"/>
-    </xacro:viscol>
+      <box size="${lenBottomX - geo_track_r - geo_track_r} ${geo_track_w} ${geo_track_h}"/>
+    </xacro:viscol>
+    <xacro:detail material="xpanner_dark"
+                  xyz="${geo_track_wheel_dx} 0 ${(lenBottomZ1 + lenUppZ1) * half}"
+                  rpy="${half_pi} 0 0">
+      <cylinder radius="${geo_track_r}" length="${geo_track_w}"/>
+    </xacro:detail>
+    <xacro:detail material="xpanner_dark"
+                  xyz="${-geo_track_wheel_dx} 0 ${(lenBottomZ1 + lenUppZ1) * half}"
+                  rpy="${half_pi} 0 0">
+      <cylinder radius="${geo_track_r}" length="${geo_track_w}"/>
+    </xacro:detail>
   </link>
   <joint name="track_left_joint" type="fixed">
@@ -369,8 +382,19 @@
                         x="${lenBottomX}" y="${geo_track_w}" z="${lenUppZ1 - lenBottomZ1}"
                         xyz="0 0 ${(lenBottomZ1 + lenUppZ1) * half}"/>
+    <!-- SHAPE: mirror of track_left_link. See the note there. -->
     <xacro:viscol name="track_right_link" material="xpanner_dark"
                   xyz="0 0 ${(lenBottomZ1 + lenUppZ1) * half}">
-      <box size="${lenBottomX} ${geo_track_w} ${lenUppZ1 - lenBottomZ1}"/>
-    </xacro:viscol>
+      <box size="${lenBottomX - geo_track_r - geo_track_r} ${geo_track_w} ${geo_track_h}"/>
+    </xacro:viscol>
+    <xacro:detail material="xpanner_dark"
+                  xyz="${geo_track_wheel_dx} 0 ${(lenBottomZ1 + lenUppZ1) * half}"
+                  rpy="${half_pi} 0 0">
+      <cylinder radius="${geo_track_r}" length="${geo_track_w}"/>
+    </xacro:detail>
+    <xacro:detail material="xpanner_dark"
+                  xyz="${-geo_track_wheel_dx} 0 ${(lenBottomZ1 + lenUppZ1) * half}"
+                  rpy="${half_pi} 0 0">
+      <cylinder radius="${geo_track_r}" length="${geo_track_w}"/>
+    </xacro:detail>
   </link>
   <joint name="track_right_joint" type="fixed">
@@ -415,7 +439,23 @@
       <box size="${geo_cw_x} ${lenUppY * 0.94} ${geo_cw_h}"/>
     </xacro:detail>
+    <!-- SHORT TAIL SWING. The ECR88 is a reduced-tail-swing machine: its house rear is
+         a circular ARC about the swing axis, which is the whole point of the model and
+         the most recognisable thing about its silhouette from above. Radius is half the
+         measured house length, so the arc reaches exactly the same rear extent as the
+         deck box and never grows the envelope. -->
+    <xacro:detail material="xpanner_dark"
+                  xyz="0 0 ${lenUppZ1 + geo_cw_h * half}">
+      <cylinder radius="${lenUppX * half}" length="${geo_cw_h}"/>
+    </xacro:detail>
+    <!-- Cab: lower body + inset glasshouse, so it reads as a cab and not a second
+         counterweight. This is the piece milestone 1 is judged against - camera and
+         lidar candidates get argued about relative to what the operator can see. -->
     <xacro:detail material="xpanner_yellow"
-                  xyz="${(lenUppX * half) - geo_cab_x * half} ${(lenUppY * half) - geo_cab_y * half} ${lenUppZ1 + geo_deck_h + geo_cab_h * half}">
-      <box size="${geo_cab_x} ${geo_cab_y} ${geo_cab_h}"/>
+                  xyz="${(lenUppX * half) - geo_cab_x * half} ${(lenUppY * half) - geo_cab_y * half} ${lenUppZ1 + geo_deck_h + geo_cab_h * 0.30}">
+      <box size="${geo_cab_x} ${geo_cab_y} ${geo_cab_h * 0.60}"/>
+    </xacro:detail>
+    <xacro:detail material="xpanner_frame"
+                  xyz="${(lenUppX * half) - geo_cab_x * half} ${(lenUppY * half) - geo_cab_y * half} ${lenUppZ1 + geo_deck_h + geo_cab_h * 0.80}">
+      <box size="${geo_cab_x - geo_cab_upper_inset} ${geo_cab_y - geo_cab_upper_inset} ${geo_cab_h * 0.40}"/>
     </xacro:detail>
   </link>
@@ -528,5 +568,5 @@
                   xyz="${bm_apex_x + bm_tip_dx * half} 0 ${geo_boom_rise * half}"
                   rpy="0 ${atan2(geo_boom_rise, bm_tip_dx)} 0">
-      <box size="${sqrt(bm_tip_dx * bm_tip_dx + geo_boom_rise * geo_boom_rise)} ${geo_boom_sec_w} ${geo_boom_sec_h}"/>
+      <box size="${sqrt(bm_tip_dx * bm_tip_dx + geo_boom_rise * geo_boom_rise)} ${geo_boom_sec_w * geo_boom_taper} ${geo_boom_sec_h * geo_boom_taper}"/>
     </xacro:detail>
   </link>
@@ -583,7 +623,12 @@
          quantity, see the note in ecr88_params.xacro [15][D2]. -->
     <xacro:viscol name="arm_link" material="xpanner_yellow"
-                  xyz="${lenArm * half} 0 0">
-      <box size="${lenArm} ${geo_arm_sec_w} ${geo_arm_sec_h}"/>
-    </xacro:viscol>
+                  xyz="${lenArm * 0.25} 0 0">
+      <box size="${lenArm * half} ${geo_arm_sec_w} ${geo_arm_sec_h}"/>
+    </xacro:viscol>
+    <!-- Tapered tip half. Every dipper narrows toward the bucket pin. Cosmetic. -->
+    <xacro:detail material="xpanner_yellow"
+                  xyz="${lenArm * 0.75} 0 0">
+      <box size="${lenArm * half} ${geo_arm_sec_w * geo_arm_taper} ${geo_arm_sec_h * geo_arm_taper}"/>
+    </xacro:detail>
   </link>
   <joint name="arm_joint" type="revolute">

File: assets/ecr88/urdf/ecr88_params.xacro (robot description, xacro)
@@ -1008,4 +1008,20 @@
   <xacro:property name="geo_blade_h"           value="0.42"/>    <!-- ASSUMPTION  m -->
   <xacro:property name="geo_blade_t"           value="0.13"/>    <!-- ASSUMPTION  m -->
+  <!-- Crawler side profile. A track is a belt wrapped round an idler and a sprocket,
+       so its silhouette is a rounded rectangle, not a slab. Rolling radius is half the
+       track height (lenUppZ1 - lenBottomZ1, the measured car-body clearance), and the
+       two wheels sit one radius in from each end so the belt envelope still spans
+       exactly lenBottomX. Derived from measured numbers, so the track can never
+       outgrow the surveyed undercarriage; only the roundness is cosmetic. -->
+  <xacro:property name="geo_track_h"           value="${lenUppZ1 - lenBottomZ1}"/>   <!-- DERIVED -->
+  <xacro:property name="geo_track_r"           value="${geo_track_h * half}"/>       <!-- DERIVED -->
+  <xacro:property name="geo_track_wheel_dx"    value="${lenBottomX * half - geo_track_r}"/> <!-- DERIVED -->
+  <!-- Cab glasshouse: the upper box is inset so the cab reads as a cab rather than a
+       second counterweight. Cosmetic. -->
+  <xacro:property name="geo_cab_upper_inset"   value="0.14"/>    <!-- ASSUMPTION  m -->
+  <!-- Boom taper: the tip section is narrower than the foot section on every excavator
+       boom. Fraction of geo_boom_sec_*. Cosmetic. -->
+  <xacro:property name="geo_boom_taper"        value="0.72"/>    <!-- ASSUMPTION -->
+  <xacro:property name="geo_arm_taper"         value="0.68"/>    <!-- ASSUMPTION -->
   <!-- ..................................................................
        [15][E] Joint limits / actuation.  ALL ALIASES onto section [13].
