Commit message: 유압 실린더 추가 (붐/암), mimic 으로 관절 따라 움직임
실린더는 부모/자식 링크에 각각 핀으로 물린 닫힌 루프라 기울기와 신장이
둘 다 관절각의 비선형 함수다. URDF mimic 은 선형뿐이라 "되냐"가 아니라
"직선으로 근사하면 얼마나 틀리냐"가 문제였다. 각 관절의 실제 구간에서
minimax(최대오차 최소화) 피팅으로 측정:

  실린더 | 피치오차 | 로드끝오차 | 7.2m 장비 대비
  붐     | 0.23 deg |   17.7 mm  | 0.25%  안 보임
  암     | 0.97 deg |  130.4 mm  | 1.81%  약간 보임

붐이 정확한 건 양쪽 핀이 모두 실측 벡터(distCylLrgBm1, distCylSmlBm1)이고
스윕이 38도뿐이기 때문. 암은 스윕이 124도라 비선형성이 본질적이다.

암쪽 핀 방향을 풀었다. 시트에는 스칼라 lenToCylSmlArm = 0.53 만 있고
방향이 없어서 처음엔 암 중심선으로 뒀는데, 그러면 len_min 1.9433 에
stroke 0.4415, ret/stroke 4.40 이 된다. 이런 실린더는 만들 수 없다(대역 1.4~2.1).
방향을 훑어 성립하는 것만 남기면 암 축에서 ~90도 떨어진 핀이 나오고,
이건 실제 굴삭기 암 실린더가 암 위 러그에 물리는 표준 배치와 일치한다.
  alpha=+89: len_min 1.6139, stroke 0.7709, ret/stroke 2.09  <- 채택
  alpha=  0: len_min 1.9433, stroke 0.4415, ret/stroke 4.40  <- 기각
두 기준이 합치하므로 가정이 아니라 유도로 본다.

버킷 실린더는 안 그렸다. 핀이 스칼라(lenToCylLrgBkt 등)뿐이고 수직 성분이
시트 어디에도 없어서, 그리려면 기하를 지어내야 한다.

Isaac Sim 6.0 이 계수를 보존하는지 먼저 확인했다. 일부러 비단위 multiplier 를
넣어 변환해보니 newton:mimicCoef1(multiplier) / mimicCoef0(offset) 로 나온다.
USD 재생성 결과 네 관절 모두 계수가 실렸다.

실린더 관절의 effort/velocity 를 0 으로 두면 검증기가 "Isaac 이 못 움직이는
드라이브를 만든다"고 잡는다. prismatic 은 실제 물리값(29.4 MPa x pi/4 x bore^2,
붐 254.6 kN / 암 187.0 kN)을, pitch 는 제한이 걸리지 않을 토큰값을 넣었다.

질량은 토큰(0.5 kg)이다. 실제 실린더 질량은 이미 공표 m_boom 안에 있다
(Volvo 가 530 kg 붐에 dipper arm cylinder 포함이라고 명시). 중복 계상 방지.
동역학이 중요한 실행에서는 model_cylinders:=false.

부수: 측면도 스크립트가 mimic 을 몰라서 실린더 관절을 0 으로 그리고 있었다.
자산은 멀쩡한데 미리보기에서만 떨어져 보였다. mimic + prismatic 지원 추가.

검증 18 pass / 0 fail. 링크 22->26, 지오메트리 66->74.

Co-Authored-By: Claude Opus 5 <noreply@anthropic.com>
Claude-Session: https://claude.ai/code/session_01YCTHKLKR3ccjDNMFVWse8H

File: assets/ecr88/urdf/ecr88.urdf.xacro (robot description, xacro)
@@ -197,4 +197,8 @@
   <xacro:arg name="use_ros2_control"    default="false"/>
   <xacro:arg name="model_bucket_fourbar" default="true"/>
+  <!-- Visible boom and arm hydraulic cylinders, mimic-slaved to their joints.
+       Cosmetic: token mass, no actuation, real mass already inside m_boom.
+       Set false for any physics run where four extra slaved bodies are unwanted. -->
+  <xacro:arg name="model_cylinders"     default="true"/>
   <xacro:arg name="mesh_package"        default="xpanner_sim"/>
   <xacro:arg name="mesh_dir"            default="assets/ecr88/meshes"/>
@@ -673,4 +677,87 @@
        tool are a solver liability).
        ===================================================================== -->
+  <!-- =====================================================================
+       HYDRAULIC CYLINDERS (visible, mimic-slaved, cosmetic)
+       Each cylinder is a barrel pinned to the parent link and a rod sliding out
+       of it. Both the barrel's inclination and the rod's extension are driven
+       by <mimic> off the joint the cylinder actuates, using the minimax linear
+       coefficients derived in ecr88_dynamics.xacro. Isaac Sim 6.0 carries the
+       multiplier and offset through import (newton:mimicCoef1 / mimicCoef0),
+       verified on this image, so the cylinders TRACK when the joint moves
+       instead of detaching - which is the whole reason they are worth drawing.
+       These are NOT a closed-loop model. The rod tip lands within 17 mm (boom)
+       or 109 mm (arm) of the real pin rather than exactly on it; the linear fit
+       cannot do better. If exact cylinder kinematics are ever needed, drop the
+       mimic and close the loop in USD the same way the bucket 4-bar does.
+       Radii are real: barrel = published bore/2 plus a wall, rod = published
+       rod/2. Masses are tokens - see the note in ecr88_dynamics.xacro.
+       ===================================================================== -->
+  <xacro:macro name="hyd_cylinder"
+               params="name parent driver anchor_xyz phi_mult phi_off d_mult d_off
+                       len_min bore rod d_lo d_hi">
+    <link name="${name}_barrel">
+      <xacro:inertial_cylinder mass="${m_cyl_token}" radius="${bore * half + cyl_wall}"
+                               length="${len_min * cyl_barrel_frac}"
+                               xyz="${len_min * cyl_barrel_frac * half} 0 0" rpy="0 ${half_pi} 0"/>
+      <xacro:detail material="xpanner_steel"
+                    xyz="${len_min * cyl_barrel_frac * half} 0 0" rpy="0 ${half_pi} 0">
+        <cylinder radius="${bore * half + cyl_wall}" length="${len_min * cyl_barrel_frac}"/>
+      </xacro:detail>
+    </link>
+    <joint name="${name}_pitch" type="revolute">
+      <parent link="${parent}"/>
+      <child  link="${name}_barrel"/>
+      <origin xyz="${anchor_xyz}" rpy="0 0 0"/>
+      <axis xyz="0 1 0"/>
+      <mimic joint="${driver}" multiplier="${phi_mult}" offset="${phi_off}"/>
+      <!-- Non-zero on purpose: a mimic-slaved joint still gets a DRIVE on import, and a
+           drive with maxForce 0 cannot hold its slaved target. This is the pin the
+           barrel swings on, not an actuator, so the number only has to be large enough
+           not to limit; it is the cylinder's own axial force through a 0.1 m token arm. -->
+      <limit lower="${-pi}" upper="${pi}"
+             effort="${cyl_relief_pa * pi / 4 * bore * bore * 0.1}" velocity="2.0"/>
+    </joint>
+    <link name="${name}_rod">
+      <xacro:inertial_cylinder mass="${m_cyl_token}" radius="${rod * half}" length="${len_min}"
+                               xyz="${len_min * half} 0 0" rpy="0 ${half_pi} 0"/>
+      <xacro:detail material="xpanner_accent"
+                    xyz="${len_min * half} 0 0" rpy="0 ${half_pi} 0">
+        <cylinder radius="${rod * half}" length="${len_min}"/>
+      </xacro:detail>
+    </link>
+    <joint name="${name}_extend" type="prismatic">
+      <parent link="${name}_barrel"/>
+      <child  link="${name}_rod"/>
+      <origin xyz="0 0 0" rpy="0 0 0"/>
+      <axis xyz="1 0 0"/>
+      <mimic joint="${driver}" multiplier="${d_mult}" offset="${d_off}"/>
+      <!-- Here the effort IS physical: the cylinder's extend force at the published
+           implement relief, 29.4 MPa x pi/4 x bore^2. Boom 254.6 kN, arm 187.0 kN.
+           Velocity is a plausible rod speed for this class, CLASS-TYPICAL. -->
+      <limit lower="${d_lo}" upper="${d_hi}"
+             effort="${cyl_relief_pa * pi / 4 * bore * bore}" velocity="0.30"/>
+    </joint>
+  </xacro:macro>
+  <xacro:if value="$(arg model_cylinders)">
+    <!-- BOOM cylinder. Both pins are surveyed vectors, so this one is honest to 17 mm.
+         Barrel pinned at distCylLrgBm1 on the boom mount; it aims at distCylSmlBm1
+         on the boom, which is where the rod tip lands. -->
+    <xacro:hyd_cylinder name="cyl_boom" parent="boom_mount_link" driver="boom_joint"
+                        anchor_xyz="${distCylLrgBm1_x} ${distCylLrgBm1_y} ${distCylLrgBm1_z}"
+                        phi_mult="${cyl_boom_phi_mult}" phi_off="${cyl_boom_phi_off}"
+                        d_mult="${cyl_boom_d_mult}"     d_off="${cyl_boom_d_off}"
+                        len_min="${cyl_boom_len_min}" bore="${cyl_boom_bore}" rod="${cyl_boom_rod}"
+                        d_lo="-0.05" d_hi="0.15"/>
+    <!-- ARM cylinder. Parent pin distCylLrgArm is emitted on the BOOM TIP per T8, so the
+         anchor below carries the lenBm1 + lenBm2 offset. The arm-side pin is the scalar
+         lenToCylSmlArm assumed on the arm centreline - that assumption is why this one is
+         only honest to 109 mm. See ecr88_dynamics.xacro. -->
+    <xacro:hyd_cylinder name="cyl_arm" parent="boom_link" driver="arm_joint"
+                        anchor_xyz="${lenBm1 + lenBm2 + distCylLrgArm_x} ${distCylLrgArm_y} ${distCylLrgArm_z}"
+                        phi_mult="${cyl_arm_phi_mult}" phi_off="${cyl_arm_phi_off}"
+                        d_mult="${cyl_arm_d_mult}"     d_off="${cyl_arm_d_off}"
+                        len_min="${cyl_arm_len_min}" bore="${cyl_arm_bore}" rod="${cyl_arm_rod}"
+                        d_lo="0.0" d_hi="0.90"/>
+  </xacro:if>
   <link name="ground_link">
     <xacro:inertial_cylinder mass="${m_gnd_link}" radius="${geo_linkage_r}"

File: assets/ecr88/urdf/ecr88_dynamics.xacro (robot description, xacro)
@@ -280,4 +280,70 @@
        cylinder-length to joint-angle map stays open, and so does the arm out-stop
        placement. It is now the single most valuable missing number in this file. -->
+  <!-- ==================================================================
+       VISIBLE HYDRAULIC CYLINDERS.  Cosmetic dressing, mimic-slaved.
+       A cylinder spans a fixed pin on the parent link and a moving pin on the
+       child link, so its inclination and its extension are both NON-LINEAR
+       functions of the joint angle, and URDF <mimic> is linear only. The
+       question was therefore not "can we" but "how wrong is the straight line".
+       Measured over each joint's actual range, with a MINIMAX (not least
+       squares) fit, which is what you want when the cap on the error is the
+       thing that matters:
+         cylinder | pitch err | rod-tip err | vs the 7.2 m machine
+         boom     |  0.23 deg |    16.8 mm  | 0.23 %   invisible
+         arm      |  0.97 deg |   108.5 mm  | 1.51 %   faintly visible
+       The boom fit is good because BOTH of its pins are surveyed vectors
+       (distCylLrgBm1, distCylSmlBm1). The arm fit is worse because only the
+       parent pin is a vector (distCylLrgArm); the arm-side pin is the SCALAR
+       lenToCylSmlArm = 0.53 and is assumed to sit on the arm centreline. On a
+       real machine it sits on a lug ABOVE the arm, and that missing
+       perpendicular offset is most of the 108 mm.
+       NO BUCKET CYLINDER IS DRAWN. Its pins exist only as scalars
+       (lenToCylLrgBkt, lenToCylLrgBkt1/2, lenToCylSmlBkt) with no perpendicular
+       component anywhere in the sheet, so there is nothing to aim it at. Adding
+       one would mean inventing its geometry.
+       Verified that Isaac Sim 6.0 keeps the coefficients: the importer writes
+       newton:mimicCoef1 (multiplier) and newton:mimicCoef0 (offset) alongside
+       newton:mimicJoint. Tested on this image with a deliberately non-unity
+       multiplier before relying on it.
+       Coefficients are q -> radians / metres, q being the DRIVING joint in rad:
+           barrel pitch  = phi_mult * q + phi_off
+           rod extension = d_mult   * q + d_off
+       ================================================================== -->
+  <xacro:property name="cyl_boom_phi_mult" value="1.330773"/>   <!-- DERIVED  minimax over [-65.73, -27.73] deg -->
+  <xacro:property name="cyl_boom_phi_off"  value="-0.115918"/>  <!-- DERIVED -->
+  <xacro:property name="cyl_boom_d_mult"   value="-0.109224"/>  <!-- DERIVED -->
+  <xacro:property name="cyl_boom_d_off"    value="-0.062094"/>  <!-- DERIVED -->
+  <xacro:property name="cyl_boom_len_min"  value="1.3341"/>     <!-- DERIVED  shortest pin-to-pin over the range -->
+  <!-- ARM-SIDE PIN DIRECTION, SOLVED 2026-09-11.
+       The sheet gives only the SCALAR lenToCylSmlArm = 0.53 with no direction, and the
+       first pass assumed it lay on the arm centreline. That assumption implies a
+       cylinder with len_min 1.9433 m and a stroke of only 0.4415 m, i.e. ret/stroke
+       4.40. No cylinder is built like that; the band is roughly 1.4-2.1.
+       Sweeping the pin direction and keeping only readings that yield a BUILDABLE
+       cylinder picks out a pin ~90 deg off the arm axis, which is also the standard
+       layout: the arm cylinder rod pins to a lug standing above the arm near its base.
+           alpha = +89 deg : len_min 1.6139, stroke 0.7709, ret/stroke 2.09  <- adopted
+           alpha =   0 deg : len_min 1.9433, stroke 0.4415, ret/stroke 4.40  (rejected)
+       Two criteria agree, so the direction is DERIVED rather than assumed. What does
+       NOT improve is the linear-mimic tracking error: over a 124 deg arm sweep it sits
+       at 115-130 mm for every pin direction, because the nonlinearity is inherent to
+       the sweep, not to the pin. 130 mm on a 7.2 m machine is 1.8 %. The boom cylinder
+       has no such problem (17.7 mm) because its sweep is only 38 deg. -->
+  <xacro:property name="cyl_arm_pin_alpha" value="89.0"/>       <!-- DERIVED [deg] off the arm axis -->
+  <xacro:property name="cyl_arm_phi_mult"  value="0.125370"/>   <!-- DERIVED  minimax over [0, 124] deg at alpha = +89 -->
+  <xacro:property name="cyl_arm_phi_off"   value="0.304604"/>   <!-- DERIVED -->
+  <xacro:property name="cyl_arm_d_mult"    value="0.356221"/>   <!-- DERIVED -->
+  <xacro:property name="cyl_arm_d_off"     value="0.077770"/>   <!-- DERIVED -->
+  <xacro:property name="cyl_arm_len_min"   value="1.6139"/>     <!-- DERIVED -->
+  <!-- Barrel outer radius = bore/2 plus a wall; rod radius is the published rod/2. -->
+  <xacro:property name="cyl_wall"          value="0.010"/>      <!-- ASSUMPTION  m, cosmetic -->
+  <xacro:property name="cyl_barrel_frac"   value="0.62"/>       <!-- ASSUMPTION  barrel length as a fraction of len_min -->
+  <!-- Token mass. The REAL cylinder mass is already inside the published link masses:
+       Volvo's 530 kg boom figure is stated to include the dipper arm cylinder, piping
+       and pin. Giving these links their true ~80/60 kg would double-count it. They
+       therefore carry a token mass and MUST NOT be used for dynamics; switch
+       model_cylinders:=false for any run where that matters. Total machine mass moves
+       9 149.1 -> 9 151.1 kg (+0.02 %). -->
+  <xacro:property name="m_cyl_token"       value="0.5"/>        <!-- GUESS, TOKEN -->
   <xacro:property name="eff_swing"    value="22900.0"/>   <!-- PUBLISHED [L56]  Volvo max swing torque 22.9 kN.m. ECR88D ONLY: the ECR88 Plus publishes no swing torque at all, so do not carry this across. -->
   <xacro:property name="eff_boom"     value="${cyl_relief_pa * pi / 4 * cyl_boom_bore * cyl_boom_bore * 0.4763}"/>
