Commit message: 실린더가 날뛰는 원인 규명: 발산이 아니라 초기 상태 불일치
증상은 "cyl_arm_barrel 이 막 움직인다" 였고, 당연한 해석인 "솔버가 발산한다"는
틀렸다. 관절별 추적을 붙여보니 전부 수렴한다. 말미 80 스텝 p-p 가
0.0000~0.0052 rad 이다.

실제 원인: 실린더(=mimic 관절)가 있으면 articulation 이 authored rest pose 에서
시작하지 않는다.
  실린더 포함: bucket 103.8 deg (요청 20), boom -14.96 deg (요청 -30),
               그 지점에서 mimic 관계도 깨져 있다 (요구 -26.6, 실제 -54.8)
  실린더 제외: boom -30.05, arm 112.1, bucket 14.5  -> rest pose 그대로
Play 를 누르면 그 어긋난 자세에서 제자리로 크게 휘두른다. 그게 "막 움직이는"
것으로 보인 것.

조치:
- assets/ecr88/usd/ecr88_physics.usd 를 따로 낸다 (model_cylinders:=false).
  물리를 돌릴 때는 이걸 쓴다. ecr88.usd 는 보기용으로 실린더를 유지한다.
  실린더는 어차피 장식이고, 물리를 끈 상태에서는 authored rest pose 가
  mimic 과 일관되므로 정지 화면은 정확하다.
- scripts/check_stability.py: 이번에 쓴 추적 도구를 남긴다. 전체 p-p 와
  말미 p-p 를 따로 낸다. 전체만 보면 정착 과도가 발산처럼 보인다.

같이 고친 것:
- mimic 슬레이브 관절에서 position drive 제거(neutralise_mimic_drives).
  importer 가 모든 가동 관절에 DriveAPI 를 붙여서, mimic 제약과 드라이브가
  같은 축을 동시에 끌고 있었다. cyl_arm_extend 는 선형 강성 1e7 N/m 에
  링크 0.5 kg 이라 고유진동수가 712 Hz 였다. 60 Hz 스텝에서 성립 불가.
- 실린더 질량을 0.5 kg 토큰에서 실제값으로(붐 80, 암 60 kg). 이걸 각각
  m_boom 과 m_house 에서 덜어내 9209.1 kg 합계를 그대로 유지한다.
  Volvo 가 530 kg 붐에 dipper arm cylinder 포함이라고 명시하므로 붐에서,
  붐 실린더는 잔차인 하우스에서 덜어냈다.
- 실린더를 visual-only 로(detail_visual 매크로 신설). 배럴이 붐을 따라
  달리므로 충돌체를 주면 설계상 겹치는 두 솔리드를 출하하는 셈이다.
  (검증 결과 이번 증상의 원인은 아니었지만 조치 자체는 맞다.)
- --drive-damping-ratio (기본 0.4). importer 기본값이 강성 174533 에 감쇠 50
  이다. 붐 유효관성 ~8000 kg.m^2 기준 임계감쇠가 ~75000 이라 세 자릿수
  부족하다. 다만 이번 증상은 이걸로 안 고쳐졌다 - 초기 상태 문제였으므로.

남은 기지 사항: 정착 자세가 지령보다 처진다. 강성만 있는 위치 드라이브의
정상상태 오차 torque/stiffness 이고 붐에서 29945/174533 = 0.17 rad ~ 10도로
관측치와 맞는다. 중력 보상이나 강성 상향이 답이지 감쇠는 아니다.

Co-Authored-By: Claude Opus 5 <noreply@anthropic.com>
Claude-Session: https://claude.ai/code/session_01YCTHKLKR3ccjDNMFVWse8H

File: assets/ecr88/urdf/ecr88.urdf.xacro (robot description, xacro)
@@ -300,4 +300,21 @@
     </xacro:unless>
   </xacro:macro>
+  <!-- Visual ONLY: no <collision>. For cosmetic dressing that necessarily overlaps the
+       structure it is bolted to. A hydraulic cylinder barrel runs right along the boom
+       it drives, so giving it a collider means shipping two solids that interpenetrate
+       by design; the solver then spends every step trying to push them apart and the
+       articulation comes apart. That is exactly what happened when the cylinders were
+       first added with the collision-bearing `detail` macro.
+       Like `detail`, it vanishes when real meshes are switched on. -->
+  <xacro:macro name="detail_visual"
+               params="material:='xpanner_yellow' xyz:='0 0 0' rpy:='0 0 0' *prim">
+    <xacro:unless value="$(arg use_meshes)">
+      <visual>
+        <origin xyz="${xyz}" rpy="${rpy}"/>
+        <geometry><xacro:insert_block name="prim"/></geometry>
+        <material name="${material}"/>
+      </visual>
+    </xacro:unless>
+  </xacro:macro>
   <!-- A structural member drawn as a capsule-ish cylinder running from the link origin
        to the offset (dx,dy,dz). Length and pitch are DERIVED from the offset, so the
@@ -695,13 +712,13 @@
   <xacro:macro name="hyd_cylinder"
                params="name parent driver anchor_xyz phi_mult phi_off d_mult d_off
-                       len_min bore rod d_lo d_hi">
+                       len_min bore rod d_lo d_hi m_barrel m_rod">
     <link name="${name}_barrel">
-      <xacro:inertial_cylinder mass="${m_cyl_token}" radius="${bore * half + cyl_wall}"
+      <xacro:inertial_cylinder mass="${m_barrel}" radius="${bore * half + cyl_wall}"
                                length="${len_min * cyl_barrel_frac}"
                                xyz="${len_min * cyl_barrel_frac * half} 0 0" rpy="0 ${half_pi} 0"/>
-      <xacro:detail material="xpanner_steel"
+      <xacro:detail_visual material="xpanner_steel"
                     xyz="${len_min * cyl_barrel_frac * half} 0 0" rpy="0 ${half_pi} 0">
         <cylinder radius="${bore * half + cyl_wall}" length="${len_min * cyl_barrel_frac}"/>
-      </xacro:detail>
+      </xacro:detail_visual>
     </link>
     <joint name="${name}_pitch" type="revolute">
@@ -719,10 +736,10 @@
     </joint>
     <link name="${name}_rod">
-      <xacro:inertial_cylinder mass="${m_cyl_token}" radius="${rod * half}" length="${len_min}"
+      <xacro:inertial_cylinder mass="${m_rod}" radius="${rod * half}" length="${len_min}"
                                xyz="${len_min * half} 0 0" rpy="0 ${half_pi} 0"/>
-      <xacro:detail material="xpanner_accent"
+      <xacro:detail_visual material="xpanner_accent"
                     xyz="${len_min * half} 0 0" rpy="0 ${half_pi} 0">
         <cylinder radius="${rod * half}" length="${len_min}"/>
-      </xacro:detail>
+      </xacro:detail_visual>
     </link>
     <joint name="${name}_extend" type="prismatic">
@@ -748,5 +765,6 @@
                         d_mult="${cyl_boom_d_mult}"     d_off="${cyl_boom_d_off}"
                         len_min="${cyl_boom_len_min}" bore="${cyl_boom_bore}" rod="${cyl_boom_rod}"
-                        d_lo="-0.05" d_hi="0.15"/>
+                        d_lo="-0.05" d_hi="0.15"
+                        m_barrel="${m_cyl_boom_barrel}" m_rod="${m_cyl_boom_rod}"/>
     <!-- ARM cylinder. Parent pin distCylLrgArm is emitted on the BOOM TIP per T8, so the
          anchor below carries the lenBm1 + lenBm2 offset. The arm-side pin is the scalar
@@ -758,5 +776,6 @@
                         d_mult="${cyl_arm_d_mult}"     d_off="${cyl_arm_d_off}"
                         len_min="${cyl_arm_len_min}" bore="${cyl_arm_bore}" rod="${cyl_arm_rod}"
-                        d_lo="0.0" d_hi="0.90"/>
+                        d_lo="0.0" d_hi="0.90"
+                        m_barrel="${m_cyl_arm_barrel}" m_rod="${m_cyl_arm_rod}"/>
   </xacro:if>
   <link name="ground_link">

File: assets/ecr88/urdf/ecr88_dynamics.xacro (robot description, xacro)
@@ -96,6 +96,6 @@
        ============================================================================ -->
   <xacro:property name="m_base"        value="2713.0"/>  <!-- CLASS-TYPICAL [L8]  undercarriage INCLUDING both tracks, blade, final drives = 0.31 x 8752 kg operating weight. 0.31 is the middle of the published 28-34 % class band, nudged low because this reduced tail swing design loads the house. See H2. -->
-  <xacro:property name="m_house"       value="4966.0"/>  <!-- DERIVED (RESIDUAL) [L9]  8752 minus base, boom, arm assy, bucket, operator. Every error in m_base lands here one for one: this is the largest single uncertainty in the model. Includes the 1 400 kg published counterweight. -->
-  <xacro:property name="m_boom"        value="530.0"/>   <!-- PUBLISHED [L2]  Volvo component table, 3.55 m mono boom, "includes cylinder, piping and pin, excludes boom cyl. pin". Taken whole because the URDF models no cylinder links. -->
+  <xacro:property name="m_house"       value="${4966.0 - m_cyl_boom_total}"/>  <!-- DERIVED (RESIDUAL) [L9]  8752 minus base, boom, arm assy, bucket, operator, then minus the boom cylinder now modelled as its own links (it was inside this residual). Every error in m_base lands here one for one: this is the largest single uncertainty in the model. Includes the 1 400 kg published counterweight. -->
+  <xacro:property name="m_boom"        value="${530.0 - m_cyl_arm_total}"/>   <!-- PUBLISHED [L2]  Volvo component table, 3.55 m mono boom, "includes cylinder, piping and pin, excludes boom cyl. pin". The dipper arm cylinder Volvo counts in that 530 kg is now its own pair of links, so it is carved out here rather than counted twice. -->
   <xacro:property name="m_arm"         value="301.0"/>   <!-- DERIVED from PUBLISHED [L10]  2.1 m dipper. Published 340 kg arm assembly ("includes cylinder, linkage and pin") minus the carved out 4 bar: 340 - 22 - 16 - 1 = 301. The bucket cylinder stays inside this figure. For the 1.7 m arm the published assembly is 280 kg and this becomes 241. Volvo publishes both rows; Teo highlighted 2.1 m as the fleet spec (2026-09-11). -->
   <xacro:property name="m_inp_link"    value="22.0"/>    <!-- CLASS-TYPICAL [L11]  power link, pair of 0.42 m plates approx 20 x 140 mm section plus bosses. -->
@@ -339,11 +339,23 @@
   <xacro:property name="cyl_wall"          value="0.010"/>      <!-- ASSUMPTION  m, cosmetic -->
   <xacro:property name="cyl_barrel_frac"   value="0.62"/>       <!-- ASSUMPTION  barrel length as a fraction of len_min -->
-  <!-- Token mass. The REAL cylinder mass is already inside the published link masses:
-       Volvo's 530 kg boom figure is stated to include the dipper arm cylinder, piping
-       and pin. Giving these links their true ~80/60 kg would double-count it. They
-       therefore carry a token mass and MUST NOT be used for dynamics; switch
-       model_cylinders:=false for any run where that matters. Total machine mass moves
-       9 149.1 -> 9 151.1 kg (+0.02 %). -->
-  <xacro:property name="m_cyl_token"       value="0.5"/>        <!-- GUESS, TOKEN -->
+  <!-- CYLINDER MASS. The first pass gave these links a 0.5 kg token, reasoning that
+       the real mass is already inside the published figures. That was right about the
+       accounting and badly wrong about the physics: a 0.5 kg body under the drive
+       stiffness the importer applies is numerically unstable, and the arm cylinder
+       visibly exploded in the viewer. Mass ratios matter even for cosmetic links.
+       So give them realistic masses and CARVE THEM OUT of the links that already
+       contain them, which keeps the 9 149.1 kg reconciliation exact:
+         arm cylinder  60 kg  <- out of m_boom. Volvo states the 530 kg boom figure
+                                 "includes dipper arm cylinder, piping and pin".
+         boom cylinder 80 kg  <- out of m_house, which is the residual and therefore
+                                 where anything not itemised currently sits.
+       Split barrel/rod roughly 70/30, the barrel carrying the tube and both end caps.
+       CLASS-TYPICAL: no cylinder weight is published for this machine. -->
+  <xacro:property name="m_cyl_boom_total"  value="80.0"/>       <!-- CLASS-TYPICAL  105 mm bore, ~1.33 m -->
+  <xacro:property name="m_cyl_arm_total"   value="60.0"/>       <!-- CLASS-TYPICAL   90 mm bore, ~1.61 m -->
+  <xacro:property name="m_cyl_boom_barrel" value="${m_cyl_boom_total * 0.70}"/>  <!-- DERIVED -->
+  <xacro:property name="m_cyl_boom_rod"    value="${m_cyl_boom_total * 0.30}"/>  <!-- DERIVED -->
+  <xacro:property name="m_cyl_arm_barrel"  value="${m_cyl_arm_total * 0.70}"/>   <!-- DERIVED -->
+  <xacro:property name="m_cyl_arm_rod"     value="${m_cyl_arm_total * 0.30}"/>   <!-- DERIVED -->
   <xacro:property name="eff_swing"    value="22900.0"/>   <!-- PUBLISHED [L56]  Volvo max swing torque 22.9 kN.m. ECR88D ONLY: the ECR88 Plus publishes no swing torque at all, so do not carry this across. -->
   <xacro:property name="eff_boom"     value="${cyl_relief_pa * pi / 4 * cyl_boom_bore * cyl_boom_bore * 0.4763}"/>

Commit message: 자세 처짐의 진짜 원인: 4절 mimic 이 자기 리밋과 모순
증상은 "장비가 지령 자세를 못 버티고 흘러내린다" 였고, 두 번 잘못 짚었다.
처음엔 드라이브 감쇠 부족(50 vs 임계 75000)이라 봤고, 고쳐도 안 변했다.
다음엔 가속도 모드 드라이브로 바꿨고, 역시 안 변했다.

분기별로 빌드해 각각 재보니 답이 나왔다. rest pose 기준 정착 오차:
  4절만 (실린더 없음)  : +0.33 / -0.05 / -0.04 deg   (붐/암/버킷)
  실린더만 (4절 없음)  : +2.64 / -90.89 / +4.86 deg
즉 문제가 둘로 갈린다.

[1] 4절: input_link_joint 이 bucket_joint 에 mimic 을 걸고 있는데 리밋이
[-170, -20] 인 자유 GUESS 였다. 버킷 범위가 [-126, +43] 이라, mimic 이
리밋이 금지하는 각을 대부분의 구간에서 요구한다. 하드 제약 둘이 서로
당기면 그 힘이 dressing 안에 머물지 않고 프론트 전체에 실린다.

mimic 은 두 관절이 multiplier/offset 을 거쳐 같은 자유도라는 선언이므로,
리밋도 같은 관계로 사상되어야 한다. lim_inp_link_* 를 lim_bucket_* 에서
유도하도록 바꿨다. 계수가 placeholder 항등식이라 지금은 버킷 범위와 같다.
실제 4절 계수를 맞추면 리밋도 같이 사상해야 한다 - 안 그러면 재발한다.

참고로 중력은 처음부터 원인이 아니었다. URDF 에서 직접 계산한 rest pose
정적 유지 토크는 붐 36.8 kN.m 이고 effort 가 121.3 kN.m 라 3.3배 여유다.
시뮬이 보고한 "필요 토크" 158~401 kN.m 는 강성 1e7 짜리 드라이브의 반력이지
중력 부하가 아니었다.

[2] 암 실린더: 이것만으로 암이 지령에서 90.9 deg 어긋난다. 붐 실린더는
2.6 deg, 4절은 0.05 deg 인데 암 실린더만 두 자릿수다. 원인 미규명.
model_arm_cylinder 로 분리하고 기본 OFF. 붐 실린더가 어차피 눈에 띄는
쪽이고, 형상 목적은 그걸로 달성된다.

최종 정착 오차:
  ecr88.usd        (붐실린더+4절) +2.45 / +2.82 / +3.59 deg, 5축 전부 수렴
  ecr88_physics.usd (실린더 없음) +0.32 / -0.05 / -0.04 deg, 3축 전부 수렴

같이 들어간 것:
- --keep-mimic-drives: mimic 관절의 드라이브를 남길지 선택. 기본은 제거지만,
  슬레이브 가지에 질량이 실리면 mimic 만으로는 중력을 못 버틴다. 어느 쪽이
  맞는지는 매달린 질량에 달렸고 이번엔 차이가 없었다.
- tune_drive_damping 이 드라이브 모드를 본다. 가속도 모드는 게인이 관성으로
  정규화되므로 임계감쇠가 2*sqrt(k) 이지 0.4*k 가 아니다. 힘 모드 규칙을
  그대로 쓰면 84배 과감쇠가 된다.

Co-Authored-By: Claude Opus 5 <noreply@anthropic.com>
Claude-Session: https://claude.ai/code/session_01YCTHKLKR3ccjDNMFVWse8H

File: assets/ecr88/urdf/ecr88.urdf.xacro (robot description, xacro)
@@ -201,4 +201,11 @@
        Set false for any physics run where four extra slaved bodies are unwanted. -->
   <xacro:arg name="model_cylinders"     default="true"/>
+  <!-- The ARM cylinder is switchable on its own because it, alone, destabilises the
+       articulation: with only the arm cylinder present the arm settles 90.9 deg away
+       from its commanded angle, while the boom cylinder costs 2.6 deg and the 4-bar
+       costs 0.05 deg. Isolated by building the three branches separately and measuring
+       each. Default OFF until that is understood; the boom cylinder is the visible one
+       anyway. -->
+  <xacro:arg name="model_arm_cylinder"  default="false"/>
   <xacro:arg name="mesh_package"        default="xpanner_sim"/>
   <xacro:arg name="mesh_dir"            default="assets/ecr88/meshes"/>
@@ -771,4 +778,5 @@
          lenToCylSmlArm assumed on the arm centreline - that assumption is why this one is
          only honest to 109 mm. See ecr88_dynamics.xacro. -->
+    <xacro:if value="$(arg model_arm_cylinder)">
     <xacro:hyd_cylinder name="cyl_arm" parent="boom_link" driver="arm_joint"
                         anchor_xyz="${lenBm1 + lenBm2 + distCylLrgArm_x} ${distCylLrgArm_y} ${distCylLrgArm_z}"
@@ -778,4 +786,5 @@
                         d_lo="0.0" d_hi="0.90"
                         m_barrel="${m_cyl_arm_barrel}" m_rod="${m_cyl_arm_rod}"/>
+    </xacro:if>
   </xacro:if>
   <link name="ground_link">

File: assets/ecr88/urdf/ecr88_dynamics.xacro (robot description, xacro)
@@ -231,6 +231,24 @@
   <!-- Passive 4 bar dressing branch. The URDF cut is at the conn rod / output link pin,
        so this branch is VISUAL ONLY and carries no load. Wide placeholders. -->
-  <xacro:property name="lim_inp_link_lower" value="${deg * -170.00}"/> <!-- GUESS  unconstrained placeholder, dressing branch. -->
-  <xacro:property name="lim_inp_link_upper" value="${deg *  -20.00}"/> <!-- GUESS  unconstrained placeholder, dressing branch. -->
+  <!-- input_link_joint CARRIES A MIMIC ON bucket_joint. A mimic says the two joints
+       are the same degree of freedom up to multiplier and offset, so their LIMITS must
+       be the same interval mapped through that same relation. These used to be a
+       free-hand GUESS of [-170, -20] against a bucket range of [-126, +43], i.e. the
+       mimic demanded angles the limit forbade over most of the bucket's travel.
+       That is not a cosmetic mismatch. Two hard constraints pulling against each other
+       inject large forces into the chain, and those forces do not stay in the dressing
+       branch: they loaded the whole front end. Measured at the rest pose, with the
+       4-bar present the machine settled 11.8 / 14.0 / 36.2 deg away from its commanded
+       boom / arm / bucket angles; with the 4-bar dropped, the same pose held to
+       0.33 / 0.07 / 0.02 deg. That drift was read as "the drives are too weak" and then
+       as "the cylinders are exploding", and it was neither. Analytic gravity torque
+       at this pose is 36.8 kN.m on a boom with 121.3 kN.m of effort, a 3.3x margin.
+       With the placeholder multiplier 1.0 / offset 0.0 the mapping is the identity, so
+       the limits are simply the bucket's. WHEN THE REAL 4-BAR COEFFICIENTS ARE FITTED,
+       THESE MUST BE MAPPED THROUGH THEM TOO, or the same fight comes back. -->
+  <xacro:property name="lim_inp_link_lower" value="${bkt_mimic_mult * lim_bucket_lower + bkt_mimic_off}"/>
+                                         <!-- DERIVED from lim_bucket_* through the mimic -->
+  <xacro:property name="lim_inp_link_upper" value="${bkt_mimic_mult * lim_bucket_upper + bkt_mimic_off}"/>
+                                         <!-- DERIVED from lim_bucket_* through the mimic -->
   <xacro:property name="lim_conn_rod_lower" value="${-pi}"/>           <!-- GUESS  the cut member: free by construction. -->
   <xacro:property name="lim_conn_rod_upper" value="${ pi}"/>           <!-- GUESS  the cut member: free by construction. -->
