Commit message: 포크/패널적재/흡착컵 + 카메라 위치 정량 검토
작업 방식을 잘못 알고 있었다. 패널은 땅바닥 파레트가 아니라 장비 자신의
앞쪽 포크에 여러 장 실려 다니고, 어태치먼트의 흡착컵 4개로 거기서 한 장씩
집어 행에 놓는다. 시트의 dist*Fork* / LenPL* / LenSD* 블록이 전부 이 얘기였고,
"처리구분 Delete" 는 태블릿 데이터셋에 안 넣는다는 뜻이지 장비에 없다는
뜻이 아니었다.

- 앞쪽 포크 캐리지 + 패널 적재(12장) 추가. 파레트 기울기 AlphaPL2(15.7도),
  받침대 기울기 AlphaPL1(74.5도) 는 시트의 각도기 실측 그대로.
  X 만 시트값을 못 쓴다: LenPLX=1.086 을 캐리지 기준으로 잡으면 하우스가
  x=1.14 까지라 1.25m 마스트가 하우스를 관통한다. 실제로 cam_fork_mast 가
  사이클 전 구간에서 house_link 에 가리는 것으로 드러났다. 하부 앞으로 빼고
  주석에 남겼다. Y, Z 는 시트값.
- 흡착컵 4개. 판을 누르는 게 아니라 컵 4개로 한 장을 집는 게 실제 엔드이펙터고,
  카메라가 봐야 하는 건 그 컵이 유리에 닿는 순간이다.
- 2.1m 열이 포크 행에 0 을 적은 건 미측정이지 부재가 아니므로, variant 와
  무관하게 기장 열 실측값으로 세웠다.

카메라 후보 7곳을 프레임으로 넣고 scripts/camera_study.py 로 사이클 54 포즈에서
FOV + 자기 구조물 가림을 계산했다. 회의에서 말로 정하지 말고 수치로 정하자는 것.

첫 실행이 거의 전부 0% 가 나왔다. 카메라가 자기 마운트 링크의 볼록 박스
안에 박혀서 모든 시선이 자기 몸통에 막힌 것. 마운트 링크를 가림에서 제외.

--ignore-tool-adapter 를 뒀다. 틸트로테이터 어댑터 체인을 통짜 실린더로
그려놔서 컵으로 가는 모든 시선을 막는데, 실물은 얇은 프레임이라 저렇게
안 막는다. 양쪽 다 돌려서 결론이 미모델링 형상에 얼마나 의존하는지 드러낸다.

결과(어댑터 제외 기준):
  픽(적재 상단)  cam_fork_mast  98% @1.2m   - 유일하게 보이는 후보
  TCP(컵)        cam_tool_side  98% @1.1m / cam_arm_tip 98% @2.0m
  플레이스(행)   cam_cab_roof   48% / cam_house_front 43%  - 가장 약한 구간
cam_tool 은 흡착축을 따라 내려다보므로 자기 컵을 못 본다(TCP 0%). 축 위가
아니라 옆에서 봐야 한다는 게 cam_tool_side 를 만든 이유다.

같이 들어간 것:
- scripts/animate_cycle.py: 픽앤플레이스 사이클을 드라이브 타깃 타임샘플로
  씬에 굽는다. 스트리밍 세션이 이미 GPU 를 쥐고 있어 두 번째 Isaac 프로세스를
  띄울 수 없으므로, 제어 스크립트가 아니라 애니메이션으로 넣었다.
  키프레임이 리밋을 벗어나면 authoring 을 거부한다.

Co-Authored-By: Claude Opus 5 <noreply@anthropic.com>
Claude-Session: https://claude.ai/code/session_01YCTHKLKR3ccjDNMFVWse8H

File: assets/ecr88/urdf/ecr88.urdf.xacro (robot description, xacro)
@@ -208,4 +208,9 @@
        anyway. -->
   <xacro:arg name="model_arm_cylinder"  default="false"/>
+  <!-- Front fork carriage and the stack of modules riding on it. This is how the
+       machine actually feeds itself, so it is on by default. -->
+  <xacro:arg name="model_fork"          default="true"/>
+  <!-- Candidate camera/lidar mount frames. Zero mass, no geometry beyond a marker. -->
+  <xacro:arg name="model_sensor_mounts" default="true"/>
   <xacro:arg name="mesh_package"        default="xpanner_sim"/>
   <xacro:arg name="mesh_dir"            default="assets/ecr88/meshes"/>
@@ -339,4 +344,5 @@
   <material name="xpanner_accent"><color rgba="0.85 0.25 0.10 1"/></material>
   <material name="xpanner_frame"> <color rgba="0.10 0.60 0.90 1"/></material>
+  <material name="xpanner_panel"> <color rgba="0.09 0.13 0.28 1"/></material>
   <!-- =====================================================================
        1. UNDERCARRIAGE
@@ -1005,4 +1011,25 @@
       <box size="${geo_pad_x} ${geo_pad_y} ${geo_pad_t}"/>
     </xacro:viscol>
+    <!-- FOUR SUCTION CUPS. The tool does not press a plate against the module, it
+         grips one module with four cups; that is the actual end effector and it is
+         what a camera has to see land on the glass. Laid out on the corners of the
+         pad, inset by one cup radius so they sit on the module rather than over its
+         edge. Cup size is CLASS-TYPICAL: the sheet records LenSDX = LenSDY = 0 for
+         this machine, which is "not measured", so the pad itself is already the
+         LenPLWidth x LenPanelHeight stand-in (T9). -->
+    <xacro:property name="cup_dx" value="${geo_pad_x * half - geo_suction_cup_r}"/>
+    <xacro:property name="cup_dy" value="${geo_pad_y * half - geo_suction_cup_r}"/>
+    <xacro:detail_visual material="xpanner_dark" xyz="${ cup_dx} ${ cup_dy} ${-geo_suction_cup_h * half}">
+      <cylinder radius="${geo_suction_cup_r}" length="${geo_suction_cup_h}"/>
+    </xacro:detail_visual>
+    <xacro:detail_visual material="xpanner_dark" xyz="${ cup_dx} ${-cup_dy} ${-geo_suction_cup_h * half}">
+      <cylinder radius="${geo_suction_cup_r}" length="${geo_suction_cup_h}"/>
+    </xacro:detail_visual>
+    <xacro:detail_visual material="xpanner_dark" xyz="${-cup_dx} ${ cup_dy} ${-geo_suction_cup_h * half}">
+      <cylinder radius="${geo_suction_cup_r}" length="${geo_suction_cup_h}"/>
+    </xacro:detail_visual>
+    <xacro:detail_visual material="xpanner_dark" xyz="${-cup_dx} ${-cup_dy} ${-geo_suction_cup_h * half}">
+      <cylinder radius="${geo_suction_cup_r}" length="${geo_suction_cup_h}"/>
+    </xacro:detail_visual>
   </link>
   <joint name="contact_surface_joint" type="fixed">
@@ -1012,4 +1039,129 @@
             rpy="0 ${angProbeToContactSurface} 0"/>
   </joint>
+  <!-- =====================================================================
+       9b. FRONT FORK AND THE PANEL STACK IT CARRIES
+       The machine does not pick modules off the ground. It carries a STACK of
+       them on a forklift-style carriage on the front of the undercarriage, drives
+       along the row, and lifts ONE module off its own fork with the four suction
+       cups on the tool. That is what every dist*Fork* and LenPL* row in the
+       parameter sheet is describing, and it is why the sheet has a "포크리프트"
+       block at all.
+       WHICH COLUMN THESE COME FROM. The 2.1 m US#1 column records 0 for
+       distUcToForkBack and distForkBackToPanelTop. Zero there means NOT MEASURED,
+       not "no fork". The machine plainly has one. So the fork is built from the
+       "ECR88 기장" column, which carries real numbers, even when the selected
+       variant is the 2.1 m one. Flagged rather than hidden: if the 2.1 m machine's
+       fork really does sit somewhere else, this is the block to fix.
+       The sheet also marks several of these rows Delete. That marking governs what
+       goes into the TABLET's kinematic dataset, not what the machine physically
+       has; the fork is drawn here as geometry and drives nothing.
+       Pallet base tilts by AlphaPL2 (15.7 deg) and the backrest by AlphaPL1
+       (74.5 deg), both straight from the sheet's protractor readings, so the stack
+       leans back the way it does on the real carriage.
+       ===================================================================== -->
+  <xacro:if value="$(arg model_fork)">
+    <link name="fork_link">
+      <xacro:inertial_box mass="${m_fork}"
+                          x="${geo_fork_len}" y="${LenPLWidth}" z="${geo_fork_t}"
+                          xyz="${geo_fork_len * half} 0 0"/>
+      <!-- pallet base, tilted back by AlphaPL2 -->
+      <xacro:viscol name="fork_link" material="xpanner_dark"
+                    xyz="${geo_fork_len * half} 0 0" rpy="0 ${-AlphaPL2} 0">
+        <box size="${geo_fork_len} ${LenPLWidth} ${geo_fork_t}"/>
+      </xacro:viscol>
+      <!-- backrest the stack leans on, tilted by AlphaPL1 -->
+      <xacro:detail material="xpanner_dark"
+                    xyz="0 0 ${geo_fork_back_h * half}" rpy="0 ${half_pi - AlphaPL1} 0">
+        <box size="${geo_fork_back_h} ${LenPLWidth} ${geo_fork_t}"/>
+      </xacro:detail>
+    </link>
+    <joint name="fork_joint" type="fixed">
+      <parent link="base_link"/>
+      <child  link="fork_link"/>
+      <!-- X IS NOT LenPLX. Taken literally, LenPLX = 1.086 puts the carriage inside
+           the machine: the house box reaches x = +1.14 and the undercarriage +1.41,
+           so a 1.25 m mast at x = 1.086 rises straight through the house. It showed up
+           as cam_fork_mast being occluded by house_link on every pose of the cycle.
+           LenPLX is evidently measured to some other fork reference, not to the
+           carriage root. Until that is pinned down, the carriage is placed clear of
+           the undercarriage front, which is where a forklift carriage physically is.
+           Y and Z ARE the sheet's (LenPLY, LenPLZ); only X is overridden. -->
+      <origin xyz="${lenBottomX * half + geo_fork_clear} ${LenPLY} ${LenPLZ}" rpy="0 0 0"/>
+    </joint>
+    <!-- The stack itself. Modules lie flat on the tilted pallet, one on top of the
+         next; the tool takes them off the top. Count is a scene choice, not data. -->
+    <link name="panel_stack_link">
+      <xacro:inertial_box mass="${m_panel * n_panels}"
+                          x="${LenPanelHeight}" y="${LenPLWidth}" z="${n_panels * geo_panel_t}"
+                          xyz="0 0 ${n_panels * geo_panel_t * half}"/>
+      <xacro:viscol name="panel_stack_link" material="xpanner_panel"
+                    xyz="0 0 ${n_panels * geo_panel_t * half}">
+        <box size="${LenPanelHeight} ${LenPLWidth} ${n_panels * geo_panel_t}"/>
+      </xacro:viscol>
+    </link>
+    <joint name="panel_stack_joint" type="fixed">
+      <parent link="fork_link"/>
+      <child  link="panel_stack_link"/>
+      <origin xyz="${geo_fork_len * half} 0 ${geo_fork_t * half}" rpy="0 ${-AlphaPL2} 0"/>
+    </joint>
+  </xacro:if>
+  <!-- =====================================================================
+       9c. CANDIDATE SENSOR MOUNTS
+       Zero-mass frames, nothing else. They exist so the camera argument can be had
+       in numbers instead of adjectives: scripts/camera_study.py walks the work cycle
+       and reports, for each of these, whether the pick point on the fork, the suction
+       cups, and the placement point on the row are inside the field of view and not
+       hidden behind the machine's own structure.
+       Add or move one and re-run the study; do not argue about it in a meeting.
+       Each frame's +X is the optical axis, +Z up, matching the usual camera
+       convention for a sensor prim in Isaac.
+       ===================================================================== -->
+  <xacro:if value="$(arg model_sensor_mounts)">
+    <xacro:macro name="cam_mount" params="name parent xyz rpy">
+      <link name="${name}">
+        <xacro:inertial_sphere mass="${m_marker}" radius="${geo_marker_r}"/>
+        <xacro:detail_visual material="xpanner_frame">
+          <sphere radius="${geo_marker_r}"/>
+        </xacro:detail_visual>
+      </link>
+      <joint name="${name}_joint" type="fixed">
+        <parent link="${parent}"/>
+        <child  link="${name}"/>
+        <origin xyz="${xyz}" rpy="${rpy}"/>
+      </joint>
+    </xacro:macro>
+    <!-- Cab roof, front edge, looking forward and down. The operator's own viewpoint. -->
+    <xacro:cam_mount name="cam_cab_roof" parent="house_link"
+                     xyz="${lenUppX * half - 0.10} ${lenUppY * half - 0.50} ${lenUppZ1 + geo_house_h - 0.05}"
+                     rpy="0 ${pi/180*25} 0"/>
+    <!-- House front deck, beside the boom foot, on the boom's own side (-Y). -->
+    <xacro:cam_mount name="cam_house_front" parent="house_link"
+                     xyz="${lenUppX * half - 0.15} ${-0.55} ${lenUppZ1 + geo_deck_h + 0.10}"
+                     rpy="0 ${pi/180*20} 0"/>
+    <!-- Mid boom, outboard side, aimed along the boom at the tool. -->
+    <xacro:cam_mount name="cam_boom_mid" parent="boom_link"
+                     xyz="${(lenBm1 + lenBm2) * geo_boom_apex_frac} ${-(geo_boom_sec_w * half + 0.08)} ${geo_boom_rise * 0.6}"
+                     rpy="0 ${pi/180*35} 0"/>
+    <!-- Arm, just behind the bucket pin, looking at the tool. The closest a fixed
+         mount gets to the work without riding the tool itself. -->
+    <xacro:cam_mount name="cam_arm_tip" parent="arm_link"
+                     xyz="${lenArm - 0.35} ${-(geo_arm_sec_w * half + 0.06)} ${geo_arm_sec_h * half + 0.05}"
+                     rpy="0 ${pi/180*55} 0"/>
+    <!-- On the tool, above the cups, looking straight down the suction axis. -->
+    <xacro:cam_mount name="cam_tool" parent="attachment_link"
+                     xyz="0.0 0.0 -0.10" rpy="0 ${half_pi} 0"/>
+    <!-- On the rotator, offset sideways and angled in, so it sees the cups and the
+         module edge rather than looking straight down the suction axis. cam_tool
+         scored 0 % on the TCP for exactly that reason: a camera on the tool axis
+         cannot see its own contact patch. This is the variant that can. -->
+    <xacro:cam_mount name="cam_tool_side" parent="rotator_link"
+                     xyz="0.0 ${-(geo_tr_r + 0.22)} -0.15"
+                     rpy="${-pi/180*55} ${pi/180*60} 0"/>
+    <!-- On the fork backrest, looking back at the top of the stack. Sees the pick
+         point without depending on where the boom happens to be. -->
+    <xacro:cam_mount name="cam_fork_mast" parent="fork_link"
+                     xyz="0.0 ${LenPLWidth * half - 0.10} ${geo_fork_back_h}"
+                     rpy="0 ${pi/180*45} 0"/>
+  </xacro:if>
   <!-- =====================================================================
        10. ros2_control

File: assets/ecr88/urdf/ecr88_params.xacro (robot description, xacro)
@@ -959,4 +959,24 @@
   <xacro:property name="geo_marker_r"          value="0.03"/>    <!-- ESTIMATE (T11) m, cosmetic -->
   <!-- ..................................................................
+       [15][D3] FORK CARRIAGE, PANEL STACK, SUCTION CUPS.
+       Shape for the part of the machine that actually feeds it: modules ride on a
+       forklift carriage at the front and the tool lifts them off one at a time.
+       Positions come from the sheet (LenPLX/Y/Z, AlphaPL1/2, LenPLWidth,
+       LenPanelHeight); the sizes below are the bits the sheet does not carry.
+       .................................................................. -->
+  <xacro:property name="geo_fork_clear"        value="0.15"/>   <!-- ASSUMPTION  m, carriage root ahead of the track front -->
+  <xacro:property name="geo_fork_len"          value="1.45"/>    <!-- ASSUMPTION  m, tine length -->
+  <xacro:property name="geo_fork_t"            value="0.07"/>    <!-- ASSUMPTION  m, pallet/backrest plate -->
+  <xacro:property name="geo_fork_back_h"       value="1.25"/>    <!-- ASSUMPTION  m, backrest height -->
+  <xacro:property name="geo_panel_t"           value="0.040"/>   <!-- ASSUMPTION  m, one module incl. frame -->
+  <xacro:property name="n_panels"              value="12"/>      <!-- scene choice, not data -->
+  <xacro:property name="m_panel"               value="23.0"/>    <!-- CLASS-TYPICAL  kg, 72-cell glass-glass -->
+  <xacro:property name="m_fork"                value="280.0"/>   <!-- CLASS-TYPICAL  kg, carriage + backrest -->
+  <!-- Suction cup. The sheet records LenSDX = LenSDY = 0 for ECR88, i.e. the pad was
+       never measured, so the cups are sized to what lifts a module: four 200 mm cups
+       is the usual arrangement for a ~25 kg glass panel. CLASS-TYPICAL. -->
+  <xacro:property name="geo_suction_cup_r"     value="0.10"/>    <!-- CLASS-TYPICAL  m -->
+  <xacro:property name="geo_suction_cup_h"     value="0.06"/>    <!-- CLASS-TYPICAL  m -->
+  <!-- ..................................................................
        [15][D2] SHAPE, not size.  Added 2026-09-11 after the first Isaac Sim
        view: the kinematics were right but the machine did not read as an
