Commit message: Dozer blade becomes a real joint; five CAN1 IMU frames added
DOZER BLADE. This was drawn as fixed geometry with the reasoning written into
the file: "there is no blade joint in the parameter sheet, and inventing one
would put a moving part in the tree that nothing can command." The premise was
checkable and it was wrong. MACH_POST_01P publishes JntAngDozerBlade,
SYS_PARAM_01P lists autoCtrlEnaDozer among seven auto-control axes, and
ECR88D_LongArm.m carries bladeUp/bladeDown valve tables. It is now a revolute
joint on base_link, +Y positive-up to match the boom convention, and m_blade
(250 kg) comes out of m_base the way the tracks did so the machine does not
silently gain a quarter tonne.

Its range has no source, but it has a provable floor. The calibration
procedure will not start unless the blade holds "Dozer full down, Pitch > 5
deg" -- the blade alone jacking the front of an 8.75 t machine up by 5 degrees.
With the 2.82 m track and a 1.10 m blade arm that needs 0.229 m of drop below
the tracks, so 12.0 deg down at minimum: any narrower range would fail a gate
the real machine passes. Adopted roughly double (25 down / 30 up = 0.465 /
0.550 m), which also lands on the class norm. Replace from the working-range
drawing Teo has.

The blade is also the one axis whose reqSpdToActCmd table is a passthrough
(X = Y = [0, 0.001, 80]), i.e. not speed calibrated but commanded open loop,
which is why vel_dozer stays a GUESS while every other axis now carries a
measured speed.

IMU FRAMES. CAN1 runs six IMUs at 20 ms and ECR88D_LongArm.m gives each a 3x3
mounting matrix. Five are populated; the sixth is the identity because
lenBm2 = 0, so no frame is emitted for it -- the slot exists on the bus, the
sensor does not exist on the machine.

These implement one IMU per member, with every reported joint angle a
DIFFERENCE of two of them (chs/boom/arm/output/tilt -> body roll+pitch,
BodyToBoom, Boom2ToArm, ArmToBucket, Tilt). That is why the machine has no
encoders, and why the frames have to be right: a wrong mounting rotation does
not shift one reading, it corrupts the angle the controller closes on.

Rotations are OEM-FIRMWARE, positions are a GUESS -- the firmware gives a
matrix and no translation. For attitude that split is the right way round; the
rotation sets what the gyro and accelerometer read, and position only enters
through the lever-arm term. Converted to URDF fixed-axis XYZ and round-tripped
back to the matrix to 7e-7, which matters for imuTilt: its pitch is 88 deg,
so the three rpy numbers are individually ill-conditioned even though the
matrix they rebuild is exact.

We read the matrix as IMU -> link rather than its transpose because the three
arm-chain boards then decompose as Rz(yaw) * Rx(90 deg) with residuals under
0.5 deg -- the same board on a vertical side plate, the yaw being that plate's
angle to the member (32.4 deg on the curved gooseneck boom, -6.0 and -3.4 on
the arm and link). Under the transpose the calibrated angle would be a
rotation about the sensor rather than about the member, which is not a thing a
bracket has. Noted in the file as the first assumption to overturn if the
sim's CAN1 output ever disagrees with a log by a transpose.

FK confirms the frames land on the firmware's matrices, including imu_chs
reading 0.560 deg off world +Z at zero pose: that is the real mounting error
reproduced, and it is correct that it is not zero, because the sim publishes
raw sensor values and the firmware's own matrix is what removes it.

39 frames, 18 pass, 0 fail. The five new warnings are the marker-link
"mass but no collision" note the seven camera mounts already carry.

Co-Authored-By: Claude Opus 5 <noreply@anthropic.com>
Claude-Session: https://claude.ai/code/session_01YCTHKLKR3ccjDNMFVWse8H

File: assets/ecr88/urdf/ecr88.urdf.xacro (robot description, xacro)
@@ -213,4 +213,7 @@
   <!-- Candidate camera/lidar mount frames. Zero mass, no geometry beyond a marker. -->
   <xacro:arg name="model_sensor_mounts" default="true"/>
+  <!-- The five CAN1 IMU frames. On by default: they carry calibrated data, they are
+       massless markers, and the SIL loop needs them. -->
+  <xacro:arg name="model_imus"          default="true"/>
   <xacro:arg name="mesh_package"        default="xpanner_sim"/>
   <xacro:arg name="mesh_dir"            default="assets/ecr88/meshes"/>
@@ -372,14 +375,47 @@
       <box size="${lenBottomX} ${lenBottomY - geo_track_w - geo_track_w} ${lenUppZ1 - lenBottomZ1}"/>
     </xacro:viscol>
-    <!-- SHAPE: dozer blade. The machine has one and the calibration procedure gates on
-         it ("Dozer full down, Pitch angle > 5"), so it is not decoration for the SIL
-         work either. Drawn on base_link and NOT articulated: there is no blade joint
-         in the parameter sheet, and inventing one would put a moving part in the tree
-         that nothing can command. Cosmetic mass is ignored - it sits inside m_base. -->
-    <xacro:detail material="xpanner_dark"
-                  xyz="${lenBottomX * half + geo_blade_t * half} 0 ${lenBottomZ1 + geo_blade_h * half}">
+  </link>
+  <!-- ======================================================================
+       DOZER BLADE - a real joint, corrected 2026-09-11.
+       This was drawn as fixed geometry on base_link, with the reasoning written
+       into the file: "there is no blade joint in the parameter sheet, and inventing
+       one would put a moving part in the tree that nothing can command." The premise
+       was checkable and it was wrong. The firmware commands it:
+         MACH_POST_01P  publishes  JntAngDozerBlade     (12 bit, 0.1 deg)
+         SYS_PARAM_01P  carries    autoCtrlEnaDozer     (one of 7 auto-control axes)
+         ECR88D_LongArm.m          bladeUp / bladeDown valve tables
+       and the calibration procedure gates on the blade holding the machine at
+       Pitch > 5 deg. Something can command it, and the SIL loop has to be able to.
+       The blade tables are the one pair in reqSpdToActCmd that are NOT speed
+       calibrated: X and Y are both [0, 0.001, 80], i.e. a passthrough. The blade is
+       commanded open loop, which is why vel_dozer stays a GUESS while every other
+       axis now carries the firmware's measured speed.
+       Mass comes OUT of m_base (m_blade), exactly as the tracks did, or the machine
+       silently gains 250 kg - the same mistake as H2.
+       ====================================================================== -->
+  <link name="dozer_link">
+    <xacro:inertial_box mass="${m_blade}"
+                        x="${geo_blade_t}" y="${lenBottomY}" z="${geo_blade_h}"
+                        xyz="${geo_blade_arm} 0 0"/>
+    <!-- Push arms, drawn from the pivot out to the blade so the joint is visible. -->
+    <xacro:viscol name="dozer_link" material="xpanner_dark"
+                  xyz="${geo_blade_arm * half} 0 0">
+      <box size="${geo_blade_arm} ${lenBottomY - geo_track_w} 0.10"/>
+    </xacro:viscol>
+    <xacro:detail material="xpanner_dark" xyz="${geo_blade_arm} 0 0">
       <box size="${geo_blade_t} ${lenBottomY} ${geo_blade_h}"/>
     </xacro:detail>
   </link>
+  <joint name="dozer_joint" type="revolute">
+    <parent link="base_link"/>
+    <child  link="dozer_link"/>
+    <origin xyz="${blade_pivot_x} 0 ${blade_pivot_z}" rpy="0 0 0"/>
+    <!-- +Y, so a POSITIVE angle lifts the blade. Matches the boom convention
+         (blade up and boom up are both positive about +Y). -->
+    <axis xyz="0 1 0"/>
+    <limit lower="${jntDozerLower}" upper="${jntDozerUpper}"
+           effort="${eff_dozer}" velocity="${vel_dozer}"/>
+    <dynamics damping="${dyn_damping}" friction="${dyn_friction}"/>
+  </joint>
   <!-- Tracks. FIXED for now (T12): travel is not simulated yet. To drive the machine,
        change these to `continuous` with <axis xyz="0 1 0"/> and add wheel/track links,
@@ -1189,4 +1225,85 @@
        is a cut joint with no actuator behind it.
        ===================================================================== -->
+  <!-- =====================================================================
+       IMU MOUNTS - the machine's own calibrated mounting rotations.
+       CAN1 carries six IMUs into Mango at 20 ms, each publishing QUAT + ACC + GYRO.
+       Five are populated on this machine; the sixth (Boom2) is an identity matrix
+       because lenBm2 = 0, i.e. there is no Boom2 to put one on.
+       The attitude scheme these implement: ONE IMU PER MEMBER, and every joint angle
+       the firmware reports is a DIFFERENCE of two of them.
+         imuChs   -> house      JntAngBodyRoll, JntAngBodyPitch  (absolute)
+         imuBm1   -> boom       JntAngBodyToBoom   = boom  - chassis
+         imuArm   -> arm        JntAngBoom2ToArm   = arm   - boom
+         imuLink  -> output     JntAngArmToBucket  = output- arm
+         imuTilt  -> tilt       JntAngTilt
+       That is why there is no encoder anywhere in this machine, and it is why these
+       frames have to be right: a wrong mounting rotation does not shift one reading,
+       it corrupts the joint angle the controller closes its loop on.
+       ROTATIONS ARE OEM-FIRMWARE, POSITIONS ARE A GUESS.
+       ECR88D_LongArm.m gives each IMU a 3x3 direction cosine matrix (a11..a33) and
+       NO translation. So the orientations below are the machine's own calibration,
+       converted to URDF fixed-axis XYZ and round-tripped back to the matrix to 7e-7;
+       the xyz are plausible spots on each member and nothing more. For attitude that
+       split is the right way round - the rotation is what sets what the gyro and the
+       accelerometer read. Position only enters through the lever-arm term under
+       angular acceleration, which is small here and zero in steady motion.
+       All six matrices are proper rotations (det = +1, orthonormal to 1e-7), and the
+       three arm-chain boards decompose cleanly as Rz(yaw) * Rx(90 deg) with residuals
+       under 0.5 deg: the same board on a vertical side plate, the yaw being that
+       plate's angle to the member. imuBm1's yaw is 32.4 deg, which is the facet angle
+       you would expect on a curved gooseneck boom; imuArm and imuLink are -6.0 and
+       -3.4 deg, i.e. plates nearly parallel to their members. imuChs is flat and
+       yawed 101 deg (a box in the cabinet); imuTilt is a full axis permutation.
+       That consistency is the reason we read the matrix as IMU -> link rather than
+       its transpose: under the transpose the calibrated angle would be a rotation
+       about the sensor rather than about the member, which is not a thing a bracket
+       has. IF THE SIM'S CAN1 OUTPUT EVER DISAGREES WITH A RECORDED LOG BY A
+       TRANSPOSE, THIS IS THE ASSUMPTION TO OVERTURN FIRST.
+       Each frame's axes are the SENSOR's axes, so a reading taken in this frame is
+       directly comparable to the real CAN1 payload.
+       ===================================================================== -->
+  <xacro:if value="$(arg model_imus)">
+    <xacro:macro name="imu_mount" params="name parent xyz rpy">
+      <link name="${name}">
+        <xacro:inertial_sphere mass="${m_marker}" radius="${geo_marker_r}"/>
+        <xacro:detail_visual material="xpanner_accent">
+          <box size="${geo_marker_r*2} ${geo_marker_r*2} ${geo_marker_r}"/>
+        </xacro:detail_visual>
+      </link>
+      <joint name="${name}_joint" type="fixed">
+        <parent link="${parent}"/>
+        <child  link="${name}"/>
+        <origin xyz="${xyz}" rpy="${rpy}"/>
+      </joint>
+    </xacro:macro>
+    <!-- imuChs. Flat, yawed 101.012 deg. Position: in the house, low and central. -->
+    <xacro:imu_mount name="imu_chs" parent="house_link"
+                     xyz="0.20 0.30 ${lenUppZ1 + 0.25}"
+                     rpy="0.007485990 -0.006288474 1.762991172"/>
+    <!-- imuBm1. Side plate at 32.447 deg. Position: outboard face near the boom foot. -->
+    <xacro:imu_mount name="imu_boom" parent="boom_link"
+                     xyz="0.70 ${-geo_boom_sec_w * half - 0.02} 0.20"
+                     rpy="1.571657101 -0.001138020 0.566315716"/>
+    <!-- imuArm. Side plate at -6.043 deg. -->
+    <xacro:imu_mount name="imu_arm" parent="arm_link"
+                     xyz="0.45 ${-geo_arm_sec_w * half - 0.02} 0.12"
+                     rpy="1.579022612 -0.002439665 -0.105463699"/>
+    <!-- imuLink. Side plate at -3.372 deg. The firmware calls the 4-bar OUTPUT member
+         "Link" in the parameter file and "Bucket" on the bus; it is the member the
+         tool hangs from (distOutpLinkToTiltMnt = 0), so its attitude IS the tool's. -->
+    <xacro:imu_mount name="imu_link" parent="output_link"
+                     xyz="0.15 -0.12 0.05"
+                     rpy="1.575926179 0.001593256 -0.058849482"/>
+    <!-- imuTilt. Full axis permutation: sensor +X along the member's -Z. Its pitch is
+         88.0 deg, i.e. near the gimbal-lock pole of the rpy parameterization, so these
+         three numbers are individually ill-conditioned even though the matrix they
+         rebuild is exact to 7e-7. Do not hand-tune them; regenerate from a11..a33. -->
+    <xacro:imu_mount name="imu_tilt" parent="tilt_link"
+                     xyz="0.05 0.0 -0.08"
+                     rpy="0.911970428 1.536501790 2.473026331"/>
+    <!-- imuBm2 is deliberately absent. Its matrix in the firmware is the identity and
+         lenBm2 = 0: the slot exists on the bus, the sensor does not exist on the
+         machine. Emitting a frame for it would invent hardware. -->
+  </xacro:if>
   <xacro:macro name="ecr88_ros2_control_joint" params="name">
     <joint name="${name}">
@@ -1209,4 +1326,5 @@
       <xacro:ecr88_ros2_control_joint name="tilt_joint"/>
       <xacro:ecr88_ros2_control_joint name="rotator_joint"/>
+      <xacro:ecr88_ros2_control_joint name="dozer_joint"/>
     </ros2_control>
   </xacro:if>

File: assets/ecr88/urdf/ecr88_dynamics.xacro (robot description, xacro)
@@ -112,5 +112,6 @@
   <xacro:property name="m_contact_surface" value="180.0"/> <!-- CLASS-TYPICAL, NO SOURCE [L20]  suction plate assembly, the TCP link. -->
   <xacro:property name="m_track"       value="197.0"/>   <!-- DERIVED from PUBLISHED weight deltas [L21]  PER TRACK, rubber 450 mm. Volvo publishes the same machine with steel 450 (8 939 kg) and rubber 450 (8 752 kg): 187 kg for the pair, 93.5 kg per side. With a class typical steel chain of 290 kg/side (39 links at 154 mm pitch) the rubber track is 196.5 kg/side. -->
-  <xacro:property name="m_base_frame"  value="${m_base - 2*m_track}"/> <!-- DERIVED  = 2 319 kg. USE THIS for base_link when the two track links are emitted separately, so the tracks are not counted twice. See H2. -->
+  <xacro:property name="m_blade"       value="250.0"/>   <!-- CLASS-TYPICAL  kg, 2.32 m blade with its push arms and cylinder. Now that the blade is a real link it has to come OUT of m_base the same way the tracks did (H2), or the machine gains 250 kg. -->
+  <xacro:property name="m_base_frame"  value="${m_base - 2*m_track - m_blade}"/> <!-- DERIVED  = 2 319 kg. USE THIS for base_link when the two track links are emitted separately, so the tracks are not counted twice. See H2. -->
   <xacro:property name="m_marker"      value="0.01"/>    <!-- GUESS, TOKEN  coordinate frame markers (boom_mount, gnss x2, cyl anchors x3). Small enough to be dynamically irrelevant, large enough that no importer trips over it. -->
   <!-- Totals, COMPUTED so they cannot go stale. -->
@@ -421,4 +422,5 @@
   <xacro:property name="vel_conn_rod" value="${vel_bucket}"/> <!-- ALIAS  driven branch of the same 4 bar. -->
   <xacro:property name="vel_outp_link" value="${vel_bucket}"/> <!-- ALIAS  same joint as bucket_joint. -->
+  <xacro:property name="eff_dozer"    value="${cyl_relief_pa * pi / 4 * cyl_blade_bore * cyl_blade_bore * 0.55}"/> <!-- DERIVED  the blade cylinder pushes 390.2 kN and acts on roughly a 0.55 m moment arm about the blade pivot. Generous, and deliberately so: the blade's job in the calibration procedure is to jack the front of an 8.75 t machine off the ground, so an under-powered blade would silently fail the Pitch > 5 gate. -->
   <xacro:property name="vel_dozer"    value="0.5"/>       <!-- GUESS  the blade table is a passthrough (X = Y = [0, 0.001, 80]), i.e. the blade is NOT speed calibrated: it is commanded open loop. No firmware speed exists to take. -->
   <!-- ============================================================================

File: assets/ecr88/urdf/ecr88_params.xacro (robot description, xacro)
@@ -1044,6 +1044,30 @@
        "Dozer full down (Pitch angle > 5)". Cosmetic here, but it is the shape that
        most says "compact excavator" at a glance. Drawn on base_link, not articulated. -->
-  <xacro:property name="geo_blade_h"           value="0.42"/>    <!-- ASSUMPTION  m -->
-  <xacro:property name="geo_blade_t"           value="0.13"/>    <!-- ASSUMPTION  m -->
+  <xacro:property name="geo_blade_h"           value="0.42"/>    <!-- ASSUMPTION  m, blade plate height -->
+  <xacro:property name="geo_blade_t"           value="0.13"/>    <!-- ASSUMPTION  m, blade plate thickness -->
+  <xacro:property name="geo_blade_arm"         value="1.10"/>    <!-- CLASS-TYPICAL  m, pivot on the track frame to the cutting edge -->
+  <!-- Blade pivot, on the track frame just ahead of the front idler and near the track
+       bottom, which is where a compact excavator carries it. ASSUMPTION. -->
+  <xacro:property name="blade_pivot_x"         value="${lenBottomX * 0.5 - 0.10}"/>
+  <xacro:property name="blade_pivot_z"         value="${lenBottomZ1 + 0.22}"/>
+  <!-- BLADE RANGE. The firmware publishes JntAngDozerBlade and lists autoCtrlEnaDozer,
+       so this is a commanded axis, but neither the sheet nor the firmware carries its
+       limits. There IS a hard requirement to derive a floor from, though: the
+       calibration procedure will not start unless the blade can hold "Dozer full down,
+       Pitch angle > 5 deg", i.e. the blade alone has to jack the front of the machine
+       off the ground by 5 deg.
+         rear idler to cutting edge    = lenBottomX/2 + 0.10 + geo_blade_arm*cos(down)
+                                       ~ 2.62 m at the angle of interest
+         drop needed for 5 deg of pitch = 2.62 * tan(5 deg) = 0.229 m below the tracks
+         with geo_blade_arm = 1.10 m    = asin(0.229/1.10) = 12.0 deg below horizontal
+       So ANY range narrower than 12 deg down is provably wrong: it would fail a gate
+       the real machine passes. We take roughly double that, which also lands on the
+       class norm (blades in this size drop and lift about 0.4 m):
+         down 25 deg = 0.465 m below the tracks
+         up   30 deg = 0.550 m above
+       Tag CLASS-TYPICAL with a DERIVED floor. Replace from the working-range drawing
+       Teo has; that drawing carries the real numbers. -->
+  <xacro:property name="jntDozerLower"         value="${-pi/180*25}"/>
+  <xacro:property name="jntDozerUpper"         value="${ pi/180*30}"/>
   <!-- Crawler side profile. A track is a belt wrapped round an idler and a sprocket,
        so its silhouette is a rounded rectangle, not a slab. Rolling radius is half the
