Commit message: Boom swing becomes a real joint, and the firmware pins it to zero
While writing up the last change I claimed hasBmSwing was false and the
machine had no boom swing. Checked it: both ECR88D_LongArm.m and
ECR88D_ShortArm.m set hasBmSwing = true. The machine has the axis, the product
guide publishes its range (Q = 70 deg left, R = 60 deg right, offsets 760 and
860 mm), and MACH_POST_01P carries JntAngBoomSwing. boom_mount_joint was welded
shut; it is now boom_swing_joint, revolute about +Z, with the published limits.

The interesting part is what the firmware does with it:

    SysPar.m:72   JntAng_BmSwing = single(0*pi/180);

That is the only JntAng_ constant in the file, under "Kinematic parameters".
Every other joint angle on this machine is a difference of two IMU attitudes;
this one is a literal zero. It is structural rather than an oversight -- there
is no IMU on the swing post, no bmSwing entry in reqSpdToActCmd, and no
autoCtrlEnaBmSwing among the seven auto-control flags. The axis is manual-pedal
only and unsensed.

So the firmware cannot tell if somebody offsets the boom, and will keep
computing tool position as though it were centred: up to 860 mm of error
against a 20 mm placement tolerance. That is precisely what a simulation is
for, so the joint is real here rather than welded, and a SIL run can offset the
boom and watch the firmware's idea of the tool position walk away from the
truth. Rest pose is zero, the configuration the firmware assumes.

resources/X1Exc_control_surface.md is rewritten around what the parameter files
turned out to contain: the name-by-name comparison against the sheet (21/22
scalars and 10/11 vectors agreeing to 1e-6), the reqSpdToActCmd actuator
tables, the IMU scheme, and the two values where firmware and sheet disagree.

Co-Authored-By: Claude Opus 5 <noreply@anthropic.com>
Claude-Session: https://claude.ai/code/session_01YCTHKLKR3ccjDNMFVWse8H

File: assets/ecr88/urdf/ecr88.urdf.xacro (robot description, xacro)
@@ -587,8 +587,32 @@
     </xacro:viscol>
   </link>
-  <joint name="boom_mount_joint" type="fixed">
+  <!-- BOOM SWING (boom offset). Was welded shut here; corrected 2026-09-11.
+       ECR88D_LongArm.m and ECR88D_ShortArm.m both set hasBmSwing = true, and the
+       published product guide gives the range: Q = 70 deg left, R = 60 deg right.
+       The machine has this axis and MACH_POST_01P has a JntAngBoomSwing signal for it.
+       BUT THE FIRMWARE PINS IT TO ZERO, AND THAT IS WORTH KNOWING.
+         SysPar.m:72   JntAng_BmSwing = single(0*pi/180);
+       is the ONLY JntAng_ constant in the whole file, sitting under "Kinematic
+       parameters". Every other joint angle in this machine is a difference of two IMU
+       attitudes; this one is a literal. And the reason is structural, not an oversight:
+       there is no IMU on the swing post (the six are chs, bm1, bm2, arm, link, tilt),
+       there is no bmSwing entry in reqSpdToActCmd, and there is no autoCtrlEnaBmSwing
+       among the seven auto-control flags. The axis is manual-pedal only and unsensed.
+       So the firmware CANNOT TELL if somebody offsets the boom, and it will keep
+       computing the tool position as though the boom were centred. At full offset that
+       is 860 mm of error (published P), against a placement tolerance of 20 mm.
+       That is exactly the kind of thing the simulation exists to show, so the joint is
+       real here rather than welded: a SIL run can offset the boom and watch the
+       firmware's idea of where the tool is walk away from where it is. Rest pose is
+       zero, which is the configuration the firmware assumes and the one the machine
+       works panels in. -->
+  <joint name="boom_swing_joint" type="revolute">
     <parent link="house_link"/>
     <child  link="boom_mount_link"/>
     <origin xyz="${distChsToBmMnt_x} ${distChsToBmMnt_y} ${distChsToBmMnt_z}" rpy="0 0 0"/>
+    <axis xyz="0 0 1"/>
+    <limit lower="${lim_bm_swing_lower}" upper="${lim_bm_swing_upper}"
+           effort="${eff_bm_swing}" velocity="${vel_bm_swing}"/>
+    <dynamics damping="${dyn_damping}" friction="${dyn_friction}"/>
   </joint>
   <!-- Boom cylinder LARGE (cap/base) end pin, on the boom mount.
@@ -1326,4 +1350,5 @@
       <xacro:ecr88_ros2_control_joint name="tilt_joint"/>
       <xacro:ecr88_ros2_control_joint name="rotator_joint"/>
+      <xacro:ecr88_ros2_control_joint name="boom_swing_joint"/>
       <xacro:ecr88_ros2_control_joint name="dozer_joint"/>
     </ros2_control>

File: assets/ecr88/urdf/ecr88_dynamics.xacro (robot description, xacro)
@@ -423,4 +423,11 @@
   <xacro:property name="vel_outp_link" value="${vel_bucket}"/> <!-- ALIAS  same joint as bucket_joint. -->
   <xacro:property name="eff_dozer"    value="${cyl_relief_pa * pi / 4 * cyl_blade_bore * cyl_blade_bore * 0.55}"/> <!-- DERIVED  the blade cylinder pushes 390.2 kN and acts on roughly a 0.55 m moment arm about the blade pivot. Generous, and deliberately so: the blade's job in the calibration procedure is to jack the front of an 8.75 t machine off the ground, so an under-powered blade would silently fail the Pitch > 5 gate. -->
+  <xacro:property name="vel_bm_swing" value="0.3"/>       <!-- CLASS-TYPICAL  no firmware table exists: boom swing has no entry in reqSpdToActCmd and no autoCtrlEna flag, because it is not an auto-controlled axis. Manual pedal only. -->
+  <xacro:property name="eff_bm_swing" value="30000.0"/>   <!-- CLASS-TYPICAL, NO SOURCE  the offset ram's bore is not in the parts data we have. It only has to swing the front end, not dig with it. -->
+  <!-- Boom offset range, PUBLISHED: Q = 70 deg left, R = 60 deg right (product guide /
+       mateco EU guide), giving offsets O = 760 and P = 860 mm. Recorded in
+       resources/ECR88_estimated_dynamics.md section 1.1. +Z is left. -->
+  <xacro:property name="lim_bm_swing_lower" value="${-pi/180*60}"/>
+  <xacro:property name="lim_bm_swing_upper" value="${ pi/180*70}"/>
   <xacro:property name="vel_dozer"    value="0.5"/>       <!-- GUESS  the blade table is a passthrough (X = Y = [0, 0.001, 80]), i.e. the blade is NOT speed calibrated: it is commanded open loop. No firmware speed exists to take. -->
   <!-- ============================================================================
