Commit message: IMU frames transposed and imu_link moved to the input link; boom/arm/link speeds are cylinder m/s
Both corrections come from reading the X1Exc generated C, not from a log.

IMU mounting rotations: MdlApp.c:10940 is `linkOri = imuOri * mntOri`, so the
parameter-file matrix is R_imu<-link and a URDF child frame needs its transpose.
The previous revision used rpy(M) on the strength of an Rz*Rx(90) decomposition
that M' satisfies equally well, so it never discriminated. Board-normal alignment
does: under M' every side-plate board has sensor Z on its member's pin axis
(boom 0.999999, arm 0.999963, link 0.999986); under M the boom board is 32 deg off.
All five rpy regenerated from a11..a33 and round-tripped to 1.03e-7.

imu_link parent output_link -> input_link. KinematicsCalc computes
jntAng_ArmToInpLink = imus.link.euAng(2) - imus.arm.euAng(2) (MdlApp.c:11680) and
solves the four-bar for the output link from that. Emitted only when the four-bar
is modelled.

Velocity units: SetTarActuators builds the boom/arm/link actuator state with
CalStrkAndSpd (cylinder length and rate) before AutoVelDmdToVlvCmd interpolates it,
so bm1 0.41/0.48, arm 0.38/0.43, link 0.28/0.50 are m/s of stroke, not rad/s. As
joint limits they clipped the firmware's own demand by 2-4x. Limits are now the top
of the joint-rate band the firmware clamp implies through its own Jacobian over the
operating range (boom 2.1, arm 2.0, link 2.3 rad/s); the cylinder numbers move to
[4b] as cyl_spd_*. The earlier "every axis 2-3x too fast" comparison was void for
these three axes; it stands for swing, tilt and rotator.

Verified: validate_urdf 18 pass / 0 fail (same single warning as before),
USDs rebuilt, check_stability 10/10 joints converged.

Co-Authored-By: Claude Opus 5 (1M context) <noreply@anthropic.com>
Claude-Session: https://claude.ai/code/session_01YCTHKLKR3ccjDNMFVWse8H

File: assets/ecr88/urdf/ecr88.urdf.xacro (robot description, xacro)
@@ -1259,5 +1259,5 @@
          imuBm1   -> boom       JntAngBodyToBoom   = boom  - chassis
          imuArm   -> arm        JntAngBoom2ToArm   = arm   - boom
-         imuLink  -> output     JntAngArmToBucket  = output- arm
+         imuLink  -> INPUT link JntAngArmToInpLink = input - arm   (bus name: bktImu)
          imuTilt  -> tilt       JntAngTilt
        That is why there is no encoder anywhere in this machine, and it is why these
@@ -1272,16 +1272,29 @@
        accelerometer read. Position only enters through the lever-arm term under
        angular acceleration, which is small here and zero in steady motion.
-       All six matrices are proper rotations (det = +1, orthonormal to 1e-7), and the
-       three arm-chain boards decompose cleanly as Rz(yaw) * Rx(90 deg) with residuals
-       under 0.5 deg: the same board on a vertical side plate, the yaw being that
-       plate's angle to the member. imuBm1's yaw is 32.4 deg, which is the facet angle
-       you would expect on a curved gooseneck boom; imuArm and imuLink are -6.0 and
-       -3.4 deg, i.e. plates nearly parallel to their members. imuChs is flat and
-       yawed 101 deg (a box in the cabinet); imuTilt is a full axis permutation.
-       That consistency is the reason we read the matrix as IMU -> link rather than
-       its transpose: under the transpose the calibrated angle would be a rotation
-       about the sensor rather than about the member, which is not a thing a bracket
-       has. IF THE SIM'S CAN1 OUTPUT EVER DISAGREES WITH A RECORDED LOG BY A
-       TRANSPOSE, THIS IS THE ASSUMPTION TO OVERTURN FIRST.
+       All six matrices are proper rotations (det = +1, orthonormal to 1e-7).
+       THE MATRIX IS R_imu<-link, SO THESE rpy ARE rpy(M TRANSPOSE). (2026-09-14)
+       An earlier revision used rpy(M) and said "if this ever disagrees by a transpose,
+       overturn this first". It did, and it is overturned - by the firmware itself, not
+       by a log. The generated code (X1Exc MdlApp.c:10940, ImuToLink) is
+           linkOri = imuOri * mntOri
+       with imuOri = R_world<-imu from the quaternion. So mntOri = R_imu<-link, and a
+       URDF child frame (whose origin rotation is R_link<-imu) needs mntOri'.
+       The old argument for rpy(M) - "the arm-chain boards decompose as Rz(yaw)*Rx(90)"
+       - was never discriminating: M' decomposes just as cleanly as Rx(-90)*Rz(-yaw).
+       A test that DOES discriminate is where the board's normal points. A board bolted
+       flat to a side plate has its sensor Z on the member's pin axis (link Y):
+                    |<imu z, link Y>| under M'     under M (old)
+           imuBm1            0.999999            0.843883   <- 32 deg off
+           imuArm            0.999963            0.994412
+           imuLink           0.999986            0.998255
+           imuChs (vs Z)     0.999952            0.999952
+       Only the transpose puts every board flat on its plate. The yaw angles quoted in
+       the per-frame comments (32.4 / -6.0 / -3.4 / 101 deg) are unchanged in magnitude;
+       what changed is which frame they rotate.
+       OPEN: the SENSE of each axis. The firmware also mirrors the raw quaternion on
+       the way in, (w,x,y,z) -> (w,-x,y,-z) with acc/gyro X and Z negated ("Left handed
+       to right handed", MdlApp.c:10904-10915). A SIL publisher must pre-apply that
+       mirror. Whether any axis then comes out inverted is not decidable from source -
+       check MdlApp_Y.jnts.*.q against Isaac ground truth at one known pose.
        Each frame's axes are the SENSOR's axes, so a reading taken in this frame is
        directly comparable to the real CAN1 payload.
@@ -1304,26 +1317,35 @@
     <xacro:imu_mount name="imu_chs" parent="house_link"
                      xyz="0.20 0.30 ${lenUppZ1 + 0.25}"
-                     rpy="0.007485990 -0.006288474 1.762991172"/>
+                     rpy="-0.004742750 -0.008549333 -1.762994439"/>
     <!-- imuBm1. Side plate at 32.447 deg. Position: outboard face near the boom foot. -->
     <xacro:imu_mount name="imu_boom" parent="boom_link"
                      xyz="0.70 ${-geo_boom_sec_w * half - 0.02} 0.20"
-                     rpy="1.571657101 -0.001138020 0.566315716"/>
+                     rpy="-1.571816342 -0.566316481 -0.000590754"/>
     <!-- imuArm. Side plate at -6.043 deg. -->
     <xacro:imu_mount name="imu_arm" parent="arm_link"
                      xyz="0.45 ${-geo_arm_sec_w * half - 0.02} 0.12"
-                     rpy="1.579022612 -0.002439665 -0.105463699"/>
-    <!-- imuLink. Side plate at -3.372 deg. The firmware calls the 4-bar OUTPUT member
-         "Link" in the parameter file and "Bucket" on the bus; it is the member the
-         tool hangs from (distOutpLinkToTiltMnt = 0), so its attitude IS the tool's. -->
-    <xacro:imu_mount name="imu_link" parent="output_link"
-                     xyz="0.15 -0.12 0.05"
-                     rpy="1.575926179 0.001593256 -0.058849482"/>
-    <!-- imuTilt. Full axis permutation: sensor +X along the member's -Z. Its pitch is
-         88.0 deg, i.e. near the gimbal-lock pole of the rpy parameterization, so these
-         three numbers are individually ill-conditioned even though the matrix they
-         rebuild is exact to 7e-7. Do not hand-tune them; regenerate from a11..a33. -->
+                     rpy="-1.579068528 0.105440054 -0.003310372"/>
+    <!-- imuLink (bus: bktImu, CAN node 0x74). Side plate at -3.372 deg.
+         It is on the four-bar INPUT link, not the output link this frame used to hang
+         from. X1Exc KinematicsCalc (MdlApp.c:11680-11686):
+             jntAng_ArmToInpLink = imus.link.euAng(2) - imus.arm.euAng(2)
+             angInpLink = jntAng_ArmToInpLink - angArmToGndLink
+             [angConnRod, angOutpLink] = CalcAngLinkOutp(..., angInpLink)
+         i.e. the firmware reads the input-link angle and SOLVES the four-bar for the
+         output link. Mounting it on output_link would feed the solver the wrong member
+         and produce a silent tool-attitude error - the exact class of fault SIL is for.
+         Only emitted when the four-bar is modelled: without input_link there is no
+         member this sensor could honestly report. Position is a GUESS (side face). -->
+    <xacro:if value="$(arg model_bucket_fourbar)">
+      <xacro:imu_mount name="imu_link" parent="input_link"
+                       xyz="${lenInpLink * half} ${-geo_linkage_r - 0.02} 0"
+                       rpy="-1.575935070 0.058856870 0.001290998"/>
+    </xacro:if>
+    <!-- imuTilt. Full axis permutation. Under the transpose its pitch is -0.57 deg, so
+         the old gimbal-lock warning (pitch 88 deg under M) no longer applies; still,
+         regenerate from a11..a33 rather than hand-tuning. -->
     <xacro:imu_mount name="imu_tilt" parent="tilt_link"
                      xyz="0.05 0.0 -0.08"
-                     rpy="0.911970428 1.536501790 2.473026331"/>
+                     rpy="1.549803632 -0.010023128 -1.597706287"/>
     <!-- imuBm2 is deliberately absent. Its matrix in the firmware is the identity and
          lenBm2 = 0: the slot exists on the bus, the sensor does not exist on the

File: assets/ecr88/urdf/ecr88_dynamics.xacro (robot description, xacro)
@@ -390,15 +390,41 @@
   <!-- ============================================================================
        [4]  VELOCITY  [rad/s]
-       THESE ARE THE MACHINE'S OWN CALIBRATED NUMBERS, not our derivation.
-       XpannerLab/X1Exc  ControlModel/Data/ECR88D_LongArm.m, struct reqSpdToActCmd.
+       SOURCE: XpannerLab/X1Exc  ControlModel/Data/ECR88D_LongArm.m, struct reqSpdToActCmd.
        Each axis carries a 3 point table  X = [0, 0.001, vmax]  ->  Y = [0, deadband, cmdmax]
-       mapping a REQUESTED JOINT SPEED to a proportional valve command in percent. The
-       last X entry is therefore the fastest speed the firmware will ever ask for, and
-       the last Y entry is the command it asks for there.
-       WHAT THIS REPLACED, AND WHY IT WAS WRONG
-       The previous values here were derived as flow / bore area / moment arm with the
-       Stage V triple pump (2x68+54 l/min) summed onto one function. Every one of them
-       came out 2.0 to 3.0x the firmware number, consistently, which is the signature of
-       a wrong assumption rather than scattered error. Two reasons, both checkable:
+       mapping a REQUESTED ACTUATOR SPEED to a proportional valve command in percent. The
+       last X entry is the fastest speed the firmware will ever ask for.
+       !! THE X UNIT IS NOT THE SAME ON EVERY AXIS (corrected 2026-09-14) !!
+         swing, tilt, rot     joint rate, rad/s
+         bm1, arm, link       CYLINDER STROKE RATE, m/s
+       X1Exc SetTarActuators (Stateflow chart_1076) builds the boom/arm/link "actuator"
+       state as [q, qDot] = CalStrkAndSpd(lenToCylLrg*, lenToCylSml*, angCylLrg*, angCylSml*,
+       isCyl*TopMnt, jnt.q, jnt.qDot) - cylinder length and its rate - and AutoVelDmdToVlvCmd
+       (chart_2463) interpolates THAT into the table. An earlier revision of this file
+       wrote bm1 0.48 / arm 0.43 / link 0.50 straight in as rad/s. As joint limits they cut
+       what the firmware itself commands by 2-4x (table below), so a SIL run would have
+       shown a tracking error that is really the plant clipping the controller.
+       Joint rate implied by the firmware's own cylinder clamp, |qDot| = vmax / |dL/dq|, with
+       dL/dq from CalStrkAndSpd and LongArm geometry, over Olivia's range read in the
+       firmware sign convention (boom q <= 0, arm q >= 0; chart_1011 qBm1Max = 0, qArmMin = 0):
+         boom  0.48 m/s   q -69..-31 deg   |dL/dq| 0.235..0.412 m/rad   1.17..2.04 rad/s
+         arm   0.43 m/s   q  31..155 deg   |dL/dq| 0.215..0.515 m/rad   0.83..2.00 rad/s
+         link  0.50 m/s   q -120..-24 deg  |dL/dq| 0.220..0.420 m/rad   1.19..2.27 rad/s
+       The URDF limit takes the top of each band: it is a runaway guard, and it must not
+       bind before the (future) valve model does. The link band stops at -24 deg because
+       dL/dq -> 0 as the link cylinder goes over-centre near +16 deg, where any finite
+       stroke rate maps to an unbounded joint rate; that is a geometric singularity to keep
+       the joint away from, not a speed to allow.
+       CAUTION ON PHYSICAL REALISM: 0.48 m/s through a 105 mm bore is far more flow than
+       one function gets from this pump (the flow derivation below gave 0.262 m/s rod
+       speed). The boom/arm/link vmax look like DEMAND CLAMPS - they are round 2-figure
+       values, byte-identical between LongArm and ShortArm, where swing/tilt/rot carry
+       7-9 significant figures from a real calibration. So the tags on those three below
+       say what the number is: the firmware's clamp, not the machine's measured speed.
+       WHAT THE ROTARY AXES REPLACED (swing / tilt / rot - these comparisons stand)
+       The previous values were derived as flow / bore area / moment arm with the
+       Stage V triple pump (2x68+54 l/min) summed onto one function, or class-typical.
+       Swing, tilt and rotator came out 1.5 to 2.9x the firmware number. (This paragraph
+       used to say "every axis, 2.0 to 3.0x"; for boom/arm/link that compared m/s to
+       rad/s and was void.) Two reasons, both checkable:
          - the pump does not sum onto one implement function the way that derivation
            assumed (flagged there as an assumption, [L65]);
@@ -414,7 +440,7 @@
        ============================================================================ -->
   <xacro:property name="vel_swing"    value="0.5889427"/> <!-- OEM-FIRMWARE  swingLe 0.5889 / swingRi 0.5196 rad/s = 5.6 / 5.0 r/min. NOTE this is well under the published free swing speed (8.3 r/min, 0.869 rad/s): swing is the one axis whose command is capped at 60 % instead of 80 %, which is what you would do on a machine carrying glass. The published figure describes the bare ECR88; this one describes it under X1. -->
-  <xacro:property name="vel_boom"     value="0.48"/>      <!-- OEM-FIRMWARE  bm1Up 0.41 / bm1Down 0.48 rad/s -->
-  <xacro:property name="vel_arm"      value="0.43"/>      <!-- OEM-FIRMWARE  armIn 0.38 / armOut 0.43 rad/s -->
-  <xacro:property name="vel_bucket"   value="0.50"/>      <!-- OEM-FIRMWARE  linkIn 0.28 / linkOut 0.50 rad/s. The firmware calls this axis "link", not "bucket": on this machine the cylinder drives the 4 bar input link and the attachment hangs off the output link. Same joint, the firmware's name for it is the more accurate one. -->
+  <xacro:property name="vel_boom"     value="2.1"/>       <!-- DERIVED (OEM-FIRMWARE demand clamp x CalStrkAndSpd Jacobian)  0.48 m/s cylinder -> 1.17..2.04 rad/s over the boom range; see the table above. The cylinder numbers themselves are cyl_spd_bm1_* in [4b]. -->
+  <xacro:property name="vel_arm"      value="2.0"/>       <!-- DERIVED (same)  0.43 m/s cylinder -> 0.83..2.00 rad/s. -->
+  <xacro:property name="vel_bucket"   value="2.3"/>       <!-- DERIVED (same)  0.50 m/s cylinder -> 1.19..2.27 rad/s. The firmware calls this axis "link", not "bucket": the cylinder drives the 4 bar input link and the attachment hangs off the output link. Same joint, the firmware's name for it is the more accurate one. -->
   <xacro:property name="vel_tilt"     value="0.2311245"/> <!-- OEM-FIRMWARE  tiltPosi 0.2033 / tiltNega 0.2311 rad/s -->
   <xacro:property name="vel_rotator"  value="0.342202"/>  <!-- OEM-FIRMWARE  rotPosi 0.3186 / rotNega 0.3422 rad/s = 3.3 r/min. Our CLASS-TYPICAL guess of 9.5 r/min was 2.9x too fast. -->
@@ -443,4 +469,6 @@
          PropVlvCmdAutoLimit   = 70 %                (SysPar.m:251)
              ceiling in auto mode, below several of the cmdmax values below
+       Actuator speed at cmdmax (table X end). UNITS DIFFER BY AXIS - see [4]:
+       rad/s for swing/tilt/rot (vel_* above), m/s of CYLINDER STROKE for these three.
        Nothing in the URDF consumes these yet. They live here so the number sits with the
        joint it belongs to when the valve model is written.
@@ -448,4 +476,10 @@
   <xacro:property name="vlv_swing_le"  value="32.0"/>  <xacro:property name="vlv_swing_le_max"  value="60.0"/>
   <xacro:property name="vlv_swing_ri"  value="28.7"/>  <xacro:property name="vlv_swing_ri_max"  value="60.0"/>
+  <xacro:property name="cyl_spd_bm1_up"   value="0.41"/> <!-- OEM-FIRMWARE  m/s cylinder, reqSpdToActCmd.bm1Up_X(end). Demand clamp, see [4]. -->
+  <xacro:property name="cyl_spd_bm1_dn"   value="0.48"/> <!-- OEM-FIRMWARE  m/s cylinder, bm1Down_X(end) -->
+  <xacro:property name="cyl_spd_arm_in"   value="0.38"/> <!-- OEM-FIRMWARE  m/s cylinder, armIn_X(end) -->
+  <xacro:property name="cyl_spd_arm_out"  value="0.43"/> <!-- OEM-FIRMWARE  m/s cylinder, armOut_X(end) -->
+  <xacro:property name="cyl_spd_link_in"  value="0.28"/> <!-- OEM-FIRMWARE  m/s cylinder, linkIn_X(end) -->
+  <xacro:property name="cyl_spd_link_out" value="0.50"/> <!-- OEM-FIRMWARE  m/s cylinder, linkOut_X(end) -->
   <xacro:property name="vlv_boom_up"   value="34.0"/>  <xacro:property name="vlv_boom_up_max"   value="80.0"/>
   <xacro:property name="vlv_boom_dn"   value="31.0"/>  <xacro:property name="vlv_boom_dn_max"   value="80.0"/>
