Commit message: Fork, joint limits and work cycle rebuilt on the firmware's own frames
Three things were wrong together, and each hid the others.

1. The panel stack. X1Exc defines the carriage as forkBack = uc (+) Ry(angForkUpLimit)
   (+) distUcToForkBack and panelTop = forkBack (+) Ry(pi/2) (+) distForkBackToPanelTop
   (MdlApp.c:12754-12949): modules STAND on the tip-up pallet leaning on the backrest,
   the pick point is the outermost face 1.0165 m out along the blade, and the tool meets
   it face-on (approach = panelTop + 0.5 m, dirRef = -blade). The asset drew them lying
   flat and placed the carriage from the `old` sheet's LenPL* rows with an assumed X.
   Now: fork_back_link / panel_top_link / panel_pick_approach_link / panel_lift_posn_link
   under the firmware's names, distUcToForkBack = (1.844, 0, -0.7022) from the compiled
   binary (sheet 1.988/-0.66 was the pre-calibration entry), angForkUpLimit and
   distPanelTopToLiftPosn per variant, a full 30 x 30 mm stack whose outer face is at
   panelTop.

2. Boom and arm limits. The tablet angle Olivia's figures come from is
   MdlApp_Y.jnts.*.q x RAD_TO_DEG with no offset (AppCtrlIf.c:723 -> PrePostProc_If.c:1810
   -> CAN2 JntAngBodyToBoom), and the SIL suite showed firmware q == URDF q in zero and
   sign. So boom -69..-31 and arm 31..155 are used literally, as bucket already was. The
   old arm 0..124 began past the firmware arm cylinder's +5.6 deg dead centre.

3. The work cycle. It picked from a ground pallet to the machine's right, which the
   machine never does, while the camera study scored a point on the fork stack that the
   cycle never visited. assets/ecr88/cycle.json is now the single source for
   animate_cycle.py and camera_study.py / optimize_cameras.py, shaped after the state
   machine: raised home -> approach -> contact (tool on panelTop, 0.2 mm) -> grip ->
   lift past the firmware clearance gates (output link 1.98 m, tool 0.95 m) -> slew ->
   set down on the row (0.1 mm) -> release -> return. Solved by planar IK inside the
   new limits. With the old limits the tool could not reach the stack at all.

Camera scoring: the pick target is the outer module's upper edge (the face centre is
under the suction pad from ~0.3 m out). The house-front and arm-root mounts already sit
at the new optimum (pick 67 %, the ceiling for every candidate; place 100 % / cups 75 %).
Since 7fc1a4f (fork blade 1.45 -> 1.06) the published "fork mast sees the pick 100 %"
no longer held; it was scoring the old flat-stack point.

Verified: validate_urdf 18 pass / 0 fail on all three variants, USDs rebuilt, animation
authored within USD joint limits, check_stability 10/10 converged at the new rest pose.

Co-Authored-By: Claude Opus 5 (1M context) <noreply@anthropic.com>
Claude-Session: https://claude.ai/code/session_01YCTHKLKR3ccjDNMFVWse8H

File: assets/ecr88/urdf/ecr88.urdf.xacro (robot description, xacro)
@@ -1116,52 +1116,111 @@
        goes into the TABLET's kinematic dataset, not what the machine physically
        has; the fork is drawn here as geometry and drives nothing.
-       Pallet base tilts by AlphaPL2 (15.7 deg) and the backrest by AlphaPL1
-       (74.5 deg), both straight from the sheet's protractor readings, so the stack
-       leans back the way it does on the real carriage.
+       GEOMETRY IS THE FIRMWARE'S (rebuilt 2026-09-14). The X1Exc kinematics define the
+       carriage entirely through three frames (MdlApp.c:12754-12949):
+           uc        = chassis (+) Rz(swing)                      zero offset
+           forkBack  = uc (+) Ry(angForkUpLimit) (+) distUcToForkBack
+           panelTop  = forkBack (+) Ry(pi/2) (+) distForkBackToPanelTop (along the blade)
+           approach  = panelTop (+) [0, 0, TarPanelPickupMargin]
+           liftPosn  = panelTop (+) distPanelTopToLiftPosn
+       and they are emitted below under exactly those names, so a SIL comparator can put
+       Isaac ground truth next to MdlApp_Y.objects/links frame for frame.
+       WHAT THAT MEANS PHYSICALLY. The pallet base is tilted tip-up by angForkUpLimit
+       (sheet AlphaPL2 = 15.7 deg agrees), the backrest is square to it (AlphaPL1 +
+       AlphaPL2 = 90.2 deg), and the modules STAND on the base leaning on the backrest.
+       The stack's "top" is its outermost face, 1.0165 m out along the blade; the tool
+       meets it face-on with contact_surface Z along the blade, approaching back toward
+       the machine (dirRef = -panelTopWithMargin.R(:,3), MdlApp.c:6760). forkBack's
+       origin is where CalibForkRefPose found the cups against the bare backrest, so it
+       sits at cup height, not at the pallet corner.
+       WHAT THIS REPLACED. The carriage used to be placed from the `old` sheet's LenPL*
+       rows with an assumed X (LenPLX taken literally put it inside the house), and the
+       modules were drawn LYING FLAT on the pallet with the tool expected to come down
+       on them from above. Two consequences surfaced when the firmware frames were
+       checked: no pose in the joint limits could put the tool face-down on that flat
+       stack, and the camera study was scoring a "pick" point the work cycle never
+       visited. The LenPL* rows stay in the params file for reference only.
+       STILL ASSUMED (flagged, not hidden): the stack's vertical extent is the sheet's
+       LenPanelHeight centred on cup height, its width is LenPLWidth, and the 2.1 m
+       build borrows the 1.7 m unit's calibrated carriage (the LongArm parameter file is
+       on the old schema and has no distUcToForkBack).
        ===================================================================== -->
   <xacro:if value="$(arg model_fork)">
+    <xacro:property name="stack_depth" value="${panels_per_stack * geo_panel_t}"/>
+    <!-- forkBack: firmware frame, zero mass. -->
+    <link name="fork_back_link">
+      <xacro:inertial_sphere mass="${m_marker}" radius="${geo_marker_r}"/>
+      <xacro:detail_visual material="xpanner_accent"><sphere radius="${geo_marker_r}"/></xacro:detail_visual>
+    </link>
+    <joint name="fork_back_joint" type="fixed">
+      <parent link="base_link"/>
+      <child  link="fork_back_link"/>
+      <origin xyz="${distUcToForkBackX} ${distUcToForkBackY} ${distUcToForkBackZ}"
+              rpy="0 ${angForkUpLimit} 0"/>
+    </joint>
+    <!-- Carriage: pallet base along forkBack +X, backrest along +Z, square to each other.
+         Its origin is the base/backrest corner, stack_bottom below cup height. -->
     <link name="fork_link">
       <xacro:inertial_box mass="${m_fork}"
                           x="${geo_fork_len}" y="${LenPLWidth}" z="${geo_fork_t}"
-                          xyz="${geo_fork_len * half} 0 0"/>
-      <!-- pallet base, tilted back by AlphaPL2 -->
+                          xyz="${geo_fork_len * half} 0 ${-geo_fork_t * half}"/>
       <xacro:viscol name="fork_link" material="xpanner_dark"
-                    xyz="${geo_fork_len * half} 0 0" rpy="0 ${-AlphaPL2} 0">
+                    xyz="${geo_fork_len * half} 0 ${-geo_fork_t * half}">
         <box size="${geo_fork_len} ${LenPLWidth} ${geo_fork_t}"/>
       </xacro:viscol>
-      <!-- backrest the stack leans on, tilted by AlphaPL1 -->
       <xacro:detail material="xpanner_dark"
-                    xyz="0 0 ${geo_fork_back_h * half}" rpy="0 ${half_pi - AlphaPL1} 0">
-        <box size="${geo_fork_back_h} ${LenPLWidth} ${geo_fork_t}"/>
+                    xyz="${-geo_fork_t * half} 0 ${geo_fork_back_h * half}">
+        <box size="${geo_fork_t} ${LenPLWidth} ${geo_fork_back_h}"/>
       </xacro:detail>
     </link>
     <joint name="fork_joint" type="fixed">
-      <parent link="base_link"/>
+      <parent link="fork_back_link"/>
       <child  link="fork_link"/>
-      <!-- X IS NOT LenPLX. Taken literally, LenPLX = 1.086 puts the carriage inside
-           the machine: the house box reaches x = +1.14 and the undercarriage +1.41,
-           so a 1.25 m mast at x = 1.086 rises straight through the house. It showed up
-           as cam_fork_mast being occluded by house_link on every pose of the cycle.
-           LenPLX is evidently measured to some other fork reference, not to the
-           carriage root. Until that is pinned down, the carriage is placed clear of
-           the undercarriage front, which is where a forklift carriage physically is.
-           Y and Z ARE the sheet's (LenPLY, LenPLZ); only X is overridden. -->
-      <origin xyz="${lenBottomX * half + geo_fork_clear} ${LenPLY} ${LenPLZ}" rpy="0 0 0"/>
+      <origin xyz="0 0 ${-LenPanelHeight * half}" rpy="0 0 0"/>
     </joint>
-    <!-- The stack itself. Modules lie flat on the tilted pallet, one on top of the
-         next; the tool takes them off the top. Count is a scene choice, not data. -->
+    <!-- The stack: a full load of panels_per_stack modules standing on the base. The
+         firmware has no stack model - it commands the same fork-relative panelTop every
+         cycle and relies on the all-four-cups contact to stop the approach - so the
+         OUTER FACE is what has to be right, and it is drawn at panelTop. -->
     <link name="panel_stack_link">
-      <xacro:inertial_box mass="${m_panel * n_panels}"
-                          x="${LenPanelHeight}" y="${LenPLWidth}" z="${n_panels * geo_panel_t}"
-                          xyz="0 0 ${n_panels * geo_panel_t * half}"/>
+      <xacro:inertial_box mass="${m_panel * panels_per_stack}"
+                          x="${stack_depth}" y="${LenPLWidth}" z="${LenPanelHeight}"
+                          xyz="${distForkBackToPanelTopX - stack_depth * half} 0 0"/>
       <xacro:viscol name="panel_stack_link" material="xpanner_panel"
-                    xyz="0 0 ${n_panels * geo_panel_t * half}">
-        <box size="${LenPanelHeight} ${LenPLWidth} ${n_panels * geo_panel_t}"/>
+                    xyz="${distForkBackToPanelTopX - stack_depth * half} 0 0">
+        <box size="${stack_depth} ${LenPLWidth} ${LenPanelHeight}"/>
       </xacro:viscol>
     </link>
     <joint name="panel_stack_joint" type="fixed">
-      <parent link="fork_link"/>
+      <parent link="fork_back_link"/>
       <child  link="panel_stack_link"/>
-      <origin xyz="${geo_fork_len * half} 0 ${geo_fork_t * half}" rpy="0 ${-AlphaPL2} 0"/>
+      <origin xyz="0 0 0" rpy="0 0 0"/>
+    </joint>
+    <!-- panelTop: the firmware's pick frame. contact_surface must reach this pose. -->
+    <link name="panel_top_link">
+      <xacro:inertial_sphere mass="${m_marker}" radius="${geo_marker_r}"/>
+    </link>
+    <joint name="panel_top_joint" type="fixed">
+      <parent link="fork_back_link"/>
+      <child  link="panel_top_link"/>
+      <origin xyz="${distForkBackToPanelTopX} ${distForkBackToPanelTopY} ${distForkBackToPanelTopZ}"
+              rpy="0 ${half_pi} 0"/>
+    </joint>
+    <!-- panelTopWithMargin: where ApproachPanel starts. -->
+    <link name="panel_pick_approach_link">
+      <xacro:inertial_sphere mass="${m_marker}" radius="${geo_marker_r}"/>
+    </link>
+    <joint name="panel_pick_approach_joint" type="fixed">
+      <parent link="panel_top_link"/>
+      <child  link="panel_pick_approach_link"/>
+      <origin xyz="0 0 ${TarPanelPickupMargin}" rpy="0 0 0"/>
+    </joint>
+    <!-- panelLiftPosn: the Placing/Lift target (variant specific). -->
+    <link name="panel_lift_posn_link">
+      <xacro:inertial_sphere mass="${m_marker}" radius="${geo_marker_r}"/>
+    </link>
+    <joint name="panel_lift_posn_joint" type="fixed">
+      <parent link="panel_top_link"/>
+      <child  link="panel_lift_posn_link"/>
+      <origin xyz="${distPanelTopToLiftPosnX} 0 ${distPanelTopToLiftPosnZ}" rpy="0 0 0"/>
     </joint>
   </xacro:if>

File: assets/ecr88/urdf/ecr88_dynamics.xacro (robot description, xacro)
@@ -151,8 +151,25 @@
          jntBm1Lower/Upper in params compute the same thing; they are the same two
          numbers by construction and are now unused aliases. -->
-  <xacro:property name="lim_boom_lower"   value="${deg * (bm1GroundContactUrdf - oemBm1AngleSpan)}"/>
-                                      <!-- OEM-TEAM span + DERIVED placement [L42]  boom fully UP. -->
-  <xacro:property name="lim_boom_upper"   value="${deg * bm1GroundContactUrdf}"/>
-                                      <!-- OEM-TEAM span + DERIVED placement [L42]  boom DOWN, TCP at ground. -->
+  <!-- 2026-09-14: SUPERSEDED. Olivia's numbers are now used LITERALLY, boom -69..-31 and
+       arm 31..155 deg, because the chain from firmware joint angle to the tablet she
+       reads them from has been traced end to end and it has no offset:
+           MdlApp_Y.jnts.BmMntToBm1.q [rad]      X1Exc AppCtrlIf.c:723
+             x RAD_TO_DEG, nothing added          PrePostProc_If.c:1810
+             -> CAN2 JntAngBodyToBoom [deg] -> HMI OutpHndlr.c:122, CAN2_X1Exc.dbc:224
+       (same for Bm2ToArm -> JntAngBoom2ToArm, and ArmToOutpLink -> JntAngArmToBucket),
+       and the SIL suite showed the firmware's joint angles have the SAME zero and sign
+       as this URDF's boom_joint / arm_joint / bucket_joint (sil/tests/
+       test_imu_kinematics.py, published poses reproduced to 0.002 deg). The bucket
+       limit was already taken literally; boom and arm were not, which was inconsistent.
+       Independent support: the firmware's own arm-cylinder geometry has a dead centre at
+       q = +5.6 deg, so the old arm range 0..124 started in a pose the hydraulics cannot
+       drive through, while 31..155 lies entirely on the valid side; and with these limits
+       the tool reaches the firmware's panelTop pick frame (0.2 mm), which the old limits
+       could not do for the flat-stack geometry. Remaining assumption: that Olivia read the
+       values off the tablet. The bisection anchor below is kept for the record only. -->
+  <xacro:property name="lim_boom_lower"   value="${deg * -69.00}"/>
+                                      <!-- OEM-TEAM literal, firmware convention verified [L42]  boom fully UP. -->
+  <xacro:property name="lim_boom_upper"   value="${deg * -31.00}"/>
+                                      <!-- OEM-TEAM literal, firmware convention verified [L42]  boom DOWN ("붐다운 바닥기준"). -->
   <!-- BOOM, MECHANICAL envelope. Needed for trenching; the PanelLift range above cannot
        dig at all (38 deg of boom never reaches below ground, and the published 4 130 mm
@@ -187,6 +204,11 @@
        So the span is kept and the out stop is ASSUMED at collinear, on the standard
        layout plus ref_arm_deadcentre. NOTE H3 on the sign and H5 on the tag. -->
-  <xacro:property name="lim_arm_lower"    value="${deg *   0.00}"/>   <!-- ASSUMPTION [L44], was DERIVED until the H residual was withdrawn (H5)  arm fully OUT, collinear with the boom. NO published figure discriminates this placement. Standing support: it is the standard layout, and the arm cylinder is within 5.6 deg of dead centre here (moment arm 72 mm), so a STRUCTURAL stop belongs about there: prefer a SOFT joint limit. If the true out stop is -10 deg instead, ref_bucket_radius becomes 0.802 and lim_boom_mech_lower becomes -66.56 deg. Teo's cylinder strokes settle it. -->
-  <xacro:property name="lim_arm_upper"    value="${deg * 124.00}"/>   <!-- OEM-TEAM span [L43]  arm fully IN (interior angle 56 deg). -->
+  <!-- 2026-09-14: SUPERSEDED by the literal 31..155, see the boom block above. The
+       stroke-ratio objection (a) does not survive the firmware cylinder geometry: arm
+       stroke 1.395 -> 2.327 m over 31..155 is an extended/retracted ratio of 1.67,
+       buildable; and the old 0 lower bound sits past the +5.6 deg dead centre. -->
+  <xacro:property name="lim_arm_lower_superseded" value="${deg *   0.00}"/>   <!-- ASSUMPTION [L44], was DERIVED until the H residual was withdrawn (H5)  arm fully OUT, collinear with the boom. NO published figure discriminates this placement. Standing support: it is the standard layout, and the arm cylinder is within 5.6 deg of dead centre here (moment arm 72 mm), so a STRUCTURAL stop belongs about there: prefer a SOFT joint limit. If the true out stop is -10 deg instead, ref_bucket_radius becomes 0.802 and lim_boom_mech_lower becomes -66.56 deg. Teo's cylinder strokes settle it. -->
+  <xacro:property name="lim_arm_lower"    value="${deg *  31.00}"/>   <!-- OEM-TEAM literal "31(암아웃)", firmware convention verified [L43] -->
+  <xacro:property name="lim_arm_upper"    value="${deg * 155.00}"/>   <!-- OEM-TEAM literal "155(암인)", firmware convention verified [L43] -->
   <!-- 2026-09-11 UPDATE, Olivia (Slack #simulation, 11:28 KST). The original relay of her
        figures carried no direction words; the full message does:

File: assets/ecr88/urdf/ecr88_params.xacro (robot description, xacro)
@@ -422,12 +422,28 @@
                              measurements, no release row exists.
        ======================================================================== -->
-  <!-- 처리구분 = Update after Calibration. Do NOT hardcode downstream. -->
-  <xacro:property name="distUcToForkBackX"     value="1.988"/>
-  <xacro:property name="distUcToForkBackY"     value="0.0"/>
-  <xacro:property name="distUcToForkBackZ"     value="-0.66"/>
+  <!-- 처리구분 = Update after Calibration. Do NOT hardcode downstream.
+       2026-09-14: the sheet's 기장 values (1.988, 0, -0.66) are the PRE-calibration
+       entry; the calibrated value the firmware actually runs is in the compiled X1Exc
+       binary (ECR88D_ShortArm.m:176, MdlApp.c:499): (1.844, 0, -0.7022). Adopted.
+       ForkBack is the pose CalibForkRefPose (step 28) records with the contact surface
+       held against the backrest, so its origin is where the cups meet the stack, not
+       the corner of the pallet. The uc frame is the chassis origin (MdlApp.c:12754,
+       zero offset). ECR88D_LongArm.m is on the OLD schema and has no distUcToForkBack,
+       so the 2.1 m build borrows the 1.7 m unit's calibrated carriage: same
+       undercarriage and fork hardware assumed. -->
+  <xacro:property name="distUcToForkBackX"     value="1.844"/>  <!-- OEM-FIRMWARE (ShortArm unit; sheet pre-calibration 1.988) -->
+  <xacro:property name="distUcToForkBackY"     value="0.0"/>    <!-- OEM-FIRMWARE -->
+  <xacro:property name="distUcToForkBackZ"     value="-0.7022"/> <!-- OEM-FIRMWARE (sheet pre-calibration -0.66) -->
   <!-- 처리구분 = Update after Calibration. -->
   <xacro:property name="distForkBackToPanelTopX" value="1.0165"/>
   <xacro:property name="distForkBackToPanelTopY" value="0.0"/>
   <xacro:property name="distForkBackToPanelTopZ" value="0.0"/>
+  <!-- 1.0165 matches the compiled firmware exactly (ECR88D_ShortArm.m:177). It is measured
+       ALONG THE FORK BLADE: panelTop = forkBack * Ry(pi/2) (+) this offset in the forkBack
+       frame (MdlApp.c:12788). The modules stand on the tilted pallet leaning on the
+       backrest; "top" is the outermost module face, 1.0165 m out along the blade, and the
+       tool meets it face-on, approaching back toward the machine. 30 x 30 mm = 0.90 m of
+       glass fills that blade. -->
+  <xacro:property name="TarPanelPickupMargin"  value="0.5"/>    <!-- OEM-FIRMWARE  SysPar.m, m. Approach point = panelTop (+) [0,0,margin]: 0.5 m out in front of the outer face (MdlApp.c:12930). -->
   <!-- 처리구분 = Update after Calibration.
        The ONE row in the whole parameter set that is genuinely a joint LIMIT
@@ -517,4 +533,7 @@
     <xacro:property name="distAttToContactSurfaceZ"   value="-0.836" scope="global"/>
     <xacro:property name="fork_chain_valid"    value="true"    scope="global"/>
+    <xacro:property name="angForkUpLimit"      value="${-pi/180*16.3246}" scope="global"/> <!-- OEM-FIRMWARE ECR88D_ShortArm.m:210 -->
+    <xacro:property name="distPanelTopToLiftPosnX" value="-3.0" scope="global"/> <!-- OEM-FIRMWARE ECR88D_ShortArm.m:178 -->
+    <xacro:property name="distPanelTopToLiftPosnZ" value="2.0"  scope="global"/>
   </xacro:if>
   <xacro:if value="${machine_variant == 'ECR88_US1_2P1M'}">
@@ -535,4 +554,6 @@
          suppressed for this variant rather than built at the origin. -->
     <xacro:property name="fork_chain_valid"    value="false"   scope="global"/>
+    <xacro:property name="distPanelTopToLiftPosnX" value="-1.0" scope="global"/> <!-- OEM-FIRMWARE ECR88D_LongArm.m:170 -->
+    <xacro:property name="distPanelTopToLiftPosnZ" value="2.0"  scope="global"/>
   </xacro:if>
   <xacro:if value="${machine_variant == 'ECR88_US1_2P1M_NEWSUCTION'}">
@@ -551,4 +572,6 @@
     <xacro:property name="distAttToContactSurfaceZ"   value="-0.832" scope="global"/>
     <xacro:property name="fork_chain_valid"    value="true"    scope="global"/>
+    <xacro:property name="distPanelTopToLiftPosnX" value="-1.0" scope="global"/> <!-- OEM-FIRMWARE ECR88D_LongArm.m:170 -->
+    <xacro:property name="distPanelTopToLiftPosnZ" value="2.0"  scope="global"/>
   </xacro:if>
   <!-- ========================================================================
