Commit message: IMU mount rotations are per machine variant
Mount matrices are per-unit calibration results. The 2.1 m variants keep rpy(M') of
ECR88D_LongArm.m (output byte-identical); ECR88_KIJANG now uses ECR88D_ShortArm.m, the
unit the repo's X1Exc binary is compiled with, so a 1.7 m SIL run reads its own IMUs.
Mixing the two misreads arm/link by ~4 deg with no fault (sil/tests/test_imu_kinematics).
Values recomputed independently and matched the SIL agent's to 4e-9. The five literals
moved from the URDF body into the params branches.

Co-Authored-By: Claude Opus 5 (1M context) <noreply@anthropic.com>
Claude-Session: https://claude.ai/code/session_01YCTHKLKR3ccjDNMFVWse8H

File: assets/ecr88/urdf/ecr88.urdf.xacro (robot description, xacro)
@@ -1376,13 +1376,13 @@
     <xacro:imu_mount name="imu_chs" parent="house_link"
                      xyz="0.20 0.30 ${lenUppZ1 + 0.25}"
-                     rpy="-0.004742750 -0.008549333 -1.762994439"/>
+                     rpy="${imu_rpy_chs}"/>
     <!-- imuBm1. Side plate at 32.447 deg. Position: outboard face near the boom foot. -->
     <xacro:imu_mount name="imu_boom" parent="boom_link"
                      xyz="0.70 ${-geo_boom_sec_w * half - 0.02} 0.20"
-                     rpy="-1.571816342 -0.566316481 -0.000590754"/>
+                     rpy="${imu_rpy_boom}"/>
     <!-- imuArm. Side plate at -6.043 deg. -->
     <xacro:imu_mount name="imu_arm" parent="arm_link"
                      xyz="0.45 ${-geo_arm_sec_w * half - 0.02} 0.12"
-                     rpy="-1.579068528 0.105440054 -0.003310372"/>
+                     rpy="${imu_rpy_arm}"/>
     <!-- imuLink (bus: bktImu, CAN node 0x74). Side plate at -3.372 deg.
          It is on the four-bar INPUT link, not the output link this frame used to hang
@@ -1399,5 +1399,5 @@
       <xacro:imu_mount name="imu_link" parent="input_link"
                        xyz="${lenInpLink * half} ${-geo_linkage_r - 0.02} 0"
-                       rpy="-1.575935070 0.058856870 0.001290998"/>
+                       rpy="${imu_rpy_link}"/>
     </xacro:if>
     <!-- imuTilt. Full axis permutation. Under the transpose its pitch is -0.57 deg, so
@@ -1406,5 +1406,5 @@
     <xacro:imu_mount name="imu_tilt" parent="tilt_link"
                      xyz="0.05 0.0 -0.08"
-                     rpy="1.549803632 -0.010023128 -1.597706287"/>
+                     rpy="${imu_rpy_tilt}"/>
     <!-- imuBm2 is deliberately absent. Its matrix in the firmware is the identity and
          lenBm2 = 0: the slot exists on the bus, the sensor does not exist on the

File: assets/ecr88/urdf/ecr88_params.xacro (robot description, xacro)
@@ -536,4 +536,12 @@
     <xacro:property name="distPanelTopToLiftPosnX" value="-3.0" scope="global"/> <!-- OEM-FIRMWARE ECR88D_ShortArm.m:178 -->
     <xacro:property name="distPanelTopToLiftPosnZ" value="2.0"  scope="global"/>
+    <!-- IMU mounting rotations = rpy(M transpose) of the ECR88D_ShortArm.m (1.7 m, the unit the repo's binary is compiled for) imu* matrices. Mounts are PER-UNIT calibration
+         results: pairing a URDF from one unit with a firmware carrying another misreads arm/link by ~4 deg
+         with no fault (sil/tests/test_imu_kinematics.py). -->
+    <xacro:property name="imu_rpy_chs" value="-0.001755416 -0.002555442 -1.783640195" scope="global"/>
+    <xacro:property name="imu_rpy_boom" value="-1.567613598 -0.571866959 0.006005104" scope="global"/>
+    <xacro:property name="imu_rpy_arm" value="-1.573310335 0.033289461 -0.003775542" scope="global"/>
+    <xacro:property name="imu_rpy_link" value="-1.575791294 0.068579979 -0.006844645" scope="global"/>
+    <xacro:property name="imu_rpy_tilt" value="1.579079426 -0.015406954 -1.622796371" scope="global"/>
   </xacro:if>
   <xacro:if value="${machine_variant == 'ECR88_US1_2P1M'}">
@@ -556,4 +564,12 @@
     <xacro:property name="distPanelTopToLiftPosnX" value="-1.0" scope="global"/> <!-- OEM-FIRMWARE ECR88D_LongArm.m:170 -->
     <xacro:property name="distPanelTopToLiftPosnZ" value="2.0"  scope="global"/>
+    <!-- IMU mounting rotations = rpy(M transpose) of the ECR88D_LongArm.m (2.1 m US unit) imu* matrices. Mounts are PER-UNIT calibration
+         results: pairing a URDF from one unit with a firmware carrying another misreads arm/link by ~4 deg
+         with no fault (sil/tests/test_imu_kinematics.py). -->
+    <xacro:property name="imu_rpy_chs" value="-0.004742750 -0.008549333 -1.762994439" scope="global"/>
+    <xacro:property name="imu_rpy_boom" value="-1.571816342 -0.566316481 -0.000590754" scope="global"/>
+    <xacro:property name="imu_rpy_arm" value="-1.579068528 0.105440054 -0.003310372" scope="global"/>
+    <xacro:property name="imu_rpy_link" value="-1.575935070 0.058856870 0.001290998" scope="global"/>
+    <xacro:property name="imu_rpy_tilt" value="1.549803632 -0.010023128 -1.597706287" scope="global"/>
   </xacro:if>
   <xacro:if value="${machine_variant == 'ECR88_US1_2P1M_NEWSUCTION'}">
@@ -574,4 +590,12 @@
     <xacro:property name="distPanelTopToLiftPosnX" value="-1.0" scope="global"/> <!-- OEM-FIRMWARE ECR88D_LongArm.m:170 -->
     <xacro:property name="distPanelTopToLiftPosnZ" value="2.0"  scope="global"/>
+    <!-- IMU mounting rotations = rpy(M transpose) of the ECR88D_LongArm.m (2.1 m US unit) imu* matrices. Mounts are PER-UNIT calibration
+         results: pairing a URDF from one unit with a firmware carrying another misreads arm/link by ~4 deg
+         with no fault (sil/tests/test_imu_kinematics.py). -->
+    <xacro:property name="imu_rpy_chs" value="-0.004742750 -0.008549333 -1.762994439" scope="global"/>
+    <xacro:property name="imu_rpy_boom" value="-1.571816342 -0.566316481 -0.000590754" scope="global"/>
+    <xacro:property name="imu_rpy_arm" value="-1.579068528 0.105440054 -0.003310372" scope="global"/>
+    <xacro:property name="imu_rpy_link" value="-1.575935070 0.058856870 0.001290998" scope="global"/>
+    <xacro:property name="imu_rpy_tilt" value="1.549803632 -0.010023128 -1.597706287" scope="global"/>
   </xacro:if>
   <!-- ========================================================================

Commit message: First firmware-in-the-loop run in Isaac Sim: calibration step 28 passes, after it found two model defects
scripts/sil_isaac_step28.py runs the compiled X1Exc firmware inside the Isaac container in
10 ms lockstep with the 1.7 m asset as the plant: physics advances, five IMUs are published
from Isaac's link poses (sil.kinematics), MdlApp_step() runs. Step 28 (CalibForkRefPose:
stb 8 s -> log 1 s -> save) is a pure FK read, so it isolates the IMU chain and geometry.
The oracle applies chart_2352's formula to Isaac ground truth.

Result now:  joints <= 3e-5 deg, angForkUpLimit 1e-4 deg, distUcToForkBack 0.008 mm.
First run:   joints and orientation already exact, position off by (-33, +96) mm.
Link-by-link against MdlApp_Y.links pinned both causes:

1. Tilt chain order (all variants, 10.8 mm). The firmware composes
   tiltMnt = outpLink (+) Ry(angOutpLinkToTiltMnt + angTiltMntToTilt) and translates by
   distTiltMntToTilt in that rotated frame (MdlApp.c:12508, :12659). The URDF rotated by
   angTiltMntToTilt after the translation. The rotation now sits on tilt_mount_joint.
2. Suction head offsets on the 1.7 m unit (92 mm). ECR88D_ShortArm.m carries the new head
   (distAttToProbe 0.255/-0.57, distProbeToContactSurface 0.1/-0.262, the sheet's
   신규흡착기 column); the sheet's 기장 column still had the old one. LongArm.m matches the
   2.1 m variant as built. validate_urdf.py firmware overrides are now per variant.

Also:
- sil/urdf_fk.py, sil/ik.py: FK from the expanded URDF and the planar IK the cycle was
  solved with, usable on the host and in the container.
- sil.kinematics.fourbar_input: inverse of the firmware four-bar. The URDF input_link is a
  1:1 mimic placeholder, so the bktImu attitude published is the real linkage's.
- scripts/make_cycle.py regenerates cycle.json from the asset (was solved in scratch); the
  tilt fix moved the tool ~11 mm, keyframes re-solved to <= 0.2 mm.
- xacro arg model_panel_stack (step 28 is recorded against the bare backrest).

Rebuilt: USDs, site, animation (limits check passes), cameras; check_stability 10/10.
Camera study: cups coverage from arm root / tool / tool side 75 -> 100 %; pick and place
conclusions unchanged.

Co-Authored-By: Claude Opus 5 (1M context) <noreply@anthropic.com>
Claude-Session: https://claude.ai/code/session_01YCTHKLKR3ccjDNMFVWse8H

File: assets/ecr88/urdf/ecr88.urdf.xacro (robot description, xacro)
@@ -211,4 +211,7 @@
        machine actually feeds itself, so it is on by default. -->
   <xacro:arg name="model_fork"          default="true"/>
+  <!-- The module stack on the fork. Off for CalibForkRefPose (step 28), which is recorded with
+       the tool held against the BARE backrest, where the stack would otherwise be. -->
+  <xacro:arg name="model_panel_stack"   default="true"/>
   <!-- Candidate camera/lidar mount frames. Zero mass, no geometry beyond a marker. -->
   <xacro:arg name="model_sensor_mounts" default="true"/>
@@ -968,6 +971,12 @@
     <parent link="output_link"/>
     <child  link="tilt_mount_link"/>
+    <!-- angTiltMntToTilt is applied HERE, on the tilt mount, not on tilt_joint. The firmware
+         composes tiltMnt = outpLink (+) Ry(angOutpLinkToTiltMnt + angTiltMntToTilt) and only then
+         translates by distTiltMntToTilt in that rotated frame (MdlApp.c:12508, :12659). Rotating
+         after the translation, as this file used to, put tilt_link 10.8 mm away from where the
+         firmware computes it (0.356 m lever x 1.736 deg) - found by the first Isaac SIL run
+         (scripts/sil_isaac_step28.py), link-by-link against MdlApp_Y.links. -->
     <origin xyz="${distOutpLinkToTiltMnt_x} ${distOutpLinkToTiltMnt_y} ${distOutpLinkToTiltMnt_z}"
-            rpy="0 ${angOutpLinkToTiltMnt} 0"/>
+            rpy="0 ${angOutpLinkToTiltMnt + angTiltMntToTilt} 0"/>
   </joint>
   <!-- TILT. Axis ASSUMED +X (T3): a tiltrotator tilts the tool sideways, i.e. rolls
@@ -983,5 +992,5 @@
     <child  link="tilt_link"/>
     <origin xyz="${distTiltMntToTilt_x} ${distTiltMntToTilt_y} ${distTiltMntToTilt_z}"
-            rpy="0 ${angTiltMntToTilt} 0"/>
+            rpy="0 0 0"/>
     <axis xyz="1 0 0"/>
     <limit lower="${lim_tilt_lower}" upper="${lim_tilt_upper}"
@@ -1182,4 +1191,5 @@
          cycle and relies on the all-four-cups contact to stop the approach - so the
          OUTER FACE is what has to be right, and it is drawn at panelTop. -->
+    <xacro:if value="$(arg model_panel_stack)">
     <link name="panel_stack_link">
       <xacro:inertial_box mass="${m_panel * panels_per_stack}"
@@ -1196,4 +1206,5 @@
       <origin xyz="0 0 0" rpy="0 0 0"/>
     </joint>
+    </xacro:if>
     <!-- panelTop: the firmware's pick frame. contact_surface must reach this pose. -->
     <link name="panel_top_link">

File: assets/ecr88/urdf/ecr88_params.xacro (robot description, xacro)
@@ -526,10 +526,15 @@
     <xacro:property name="lenToCylLrgBkt2"     value="1.441"   scope="global"/>
     <xacro:property name="angCylLrgBkt"        value="${-pi/180*165.8}" scope="global"/>
-    <xacro:property name="distAttToProbeX"     value="0.35"    scope="global"/>
-    <xacro:property name="distAttToProbeZ"     value="-0.572"  scope="global"/>
+    <!-- 2026-09-15: suction head offsets are the FIRMWARE's for this unit. ECR88D_ShortArm.m:173-174
+         (the 1.7 m unit the repo's binary is compiled with) carries (0.255, 0, -0.57) and
+         (0.1, 0, -0.262) - the sheet's 신규흡착기 values - while the sheet's 기장 column still has
+         the older head (0.35/-0.572, 0.1/-0.264). OEM-FIRMWARE beats the sheet. Found by the
+         Isaac step-28 SIL run: the tool sat 92 mm off the firmware's contact surface. -->
+    <xacro:property name="distAttToProbeX"     value="0.255"   scope="global"/> <!-- OEM-FIRMWARE ShortArm -->
+    <xacro:property name="distAttToProbeZ"     value="-0.57"   scope="global"/> <!-- OEM-FIRMWARE ShortArm -->
     <xacro:property name="distProbeToContactSurfaceX" value="0.1"    scope="global"/>
-    <xacro:property name="distProbeToContactSurfaceZ" value="-0.264" scope="global"/>
-    <xacro:property name="distAttToContactSurfaceX"   value="0.45"   scope="global"/>
-    <xacro:property name="distAttToContactSurfaceZ"   value="-0.836" scope="global"/>
+    <xacro:property name="distProbeToContactSurfaceZ" value="-0.262" scope="global"/> <!-- OEM-FIRMWARE ShortArm -->
+    <xacro:property name="distAttToContactSurfaceX"   value="0.355"  scope="global"/>
+    <xacro:property name="distAttToContactSurfaceZ"   value="-0.832" scope="global"/>
     <xacro:property name="fork_chain_valid"    value="true"    scope="global"/>
     <xacro:property name="angForkUpLimit"      value="${-pi/180*16.3246}" scope="global"/> <!-- OEM-FIRMWARE ECR88D_ShortArm.m:210 -->
