Commit message: Olivia 전체 조인트 limit 반영 (버킷/틸트 실측값 채용)
Slack #simulation 스레드(2026-09-11 11:28 KST)에서 Olivia가 ECR88 기준
전체 조인트 각도를 제공. 앞서 전달받은 암/붐 외에 버킷/틸트/로테이트가 추가로
있었고, 방향 라벨(암아웃/암인, 붐업, 버킷아웃/버킷인)도 함께 확인됨.

  암 : 31(암아웃) ~ 155(암인)
  붐 : -31(붐다운 바닥기준) ~ -69(붐업)
  버킷 : -126(버킷아웃) ~ 43(버킷인)
  틸트 : -45 ~ 45
  로테이트 : -180 ~ 180

- 버킷: -100..+90 -> -126..+43. 종전 값은 Volvo 공표 회전각 190도에서 유도한
  PUBLISHED span + CLASS-TYPICAL 배치였다. 190도는 러그에 직결된 버킷의 값이고,
  틸트로테이터 + PanelLift 헤드가 달린 실기는 169도다. 부호는 가정하지 않고
  FK 로 확인함: 붐 +11.53, 암 +60 고정에서 버킷핀 기준 TCP 가
    -126 -> (+1.488, -0.206) 앞으로 뻗음 = 버킷아웃
     +43 -> (-1.500, -0.081) 접힘      = 버킷인
  Olivia 규약과 동일해 오프셋/부호 변환 없이 그대로 들어감.
- 틸트: ±40(CLASS-TYPICAL, 무출처) -> ±45(OEM-TEAM).
- 로테이트: continuous 유지. -180~180 은 온전한 한 바퀴라 제약이 아니며,
  revolute + ±pi 로 모델링하면 실물에 없는 하드스톱을 wrap 지점에 만들게 된다.
- 암: 방향 라벨이 H3 의 부호 교정을 독립적으로 확인해줌(추론이 아니게 됨).
  배치(0..124)는 여전히 Teo 의 cylinder stroke 가 결정.

USD 재생성. 이번 변환은 종료 크래시 없이 완료.
검증 18 pass / 0 fail.

Co-Authored-By: Claude Opus 5 <noreply@anthropic.com>
Claude-Session: https://claude.ai/code/session_01YCTHKLKR3ccjDNMFVWse8H

File: assets/ecr88/urdf/ecr88_dynamics.xacro (robot description, xacro)
@@ -170,21 +170,45 @@
   <xacro:property name="lim_arm_lower"    value="${deg *   0.00}"/>   <!-- ASSUMPTION [L44], was DERIVED until the H residual was withdrawn (H5)  arm fully OUT, collinear with the boom. NO published figure discriminates this placement. Standing support: it is the standard layout, and the arm cylinder is within 5.6 deg of dead centre here (moment arm 72 mm), so a STRUCTURAL stop belongs about there: prefer a SOFT joint limit. If the true out stop is -10 deg instead, ref_bucket_radius becomes 0.802 and lim_boom_mech_lower becomes -66.56 deg. Teo's cylinder strokes settle it. -->
   <xacro:property name="lim_arm_upper"    value="${deg * 124.00}"/>   <!-- OEM-TEAM span [L43]  arm fully IN (interior angle 56 deg). -->
+  <!-- 2026-09-11 UPDATE, Olivia (Slack #simulation, 11:28 KST). The original relay of her
+       figures carried no direction words; the full message does:
+           "암 : 31(암아웃) ~ 155(암인)"
+       So the angle GROWS as the arm curls IN. That is the same sense as this URDF
+       (positive arm_joint = arm in, established by FK in H3), which independently
+       CONFIRMS the sign correction — it is no longer an inference.
+       It also supports the placement below: 31 = arm fully OUT maps onto lim_arm_lower,
+       and lim_arm_lower is set at the collinear out stop, giving 0..124 with a constant
+       -31 deg offset between machine and URDF frames. What Olivia's numbers still do NOT
+       settle is whether her 31 is measured at the SAME posture as our collinear zero;
+       Teo's cylinder strokes remain the thing that decides it. -->
   <!-- ARM, literal OEM-TEAM placement, sign corrected per H3. One edit away if Olivia
        confirms the interior angle reading. Cylinder infeasible as noted above. -->
   <xacro:property name="lim_arm_oem_lower" value="${deg *  25.00}"/>  <!-- OEM-TEAM literal [L45]  interior angle 155 deg. -->
   <xacro:property name="lim_arm_oem_upper" value="${deg * 149.00}"/>  <!-- OEM-TEAM literal [L45]  interior angle 31 deg. -->
-  <!-- BUCKET (the tool carrier about the bucket pin). The 190 deg SPAN is PUBLISHED and
-       survives the swap from bucket to tiltrotator because it is a property of the
-       cylinder and 4 bar, not of the tool. Only the ZERO moves, and we hold no drawing of
-       the tiltrotator hitch, so the PLACEMENT is class typical: positioned so the tool
-       collinear posture that max reach and max depth both require sits inside the range
-       with about 45 deg of over dump beyond it. -->
-  <xacro:property name="lim_bucket_lower" value="${deg * -100.00}"/>  <!-- PUBLISHED span [L47] + CLASS-TYPICAL placement [L48]  fully dumped / open. -->
-  <xacro:property name="lim_bucket_upper" value="${deg *   90.00}"/>  <!-- PUBLISHED span [L47] + CLASS-TYPICAL placement [L48]  fully curled. Span is exactly 190 deg. -->
-  <!-- TILT. Nothing whatsoever was found on the Xpanner X1 PanelLift or its tiltrotator. -->
-  <xacro:property name="lim_tilt_lower"   value="${deg * -40.00}"/>   <!-- CLASS-TYPICAL, NO SOURCE [L49]  engcon and Rototilt units in the 6-11 t class are 2 x 40 deg; Steelwrist is +/-45. -->
-  <xacro:property name="lim_tilt_upper"   value="${deg *  40.00}"/>   <!-- CLASS-TYPICAL, NO SOURCE [L49] -->
-  <!-- ROTATOR is CONTINUOUS: no lim_rotator_* exists on purpose. The survey corroborates
-       the axis, distRotToAtt being purely -Z (0, 0, -0.2615). [L50] -->
+  <!-- BUCKET (the tool carrier about the bucket pin).
+       SUPERSEDED 2026-09-11 by Olivia (Slack #simulation, 11:28 KST), quoted verbatim:
+           "ECR88 기준입니다 ... 버킷 : -126(버킷아웃) ~ 43(버킷인)"
+       That is the REAL machine as built, with the tiltrotator and PanelLift head fitted.
+       It replaces the previous PUBLISHED-span + CLASS-TYPICAL-placement pair, which read
+       -100..+90 from Volvo's published 190 deg bucket rotation. Span drops 190 -> 169 deg:
+       the published 190 belongs to a bucket on its own lugs, not to this tool stack.
+       SIGN: checked by FK before adopting, not assumed. Holding boom +11.53, arm +60 and
+       sweeping bucket_joint, the TCP measured from the bucket pin goes
+           bucket = -126  ->  (+1.488, -0.206)  reaching forward   = 버킷아웃
+           bucket =  +43  ->  (-1.500, -0.081)  folded back        = 버킷인
+       so negative = out, positive = in, which is Olivia's convention exactly. The numbers
+       transfer with NO offset and NO sign flip. -->
+  <xacro:property name="lim_bucket_lower" value="${deg * -126.00}"/>  <!-- OEM-TEAM [L47]  버킷아웃, fully dumped / open. -->
+  <xacro:property name="lim_bucket_upper" value="${deg *   43.00}"/>  <!-- OEM-TEAM [L47]  버킷인, fully curled. Span 169 deg. -->
+  <!-- TILT.
+       SUPERSEDED 2026-09-11 by Olivia (same message): "틸트 : -45~45".
+       The previous value was a CLASS-TYPICAL +/-40 with no source at all; the note there
+       already observed that Steelwrist units run +/-45, and the real machine is +/-45. -->
+  <xacro:property name="lim_tilt_lower"   value="${deg * -45.00}"/>   <!-- OEM-TEAM [L49] -->
+  <xacro:property name="lim_tilt_upper"   value="${deg *  45.00}"/>   <!-- OEM-TEAM [L49] -->
+  <!-- ROTATOR stays CONTINUOUS: no lim_rotator_* exists on purpose. Olivia's
+       "로테이트 : -180 ~ 180" is the full circle, i.e. it does NOT constrain the joint.
+       A continuous joint already covers it, and modelling it as revolute with +/-pi stops
+       would invent a hard stop at the wrap point that the real rotator does not have.
+       The survey corroborates the axis, distRotToAtt being purely -Z (0, 0, -0.2615). [L50] -->
   <!-- Passive 4 bar dressing branch. The URDF cut is at the conn rod / output link pin,
        so this branch is VISUAL ONLY and carries no load. Wide placeholders. -->

Commit message: 암 2.1m 사양으로 전환 (ECR88_US1_2P1M)
Teo(Slack #simulation, 11:34 KST): "Arm의 경우 저희가 주로 사용하는 사양은
2.1m로 보시면 될 것 같아요". 첨부한 Volvo 치수표도 2.1m 행을 하이라이트.
1.7m(기장)은 파라미터 시트의 첫 열이라 기본값이었을 뿐이다.

machine_variant 를 바꾸면 lenArm 만 움직이는 게 아니라서 따라온 것들:

- 질량/관성/CoM 재계산. 공표 암 어셈블리 280 -> 340 kg 이므로
  m_arm = 340 - 22 - 16 - 1 = 301. 관성은 공표 envelope 2684 x 562 x 305 로
  균일 박스 재산출 -> ixx/iyy/izz = 10.26 / 188.62 / 183.03.
  같은 공식이 기존 1.7m 행(241 kg, 2283x518x305)을 7.26/110.06/106.54 로
  재현하는 것을 먼저 확인하고 적용했다. 총 질량 9149.1 -> 9209.1 kg (+60).
  com_arm_x = 0.40 * lenArm = 0.840.

- 붐 지면 앵커 재계산. 이 값은 lenArm 과 툴 체인의 함수라 variant 를 넘지
  못한다. 지면(z=-1.445) 첫 접촉 붐각을 다시 이분법으로 풀어
    1.7m -> +11.53 (machine->URDF 오프셋 +42.53)
    2.1m -> -27.73 (오프셋 +3.27)
  URDF 붐 범위 -26.47..+11.53 -> -65.73..-27.73.
  덧붙여, 2.1m 에서 Olivia 기계 프레임과 우리 프레임의 오프셋이 3.3도까지
  줄어든다. 그의 각도가 2.1m 장비에서 측정됐을 가능성을 시사한다(확증은 아님).

- 두-출처 버그 하나 더 제거. ecr88_dynamics.xacro 가 params 의 앵커 계산
  결과(-26.47 / 11.53)를 리터럴로 들고 있어서, variant 를 바꿔도 붐 리밋만
  옛 1.7m 배치에 남아 있었다. params property 로부터 유도하도록 변경.

- validate_urdf.py: 기장 열을 하드코딩해 대조하던 것을 variant 인식으로 변경.
  2.1m 빌드에서 lenArm/distArmToInpLink 에 거짓 경고가 났다. 정상 자산에
  뜨는 경고는 없느니만 못하다 - 사람들이 경고 블록을 건너뛰게 만든다.
  ecr88_params.xacro 의 machine_variant 를 읽어 기본값으로 쓰고,
  --variant 로 덮어쓸 수 있다. 거짓 경고 사라짐(5 -> 4 warnings).

USD 재생성 완료, 리밋 반영 확인. 검증 18 pass / 0 fail.

Co-Authored-By: Claude Opus 5 <noreply@anthropic.com>
Claude-Session: https://claude.ai/code/session_01YCTHKLKR3ccjDNMFVWse8H

File: assets/ecr88/urdf/ecr88_dynamics.xacro (robot description, xacro)
@@ -90,5 +90,5 @@
   <xacro:property name="m_house"       value="4966.0"/>  <!-- DERIVED (RESIDUAL) [L9]  8752 minus base, boom, arm assy, bucket, operator. Every error in m_base lands here one for one: this is the largest single uncertainty in the model. Includes the 1 400 kg published counterweight. -->
   <xacro:property name="m_boom"        value="530.0"/>   <!-- PUBLISHED [L2]  Volvo component table, 3.55 m mono boom, "includes cylinder, piping and pin, excludes boom cyl. pin". Taken whole because the URDF models no cylinder links. -->
-  <xacro:property name="m_arm"         value="241.0"/>   <!-- DERIVED from PUBLISHED [L10]  published 280 kg arm assembly ("includes cylinder, linkage and pin") minus the carved out 4 bar: 280 - 22 - 16 - 1. The bucket cylinder stays inside this figure. -->
+  <xacro:property name="m_arm"         value="301.0"/>   <!-- DERIVED from PUBLISHED [L10]  2.1 m dipper. Published 340 kg arm assembly ("includes cylinder, linkage and pin") minus the carved out 4 bar: 340 - 22 - 16 - 1 = 301. The bucket cylinder stays inside this figure. For the 1.7 m arm the published assembly is 280 kg and this becomes 241. Volvo publishes both rows; Teo highlighted 2.1 m as the fleet spec (2026-09-11). -->
   <xacro:property name="m_inp_link"    value="22.0"/>    <!-- CLASS-TYPICAL [L11]  power link, pair of 0.42 m plates approx 20 x 140 mm section plus bosses. -->
   <xacro:property name="m_conn_rod"    value="16.0"/>    <!-- CLASS-TYPICAL [L12]  0.40 m idler link, lighter section than the power link. -->
@@ -134,6 +134,16 @@
        touches ground (z = lenBottomZ1). Kept unchanged from ecr88_params.xacro so the
        team's FK verification still holds. -->
-  <xacro:property name="lim_boom_lower"   value="${deg * -26.47}"/>   <!-- OEM-TEAM span + DERIVED placement [L42]  boom fully UP. -->
-  <xacro:property name="lim_boom_upper"   value="${deg *  11.53}"/>   <!-- OEM-TEAM span + DERIVED placement [L42]  boom DOWN, TCP at ground. -->
+  <!-- These used to hardcode the RESULT of the anchor solve that ecr88_params.xacro
+       performs (deg * -26.47 and deg * 11.53). That made the boom anchor a two-source
+       value: switching machine_variant re-solved bm1GroundContactUrdf in params and
+       these literals silently kept the old 1.7 m placement, so the boom limits did not
+       move with the arm. Derive them from the params properties instead, so the anchor
+       lives in exactly one place.
+         jntBm1Lower/Upper in params compute the same thing; they are the same two
+         numbers by construction and are now unused aliases. -->
+  <xacro:property name="lim_boom_lower"   value="${deg * (bm1GroundContactUrdf - oemBm1AngleSpan)}"/>
+                                      <!-- OEM-TEAM span + DERIVED placement [L42]  boom fully UP. -->
+  <xacro:property name="lim_boom_upper"   value="${deg * bm1GroundContactUrdf}"/>
+                                      <!-- OEM-TEAM span + DERIVED placement [L42]  boom DOWN, TCP at ground. -->
   <!-- BOOM, MECHANICAL envelope. Needed for trenching; the PanelLift range above cannot
        dig at all (38 deg of boom never reaches below ground, and the published 4 130 mm
@@ -302,6 +312,11 @@
   <xacro:property name="inr_boom_ixx" value="73.31"/>  <xacro:property name="inr_boom_iyy" value="669.73"/><xacro:property name="inr_boom_izz" value="606.33"/> <!-- DERIVED [L36], dims PUBLISHED [L31] -->
   <!-- arm_link: box 2.283 x 0.305 x 0.518, Volvo's PUBLISHED component envelope. -->
-  <xacro:property name="com_arm_x" value="0.680"/>     <xacro:property name="com_arm_y" value="0.0"/>   <xacro:property name="com_arm_z" value="0.030"/>  <!-- CLASS-TYPICAL [L29]  0.40 x lenArm: boom end pin bosses and cylinder ears dominate. -->
-  <xacro:property name="inr_arm_ixx" value="7.26"/>    <xacro:property name="inr_arm_iyy" value="110.07"/><xacro:property name="inr_arm_izz" value="106.54"/> <!-- DERIVED [L36], dims PUBLISHED [L32] -->
+  <xacro:property name="com_arm_x" value="0.840"/>     <xacro:property name="com_arm_y" value="0.0"/>   <xacro:property name="com_arm_z" value="0.030"/>  <!-- CLASS-TYPICAL [L29]  0.40 x lenArm = 0.40 x 2.1: boom end pin bosses and cylinder ears dominate. (1.7 m arm: 0.680) -->
+  <xacro:property name="inr_arm_ixx" value="10.26"/>   <xacro:property name="inr_arm_iyy" value="188.62"/><xacro:property name="inr_arm_izz" value="183.03"/> <!-- DERIVED [L36], dims PUBLISHED [L32]
+       2.1 m dipper, uniform box m=301 kg over the published envelope 2684 x 562 x 305 mm
+       (L x H x W): ixx = m/12 (W^2+H^2), iyy = m/12 (L^2+H^2), izz = m/12 (L^2+W^2).
+       The same formula reproduces the 1.7 m row (241 kg, 2283 x 518 x 305) as
+       7.26 / 110.06 / 106.54, which is what this file carried before the variant switch,
+       so the method is unchanged and only the dimensions and mass moved. -->
   <!-- 4 bar members: slender boxes on the surveyed pin to pin lengths. -->
   <xacro:property name="com_gnd_link_x" value="-0.1295"/><xacro:property name="com_gnd_link_y" value="0.0"/><xacro:property name="com_gnd_link_z" value="0.00925"/> <!-- DERIVED, primitive centroid [L30] -->

File: assets/ecr88/urdf/ecr88_params.xacro (robot description, xacro)
@@ -162,8 +162,18 @@
        ======================================================================== -->
   <!-- One of:
-         ECR88_KIJANG              = KinematicPara_new col "ECR88 기장"     (THIS BUILD)
-         ECR88_US1_2P1M            = KinematicPara_new col "ECR88 2.1m 미국#1"
-         ECR88_US1_2P1M_NEWSUCTION = KinematicPara_new col "... 신규흡착기"   -->
-  <xacro:property name="machine_variant"       value="ECR88_KIJANG"/>
+         ECR88_KIJANG              = KinematicPara_new col "ECR88 기장"
+         ECR88_US1_2P1M            = KinematicPara_new col "ECR88 2.1m 미국#1"  (THIS BUILD)
+         ECR88_US1_2P1M_NEWSUCTION = KinematicPara_new col "... 신규흡착기"
+       2026-09-11: switched KIJANG (arm 1.7 m) -> US1_2P1M (arm 2.1 m).
+       Teo (Slack #simulation, 11:34 KST): "Arm의 경우 저희가 주로 사용하는 사양은
+       2.1m로 보시면 될 것 같아요", and the Volvo dimension sheet he attached
+       highlights the 2.1 m dipper row. 2.1 m is the fleet spec; 1.7 m was only ever
+       the default because "기장" is the first column of the parameter sheet.
+       This moves more than lenArm. It also moves distArmToInpLinkX, lenToCylSmlArm2,
+       lenToCylLrgBkt, lenToCylLrgBkt2, angCylLrgBkt (see the branch in section [12]),
+       the arm assembly MASS (280 -> 340 kg published, see ecr88_dynamics.xacro), and
+       it invalidates the boom ground-contact anchor, which was solved with lenArm=1.7
+       and has been re-solved for 2.1 m. -->
+  <xacro:property name="machine_variant"       value="ECR88_US1_2P1M"/>
   <!-- ========================================================================
        [3] MACHINE CONFIGURATION OPTIONS
@@ -584,5 +594,16 @@
        An explicit zero reference replaces this derivation outright.
        -->
-  <xacro:property name="bm1GroundContactUrdf"  value="11.53"/>
+  <!-- 2026-09-11: RE-SOLVED for the 2.1 m arm. This anchor is a function of lenArm and
+       of the whole tool chain below the bucket pin, so it does NOT survive a variant
+       switch and must be re-bisected whenever machine_variant changes.
+           arm 1.7 m  ->  +11.53 deg   (machine->URDF offset +42.53)
+           arm 2.1 m  ->  -27.73 deg   (machine->URDF offset  +3.27)   THIS BUILD
+       Worth noting: on the 2.1 m arm the offset between Olivia's machine frame and this
+       URDF's boom frame collapses to 3.3 deg, i.e. her zero and ours very nearly coincide.
+       On the 1.7 m arm it was 42.5 deg. That is weak evidence that her figures were taken
+       on the 2.1 m machine (the fleet spec) rather than the 1.7 m one. Suggestive, not
+       proof, since the anchor still rests on our own ground-contact assumption. It is
+       another reason to ask her which arm the angles belong to. -->
+  <xacro:property name="bm1GroundContactUrdf"  value="-27.73"/>
                         <!-- DERIVED [deg] boom angle at first ground contact, see above -->
   <xacro:property name="jntBm1Lower"           value="${pi/180*(bm1GroundContactUrdf - oemBm1AngleSpan)}"/>
