Commit message: Adopt the machine's own calibrated parameters from X1Exc firmware
XpannerLab/X1Exc ships ControlModel/Data/ECR88D_LongArm.m and
ECR88D_ShortArm.m: the parameter files the real machine runs on, using the
same parameter names as the release spreadsheet. That makes a direct,
name-by-name comparison possible.

The comparison is a strong result for the asset as it stood: 21 of 22 shared
scalars and 10 of 11 shared vectors agree to 1e-6, variant-specific rows
(lenArm, angCylLrgBkt, lenToCylLrgBkt, distArmToInpLink) included. The
geometry chain is confirmed independently of the sheet it came from.

What changed, all of it a value we had estimated:

  Joint velocities.  Replaced wholesale. reqSpdToActCmd gives each axis a
  requested-speed -> valve-command table whose last X entry is the fastest
  speed the firmware will ever ask for. Ours were 2.0-3.0x too high, and
  consistently so, which pointed at the assumption rather than at arithmetic:
  the pump does not sum onto one function the way the derivation assumed, and
  auto mode caps the valve at 70% (PropVlvCmdAutoLimit). The firmware number
  is the envelope the controller actually commands inside, which is what SIL
  needs. Direction asymmetry is real (boom down 17% faster than boom up); URDF
  carries one velocity per joint, so the limit takes the faster and the pair
  is kept in the new section [4b].

  Valve model, new section [4b].  Per-axis deadband and command ceiling, plus
  PropVlvCmdMinOutpHold (32%), PropVlvCmdAutoLimit (70%) and the 100 Hz sample
  time. Nothing consumes these yet; they sit with their joints so the number is
  in place when the valve model is written.

  angForkUpLimit  -16 deg -> -14.19471 deg. The sheet rounds it and marks the
  row "Update after Calibration"; the firmware carries the calibrated value.
  It is variant specific: the Korean short-arm machine really is -16.3246, so
  the sheet's -16 was that machine's number.

  geo_fork_len  1.45 -> 1.06 m (lenForkBlade, same in both variants).
  geo_panel_t   0.040 -> 0.030 m, and panels_per_stack 30 is now recorded:
                a full stack is 0.90 m of glass.

  distAntMainToChsZ  -1.416 -> -1.345. A genuine conflict: the sheet says
  -1.416 for all three variants, both firmware variants say -1.345. X and Y
  agree exactly, so it is a mount stack height. Following the firmware because
  that is what the position solution is computed with -- but 71 mm is larger
  than the firmware's own placement tolerance (releaseHgt 20 mm), so one of
  the two numbers is stale and it is worth asking which.

validate_urdf.py gains a FIRMWARE_OVERRIDES layer applied after the variant
layer, so the one row where firmware and sheet disagree does not warn forever
on a correct asset. 18 pass, 0 fail.

Co-Authored-By: Claude Opus 5 <noreply@anthropic.com>
Claude-Session: https://claude.ai/code/session_01YCTHKLKR3ccjDNMFVWse8H

File: assets/ecr88/urdf/ecr88_dynamics.xacro (robot description, xacro)
@@ -389,20 +389,66 @@
   <!-- ============================================================================
        [4]  VELOCITY  [rad/s]
-       Derived as flow / bore area / moment arm, assuming the Stage V triple pump
-       (2x68+54 l/min) sums 136 l/min onto one implement function. THAT SUMMATION IS AN
-       ASSUMPTION [L65]. The moment arm collapses at the end stops (and passes through
-       exact zero at the arm cylinder's dead centre), so the instantaneous rate there
-       diverges: 1.0 rad/s covers at least 85 % of each joint's travel and PhysX clamps
-       near the stops, which is correct behaviour anyway.
-       ============================================================================ -->
-  <xacro:property name="vel_swing"    value="${8.3 * 2 * pi / 60}"/> <!-- PUBLISHED [L67]  8.3 r/min = 0.869 rad/s, ECR88D Stage V. SOURCE CONFLICT: the Stage IIIB brochure, the FR T4f brochure and the Volvo US site all say 9.3 r/min (0.974 rad/s). Adopted the Stage V figure to stay consistent with the Stage V mass anchor. -->
-  <xacro:property name="vel_boom"     value="1.0"/>       <!-- DERIVED [L66]  105 mm bore, 136 l/min gives 0.262 m/s rod speed; moment arm runs 0.146 to 0.476 m over the mechanical range, so the joint rate runs 0.55 to 1.80 rad/s. Full stroke in 3.2 s, class norm 3-5 s. -->
-  <xacro:property name="vel_arm"      value="1.0"/>       <!-- DERIVED [L66]  90 mm bore, 0.356 m/s rod speed; moment arm 0.181 to 0.530 m, joint rate 0.67 to 1.97 rad/s. Full stroke in 2.3 s. -->
-  <xacro:property name="vel_bucket"   value="1.0"/>       <!-- DERIVED [L66]  85 mm bore; the 4 bar gives a 0.267 m moment arm at the bucket pin, so 0.75 rad/s on one pump section and 1.50 rad/s flow summed. -->
-  <xacro:property name="vel_tilt"     value="0.5"/>       <!-- CLASS-TYPICAL, NO SOURCE [L68]  about 80 deg of tilt in 3 s. -->
-  <xacro:property name="vel_rotator"  value="1.0"/>       <!-- CLASS-TYPICAL, NO SOURCE [L68]  about 9.5 r/min continuous. Volvo's only tiltrotator relevant published figure is the "slope and rotator" aux circuit: see aux_rotator_flow_lpm in section [7], and note it is 28 l/min on Stage V, NOT the widely quoted Stage IIIB 35. -->
-  <xacro:property name="vel_inp_link" value="1.0"/>       <!-- DERIVED  follows the bucket branch it is driven by. -->
-  <xacro:property name="vel_conn_rod" value="1.0"/>       <!-- GUESS  follows the driven branch; visual only. -->
+       THESE ARE THE MACHINE'S OWN CALIBRATED NUMBERS, not our derivation.
+       XpannerLab/X1Exc  ControlModel/Data/ECR88D_LongArm.m, struct reqSpdToActCmd.
+       Each axis carries a 3 point table  X = [0, 0.001, vmax]  ->  Y = [0, deadband, cmdmax]
+       mapping a REQUESTED JOINT SPEED to a proportional valve command in percent. The
+       last X entry is therefore the fastest speed the firmware will ever ask for, and
+       the last Y entry is the command it asks for there.
+       WHAT THIS REPLACED, AND WHY IT WAS WRONG
+       The previous values here were derived as flow / bore area / moment arm with the
+       Stage V triple pump (2x68+54 l/min) summed onto one function. Every one of them
+       came out 2.0 to 3.0x the firmware number, consistently, which is the signature of
+       a wrong assumption rather than scattered error. Two reasons, both checkable:
+         - the pump does not sum onto one implement function the way that derivation
+           assumed (flagged there as an assumption, [L65]);
+         - auto mode caps the valve at PropVlvCmdAutoLimit = 70 % (SysPar.m:251), and
+           the tables top out at 60-80 %, so the machine never opens the valve fully.
+       For SIL the firmware number is the one that matters: it is the envelope the
+       controller actually commands inside. Keeping a limit 2.4x above it only gives an
+       overshooting drive room to run away to speeds the real machine cannot reach.
+       ASYMMETRY. Every axis is calibrated separately in each direction and they differ
+       (boom down is 17 % faster than boom up; link out is 79 % faster than link in).
+       URDF carries ONE velocity per joint, so the limit below takes the faster of the
+       two and the pair is preserved in section [4b] for the actuator model that needs it.
+       ============================================================================ -->
+  <xacro:property name="vel_swing"    value="0.5889427"/> <!-- OEM-FIRMWARE  swingLe 0.5889 / swingRi 0.5196 rad/s = 5.6 / 5.0 r/min. NOTE this is well under the published free swing speed (8.3 r/min, 0.869 rad/s): swing is the one axis whose command is capped at 60 % instead of 80 %, which is what you would do on a machine carrying glass. The published figure describes the bare ECR88; this one describes it under X1. -->
+  <xacro:property name="vel_boom"     value="0.48"/>      <!-- OEM-FIRMWARE  bm1Up 0.41 / bm1Down 0.48 rad/s -->
+  <xacro:property name="vel_arm"      value="0.43"/>      <!-- OEM-FIRMWARE  armIn 0.38 / armOut 0.43 rad/s -->
+  <xacro:property name="vel_bucket"   value="0.50"/>      <!-- OEM-FIRMWARE  linkIn 0.28 / linkOut 0.50 rad/s. The firmware calls this axis "link", not "bucket": on this machine the cylinder drives the 4 bar input link and the attachment hangs off the output link. Same joint, the firmware's name for it is the more accurate one. -->
+  <xacro:property name="vel_tilt"     value="0.2311245"/> <!-- OEM-FIRMWARE  tiltPosi 0.2033 / tiltNega 0.2311 rad/s -->
+  <xacro:property name="vel_rotator"  value="0.342202"/>  <!-- OEM-FIRMWARE  rotPosi 0.3186 / rotNega 0.3422 rad/s = 3.3 r/min. Our CLASS-TYPICAL guess of 9.5 r/min was 2.9x too fast. -->
+  <xacro:property name="vel_inp_link" value="${vel_bucket}"/> <!-- ALIAS  the link axis above IS this joint. -->
+  <xacro:property name="vel_conn_rod" value="${vel_bucket}"/> <!-- ALIAS  driven branch of the same 4 bar. -->
   <xacro:property name="vel_outp_link" value="${vel_bucket}"/> <!-- ALIAS  same joint as bucket_joint. -->
+  <xacro:property name="vel_dozer"    value="0.5"/>       <!-- GUESS  the blade table is a passthrough (X = Y = [0, 0.001, 80]), i.e. the blade is NOT speed calibrated: it is commanded open loop. No firmware speed exists to take. -->
+  <!-- ============================================================================
+       [4b]  VALVE COMMAND MODEL  [percent]
+       Same source. Needed the moment the firmware is in the loop, because the firmware
+       does not command joint angles, it commands these valves.
+         deadband  the command at which the axis just begins to move (table X = 0.001).
+                   Below it the spool has not cracked and the joint does not move at all.
+         cmdmax    the command at vmax above.
+       Two more from SysPar.m that shape the same signal:
+         PropVlvCmdMinOutpHold = 32 % on every axis  (SysPar.m:230-250)
+             minimum output once moving, to stop the spool hunting around the deadband
+         PropVlvCmdAutoLimit   = 70 %                (SysPar.m:251)
+             ceiling in auto mode, below several of the cmdmax values below
+       Nothing in the URDF consumes these yet. They live here so the number sits with the
+       joint it belongs to when the valve model is written.
+       ============================================================================ -->
+  <xacro:property name="vlv_swing_le"  value="32.0"/>  <xacro:property name="vlv_swing_le_max"  value="60.0"/>
+  <xacro:property name="vlv_swing_ri"  value="28.7"/>  <xacro:property name="vlv_swing_ri_max"  value="60.0"/>
+  <xacro:property name="vlv_boom_up"   value="34.0"/>  <xacro:property name="vlv_boom_up_max"   value="80.0"/>
+  <xacro:property name="vlv_boom_dn"   value="31.0"/>  <xacro:property name="vlv_boom_dn_max"   value="80.0"/>
+  <xacro:property name="vlv_arm_in"    value="27.0"/>  <xacro:property name="vlv_arm_in_max"    value="80.0"/>
+  <xacro:property name="vlv_arm_out"   value="31.0"/>  <xacro:property name="vlv_arm_out_max"   value="80.0"/>
+  <xacro:property name="vlv_link_in"   value="30.0"/>  <xacro:property name="vlv_link_in_max"   value="70.0"/>
+  <xacro:property name="vlv_link_out"  value="31.0"/>  <xacro:property name="vlv_link_out_max"  value="70.0"/>
+  <xacro:property name="vlv_tilt_pos"  value="19.5"/>  <xacro:property name="vlv_tilt_neg"      value="19.5"/>
+  <xacro:property name="vlv_rot_pos"   value="17.5"/>  <xacro:property name="vlv_rot_neg"       value="17.5"/>
+  <xacro:property name="vlv_blade"     value="25.0"/>
+  <xacro:property name="vlv_min_hold"  value="32.0"/>  <!-- SysPar.m:230  every axis -->
+  <xacro:property name="vlv_auto_max"  value="70.0"/>  <!-- SysPar.m:251  auto mode ceiling -->
+  <xacro:property name="ctrl_sample_time" value="0.01"/> <!-- SysPar.m:1  100 Hz, matches the 10 ms CAN3 rate -->
   <!-- ============================================================================
        [5]  JOINT DYNAMICS

File: assets/ecr88/urdf/ecr88_params.xacro (robot description, xacro)
@@ -340,5 +340,17 @@
   <xacro:property name="distAntMainToChsX"     value="0.57"/>
   <xacro:property name="distAntMainToChsY"     value="-0.087"/>
-  <xacro:property name="distAntMainToChsZ"     value="-1.416"/>
+  <!-- CONFLICT, resolved in favour of the firmware. The release sheet says -1.416 for
+       ALL THREE variants; ECR88D_LongArm.m and ECR88D_ShortArm.m both say -1.345, a
+       71 mm difference. X and Y agree exactly in every source, so this is a pure stack
+       height change: same antenna footprint, different mount or spacer. The sheet row is
+       marked "Display on Tablet", i.e. it feeds an operator readout, which is the kind of
+       row that does not get revised when hardware moves. The firmware value is what the
+       machine's position solution is actually computed with, so for SIL it is the one
+       that has to be here.
+       WORTH RAISING WITH OLIVIA: 71 mm is larger than the firmware's own placement
+       tolerance (releaseHgt = 20 mm, releaseEasting/Northing = 20 mm), so whichever
+       number is stale, somebody is placing panels against a shifted reference.
+       Note LenUpZ_est below is derived from this, so the cab roof estimate moves with it. -->
+  <xacro:property name="distAntMainToChsZ"     value="-1.345"/> <!-- OEM-FIRMWARE  (sheet: -1.416) -->
   <!-- AntMain -> AntAux. Dual-antenna heading baseline: |(0.682,0.959,0)|
        = 1.1797 m. Expressed relative to AntMain, NOT to the chassis. -->
@@ -405,6 +417,11 @@
   <!-- 처리구분 = Update after Calibration.
        The ONE row in the whole parameter set that is genuinely a joint LIMIT
-       rather than a mounting offset: -16 deg fork up-limit. -->
-  <xacro:property name="angForkUpLimit"        value="${-pi/180*16}"/>
+       rather than a mounting offset. The sheet gives it to the nearest degree; the
+       firmware carries the calibrated value, and "Update after Calibration" is the
+       sheet telling us to expect exactly that. VARIANT SPECIFIC:
+         ECR88D_LongArm.m  (US, 2.1 m)  -14.19471 deg   <- this build
+         ECR88D_ShortArm.m (KR, 1.7 m)  -16.3246  deg
+       so the sheet's -16 was the Korean machine's number all along. -->
+  <xacro:property name="angForkUpLimit"        value="${-pi/180*14.19471}"/> <!-- OEM-FIRMWARE -->
   <!-- Fork / panel geometry, sheet `old`, reference only -->
   <xacro:property name="LenPLX"                value="1.086"/>
@@ -966,9 +983,10 @@
        .................................................................. -->
   <xacro:property name="geo_fork_clear"        value="0.15"/>   <!-- ASSUMPTION  m, carriage root ahead of the track front -->
-  <xacro:property name="geo_fork_len"          value="1.45"/>    <!-- ASSUMPTION  m, tine length -->
+  <xacro:property name="geo_fork_len"          value="1.06"/>    <!-- OEM-FIRMWARE  m, lenForkBlade. Same 1.06 in BOTH ECR88D_LongArm.m and ECR88D_ShortArm.m, so it is the carriage, not the arm variant. Our 1.45 ASSUMPTION was 37 % long. -->
   <xacro:property name="geo_fork_t"            value="0.07"/>    <!-- ASSUMPTION  m, pallet/backrest plate -->
   <xacro:property name="geo_fork_back_h"       value="1.25"/>    <!-- ASSUMPTION  m, backrest height -->
-  <xacro:property name="geo_panel_t"           value="0.040"/>   <!-- ASSUMPTION  m, one module incl. frame -->
-  <xacro:property name="n_panels"              value="12"/>      <!-- scene choice, not data -->
+  <xacro:property name="geo_panel_t"           value="0.030"/>   <!-- OEM-FIRMWARE  m, panelThickness. Only ECR88D_ShortArm.m carries it; the long arm file has no panel block, so this is the Korean machine's module and the US one may differ. -->
+  <xacro:property name="n_panels"              value="12"/>      <!-- scene choice, not data. A FULL stack is panels_per_stack below; 12 is what we draw so the fork is not hidden behind glass. -->
+  <xacro:property name="panels_per_stack"      value="30"/>      <!-- OEM-FIRMWARE  panelCntPerStack, ECR88D_ShortArm.m. 30 x 30 mm = 0.90 m of glass, which is the height the fork and the pick sequence are designed around. -->
   <xacro:property name="m_panel"               value="23.0"/>    <!-- CLASS-TYPICAL  kg, 72-cell glass-glass -->
   <xacro:property name="m_fork"                value="280.0"/>   <!-- CLASS-TYPICAL  kg, carriage + backrest -->

Commit message: Firmware swings the house in Isaac; joint friction 10 was locking the swing (asset fix)
Positioning in Isaac (scripts/sil_isaac_positioning.py, shared setup in sil/isaac_scene.py): remote
lever 13.0 deg plus 0.31 deg inertial coast, Raise 1.85 s (tool 0.809 m), Swing 2.56 s (peak
15.9 deg/s, no overshoot, ends at 0.08 deg), Align; at rest the firmware's tool position matches
Isaac to 0.01/0.02/0.18 mm.

Asset defect found on the way: the URDF importer writes <dynamics friction> to
physxJoint:jointFriction, which PhysX treats as a unitless coefficient on the joint constraint
force. At 10 the swing joint, carrying the whole house, was locked (0.3 rad/s target -> 0.06 deg
in 1 s, 6 N.m from a 22.9 kN.m drive). dyn_friction is now 0; IsaacPlant also zeroes it at
runtime. With the friction lock gone the free 4-bar connecting rod (1 N.m token) swung as a
pendulum, so eff_conn_rod is 200 N.m. All USDs rebuilt: check_stability 0/10, step 28 unchanged.

docs/FIRMWARE_FINDINGS.md: every firmware finding so far, classified (build configuration /
firmware defect / latent in this build / procedure dependency / plant dependent), with code
locations and the test that reproduces each. Headline: EnTestPar = true (SysPar.m:5) folds every
*Stored inport to parLocalTest, so this build uses no calibration result at runtime.

Co-Authored-By: Claude Opus 5 (1M context) <noreply@anthropic.com>
Claude-Session: https://claude.ai/code/session_01YCTHKLKR3ccjDNMFVWse8H

File: assets/ecr88/urdf/ecr88_dynamics.xacro (robot description, xacro)
@@ -408,5 +408,9 @@
   <xacro:property name="eff_inp_link" value="${cyl_relief_pa * pi / 4 * cyl_bkt_bore * cyl_bkt_bore * lenInpLink}"/>
                                   <!-- DERIVED from PUBLISHED [L62]  = 62 076 N.m. CORRECTED 2026-09-11: this was 70 069 N.m, computed from an 85 mm bucket bore taken as CLASS-TYPICAL. The parts catalogue publishes 80 mm, so the old value was 11 % too high. 29.4 MPa x pi/4 x (80 mm)^2 = 147.8 kN, x lenInpLink 0.42 m. -->
-  <xacro:property name="eff_conn_rod" value="1.0"/>       <!-- GUESS, TOKEN [L63]  idler and the cut member of the 4 bar. No actuator. Do not read joint torque off this branch. -->
+  <xacro:property name="eff_conn_rod" value="200.0"/>     <!-- GUESS [L63]  idler and the cut member of the 4 bar. No actuator. Do not read joint torque off this branch.
+       2026-09-15: was a 1 N.m token. The joint friction coefficient (dyn_friction 10) had been locking this free rod;
+       at friction 0 a 1 N.m drive cannot hold its own weight (16 kg x 9.81 x 0.2 m = 31 N.m) and the rod swung as a
+       pendulum on the input link (check_stability: p-p 0.24 rad, still 0.08 rad at the end). 200 N.m lets the
+       importer's position drive hold it at its opening angle, which is what the friction lock did. -->
   <xacro:property name="eff_outp_link" value="${eff_bucket}"/> <!-- ALIAS  output_link IS the bucket_joint child, so it is the same joint and the same effort. -->
   <!-- ============================================================================
@@ -525,5 +529,12 @@
        ============================================================================ -->
   <xacro:property name="dyn_damping"  value="50.0"/>      <!-- GUESS [L69]  N.m.s/rad, solver hygiene only. -->
-  <xacro:property name="dyn_friction" value="10.0"/>      <!-- GUESS [L69]  N.m, solver hygiene only. -->
+  <!-- dyn_friction MUST stay 0. The Isaac URDF importer writes <dynamics friction> to
+       physxJoint:jointFriction, which PhysX treats as a UNITLESS COEFFICIENT on the joint's
+       constraint force, not as N.m. At 10 the swing joint, which carries the whole house,
+       was locked: a 0.3 rad/s velocity target moved it 0.06 deg in 1 s and a 22.9 kN.m drive
+       delivered 6 N.m (2026-09-15, first firmware swing in Isaac). Boom and arm still moved,
+       so it went unnoticed until the house had to turn. Coulomb friction of a hydraulic axis
+       belongs in the SIL valve model, like the damping note above. -->
+  <xacro:property name="dyn_friction" value="0.0"/>       <!-- [L69] 0 by design, see above (was GUESS 10 N.m) -->
   <!-- ============================================================================
        [6]  CENTRE OF MASS [m] and INERTIA TENSOR [kg.m^2]
